File: PCB/Spiky_Lui.kicad_sch (KiCad schematic)
At the start: 107 parts, among them J1 Oscilloscope, J2 Axon Output, J2 Conn_02x01, J3 Conn_02x01, J3 Stimulus In, J4 Syn1 Input, J5 Syn2 Input, J6 Syn3 Input, Q1 2sk3018, Q1 N_MOSFET, Q2 2sk3018, Q2 N_MOSFET, Q3 2sk3018, Q3 N_MOSFET, Q4 BSS84, Q4 P_MOSFET, Q5 BSS84, Q5 P_MOSFET, Q6 BSS84, Q6 N_MOSFET, Q7 N_MOSFET, Q8 P_MOSFET, Q9 N_MOSFET, SW1 SW_Rotary_1x6_MP, SW1 SW_SPDT, SW2 SW_SPDT, SW3 SW_SPDT, U1 MCP6004, U2 MCP6004, U3 LM339, U4 MCP6004, U5 MCP6004

Commit message: update PCB
Parts:
- removed C1, C7: 1u, Capacitor_SMD:C_0402_1005Metric, symbol Device:C_Small
- removed C10, C11, C12, C13, C14, C17, C9: 100nF, Capacitor_SMD:C_0402_1005Metric, symbol Device:C_Small
- removed C15, C16: 1uF, Capacitor_SMD:C_0402_1005Metric, symbol Device:C_Small
- removed C18: 10uF, Capacitor_SMD:C_0402_1005Metric, symbol Device:C_Small
- removed C2: 2u, Capacitor_SMD:C_0402_1005Metric, symbol Device:C_Small
- removed C3: 3u, Capacitor_SMD:C_0402_1005Metric, symbol Device:C_Small
- removed C4: 5u, Capacitor_SMD:C_0402_1005Metric, symbol Device:C_Small
- removed C5: 10u, Capacitor_SMD:C_0402_1005Metric, symbol Device:C_Small
- removed C6: 20u, Capacitor_SMD:C_0402_1005Metric, symbol Device:C_Small
- removed C8: 10nF, Capacitor_SMD:C_0402_1005Metric, symbol Device:C_Small
- removed D1: 1N4148, Diode_THT:D_DO-35_SOD27_P7.62mm_Horizontal, symbol Diode:1N4148
- removed D2: D_Zener, symbol Device:D_Zener
- removed J1: Oscilloscope, symbol Connector_Audio:AudioJack5
- removed J2, J3: Conn_02x01, Connector_PinHeader_2.54mm:PinHeader_1x02_P2.54mm_Vertical, symbol Connector_Generic:Conn_02x01
- removed J2: Axon Output, symbol Connector_Audio:AudioJack3
- removed J3: Stimulus In, symbol Connector_Audio:AudioJack3
- removed J4: Syn1 Input, symbol Connector_Audio:AudioJack3
- removed J5: Syn2 Input, symbol Connector_Audio:AudioJack3
- removed J6: Syn3 Input, symbol Connector_Audio:AudioJack3
- removed Q1, Q2, Q3: 2sk3018, Package_TO_SOT_SMD:SOT-23, symbol Transistor_FET:2N7002
- removed Q4, Q5, Q6: BSS84, Package_TO_SOT_SMD:SOT-23, symbol Transistor_FET:BSS84
- removed Q8: P_MOSFET, Package_TO_SOT_SMD:SOT-23, symbol Transistor_FET:BSS84
- removed Q9: N_MOSFET, Package_TO_SOT_SMD:SOT-23, symbol Transistor_FET:2N7002
- removed R1, R11, R13, R15, R17, R2, R20, R23, R24, R26, R27, R3: 100k, Resistor_SMD:R_0402_1005Metric, symbol Device:R_Small
- removed R1, R21, R28, R29: 1k, Resistor_SMD:R_0402_1005Metric, symbol Device:R_Small
- removed R10, R30, R34, R36, R37, R7, R9: 22k, Resistor_SMD:R_0402_1005Metric, symbol Device:R_Small
- removed R12, R25: 4.7k, Resistor_SMD:R_0402_1005Metric, symbol Device:R_Small
- removed R14, R16: 1M, Resistor_SMD:R_0402_1005Metric, symbol Device:R_Small
- removed R16, R42, R9: 470, Resistor_SMD:R_0402_1005Metric, symbol Device:R_Small
- removed R18: 70k, Resistor_SMD:R_0402_1005Metric, symbol Device:R_Small
- removed R19, R4, R5, R6 (x2): 10k, Resistor_SMD:R_0402_1005Metric, symbol Device:R_Small
- removed R2, R22: 2k, Resistor_SMD:R_0402_1005Metric, symbol Device:R_Small
- removed R3, R5: 270k, Resistor_SMD:R_0402_1005Metric, symbol Device:R_Small
- removed R31, R35: 2.2k, Resistor_SMD:R_0402_1005Metric, symbol Device:R_Small
- removed R32, R33: 47k, Resistor_SMD:R_0402_1005Metric, symbol Device:R_Small
- removed R4: 56k, Resistor_SMD:R_0402_1005Metric, symbol Device:R_Small
- removed R8: 2.2, Resistor_SMD:R_0402_1005Metric, symbol Device:R_Small
- removed R9: 27k, Resistor_SMD:R_0402_1005Metric, symbol Device:R_Small
- removed RV1, RV3: 100k, Custom:Potentiometer, symbol Device:R_Potentiometer_Small
- removed RV1, RV2, RV3, RV4: 22k, Custom:Potentiometer, symbol Device:R_Potentiometer_Small
- removed RV2: 50k, Custom:Potentiometer, symbol Device:R_Potentiometer_Small
- removed SW1: SW_Rotary_1x6_MP, symbol Switch:SW_Rotary_1x6_MP
- removed SW2, SW3: SW_SPDT, Custom:K3-1296S-E1, symbol Switch:SW_SPDT
- removed U1, U2, U4, U5: MCP6004, Package_SO:TSSOP-14_4.4x5mm_P0.65mm, symbol Amplifier_Operational:MCP6004
- removed unit 4 of U3
- removed unit 3 of U3
- added C1: 220nF, PCM_JLCPCB:C_0603, symbol PCM_JLCPCB-Capacitors:0603,220nF
- added C10, C11, C12, C15, C19, C9: 100nF, PCM_JLCPCB:C_0402, symbol PCM_JLCPCB-Capacitors:0402,100nF
- added C13: 10nF, PCM_JLCPCB:C_0402, symbol PCM_JLCPCB-Capacitors:0402,10nF
- added C14, C16, C17, C3: 1uF, PCM_JLCPCB:C_0402, symbol PCM_JLCPCB-Capacitors:0402,1uF
- added C18, C6, C8: 10uF, PCM_JLCPCB:C_0402, symbol PCM_JLCPCB-Capacitors:0402,10uF
- added C2: 470nF, PCM_JLCPCB:C_0402, symbol PCM_JLCPCB-Capacitors:0402,470nF
- added C4: 2.2uF, PCM_JLCPCB:C_0402, symbol PCM_JLCPCB-Capacitors:0402,2.2uF
- added C5: 4.7uF, PCM_JLCPCB:C_0402, symbol PCM_JLCPCB-Capacitors:0402,4.7uF
- added C7: 22uF, PCM_JLCPCB:C_0603, symbol PCM_JLCPCB-Capacitors:0603,22uF
- added D1: 1N4148W, Maxime:SOD-123_L2.8-W1.8-LS3.7-RD, symbol 1N4148W T41_1N4148W T4-altium-import:root_0_1N4148W_C2099_
- added D2: 1SMA4728A, PCM_JLCPCB:D_DO-214AC(SMA), symbol PCM_JLCPCB-Diodes:Zener,1SMA4728A
- added D3: 19-237/R6GHBHC-A01/2T, Maxime:LED-SMD_4P-L1.6-W1.6-19-237A-BHR6GHC-A01-2T, symbol 19-237_R6GHBHC-A01_2T1_19-237_R6GHBHC-A01_2T-altium-import:root_0_19-237/R6GHBH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
- added J1: Oscilloscope Jack, Maxime:AUDIO-SMD_PJ-320B, symbol PJ-320B1_PJ-320B-altium-import:root_0_PJ-320B贴片_
- added J2: Axon Output, Maxime:AUDIO-SMD_PJ-320B, symbol PJ-320B1_PJ-320B-altium-import:root_0_PJ-320B贴片_
- added J3: Syn1 Input, Maxime:AUDIO-SMD_PJ-320B, symbol PJ-320B1_PJ-320B-altium-import:root_0_PJ-320B贴片_
- added J4: Syn2 Input, Maxime:AUDIO-SMD_PJ-320B, symbol PJ-320B1_PJ-320B-altium-import:root_0_PJ-320B贴片_
- added J5: Syn3 Input, Maxime:AUDIO-SMD_PJ-320B, symbol PJ-320B1_PJ-320B-altium-import:root_0_PJ-320B贴片_
- added J6: Syn4 Input, Maxime:AUDIO-SMD_PJ-320B, symbol PJ-320B1_PJ-320B-altium-import:root_0_PJ-320B贴片_
- added Q10, Q11, Q12, Q9: SI1926DL-T1-E3, Maxime:SOT-363-6_L2.0-W1.3-P0.65-LS2.1-BL, symbol neuron-altium-import:root_0_SI1926DL-T1-E3_
- added Q13, Q14: MMBT2222A, PCM_JLCPCB:Q_SOT-23, symbol PCM_JLCPCB-Transistors:NPN,MMBT2222A
- added Q8: SI3552DV-T1-E3, Maxime:TSOP-6_L3.0-W1.5-P0.95-BL, symbol neuron-altium-import:root_0_SI3552DV-T1-E3_
- added R1: 6.8kΩ, PCM_JLCPCB:R_0402, symbol PCM_JLCPCB-Resistors:0402,6.8kΩ
- added R10, R12, R14, R19, R21, R22, R23, R25, R27, R40, R44, R48, R52, R59: 100kΩ, PCM_JLCPCB:R_0402, symbol PCM_JLCPCB-Resistors:0402,100kΩ
- added R11, R13: 1MΩ, PCM_JLCPCB:R_0402, symbol PCM_JLCPCB-Resistors:0402,1MΩ
- added R15, R18, R31, R32, R33, R36, R9: 22kΩ, PCM_JLCPCB:R_0402, symbol PCM_JLCPCB-Resistors:0402,22kΩ
- added R16: 1Ω, PCM_JLCPCB:R_0402, symbol PCM_JLCPCB-Resistors:0402,1Ω
- added R17: 27kΩ, PCM_JLCPCB:R_0402, symbol PCM_JLCPCB-Resistors:0402,27kΩ
- added R2, R26, R29, R3, R30: 1kΩ, PCM_JLCPCB:R_0402, symbol PCM_JLCPCB-Resistors:0402,1kΩ
- added R20, R28, R55: 4.7kΩ, PCM_JLCPCB:R_0402, symbol PCM_JLCPCB-Resistors:0402,4.7kΩ
- added R24, R4: 2kΩ, PCM_JLCPCB:R_0402, symbol PCM_JLCPCB-Resistors:0402,2kΩ
- added R34, R35, R6: 47kΩ, PCM_JLCPCB:R_0402, symbol PCM_JLCPCB-Resistors:0402,47kΩ
- added R37, R38: 2.4kΩ, PCM_JLCPCB:R_0402, symbol PCM_JLCPCB-Resistors:0402,2.4kΩ
- added R39, R41, R42, R43, R45, R46, R47, R49, R50, R51, R53, R54: 100Ω, PCM_JLCPCB:R_0402, symbol PCM_JLCPCB-Resistors:0402,100Ω
- added R5, R56, R57, R58, R7: 220kΩ, PCM_JLCPCB:R_0402, symbol PCM_JLCPCB-Resistors:0402,220kΩ
- added R60, R62, R63, R8: 10kΩ, PCM_JLCPCB:R_0402, symbol PCM_JLCPCB-Resistors:0402,10kΩ
- added R61: 300kΩ, PCM_JLCPCB:R_0402, symbol PCM_JLCPCB-Resistors:0402,300kΩ
- added R64: 220Ω, PCM_JLCPCB:R_0402, symbol PCM_JLCPCB-Resistors:0402,220Ω
- added RV1, RV3, RV5, RV6, RV7, RV8: 100kΩ, Maxime:RES-ADJ-SMD_G43BT, symbol G43BT-B1041_G43BT-B104-altium-import:root_0_G43BT-B104_
- added RV2: 50kΩ, Maxime:RES-ADJ-SMD_G43BT, symbol G43BT-B5031_G43BT-B503-altium-import:root_0_G43BT-B503_
- added RV4: 10kΩ, Maxime:RES-ADJ-SMD_G43BT, symbol G43BT-B1031_G43BT-B103-altium-import:root_0_G43BT-B103_
- added SW2: RS8160S, Maxime:SW-SMD_RS8160S, symbol RS8160S1_RS8160S-altium-import:root_0_RS8160S_
- added U1, U2, U3, U4: MCP6004T-I/ST, Maxime:TSSOP-14_L5.0-W4.4-P0.65-LS6.4-BL, symbol MCP6004T-I_ST1_MCP6004T-I_ST-altium-import:root_0_MCP6004T-I/ST_
- added unit 3 of U5
- added unit 4 of U5
- BT1: footprint Custom:CR2032_Holder -> Maxime:BAT-TH_CR2032-BS-6-1
- SW1: footprint Custom:K3-1296S-E1 -> Maxime:SW-SMD_SSAJ120100; LCSC C128955 -> C160864
- renumbered U3 to U5
Connections:
- net +0.375: now also U2.2 (VINA-), U2.4 (VDD)
- net +2V: now also C9.1, D2.1, R28.1, R3.2, R4.1, RV1.3, U1.4 (VDD)
- net AP: now also C13.1
- net GNDREF: now also C1.2, C10.2, C11.2, C12.2, C14.2, C15.2, C16.2, C19.2, C2.2, C3.2, C4.2, C5.2, C6.2, C7.2, C8.2, C9.2, J1.1, J2.1, J3.1, J4.1, J5.1, J6.1, Q13.2 (E), Q14.2 (E), R10.2, R11.2, R18.2, R2.2, R23.2, R32.2, R36.2, R38.2, R4.2, R40.1, R44.1, R48.1, R52.1, R57.2, R6.2, RV1.1, RV5.1, RV6.1, RV7.1, RV8.1, U1.11 (VSS), U2.11 (VSS), U3.11 (VSS), U4.11 (VSS)
- net Peak: now also R14.1
- net Reset: now also R19.2, R20.2
- net Reset_Current_Injection: now also U2.1 (VOUTA), U2.3 (VINA+)
- net Spike: now also D1.1 (K), J2.2, R11.1
- net Stimulus_In: now also J1.2
- net Syn1_Spike: now also J3.2, R39.1
- net Syn1_Vm: now also J3.3
- net Syn2_Spike: now also J4.2, R43.1
- net Syn2_Vm: now also J4.3
- net Syn3_Spike: now also J5.2, R47.1
- net Syn3_Vm: now also J5.3
- net VDD: now also SW1.1 (A), C11.1, C12.1, R1.1, R13.2, R14.2, R15.1, R17.1, R20.1, R22.1, R3.1, R31.1, R33.1, R37.1, R5.1, R56.1, R59.1, R64.1, R8.1, R9.1, RV5.3, RV6.3, RV7.3, RV8.3, U3.4 (VDD), U4.4 (VDD); no longer BT1.1 (+)
- net V_Leak: now also RV2.3, U1.1 (VOUTA), U1.2 (VINA-)
- net V_Synapses: now also C18.1, R55.2, RV4.3, U3.6 (VINB-)
- net V_Threshold: now also U5.5 (+), R5.2, R6.1, R7.1
- net Vm: now also J1.3, J2.3, Q8.4 (PD), Q8.6 (ND), R21.2, R30.2, RV2.1, RV2.2, SW2.C, U3.3 (VINA+)
- net at Q4.1 (G), Q5.1 (G): now also R12.2, R13.1
- net at Q2.3 (D): now also R16.2
- net at U5.6 (-): now also C14.1, R15.2, R16.1
- net +BATT: now reaches SW1.2 (B)
- net +BATT: now also BT1.1 (+), C8.1
- net at Q3.3 (D): now also R12.1
- net at U5.7 (+): now also R17.2, R18.1, R19.1
- net at Q1.1 (G), U5.2: now also R7.2, R8.2
- net at Q1.3 (D): now also R9.2
- net at Q7.3 (D): now also R21.1
- new net: C1.1, SW2.1
- new net: Q11.1 (S1), R49.2
- new net: Q11.2 (G1), Q11.5 (G2), R47.2, R48.2
- new net: Q11.3 (D2), Q11.6 (D1), R50.1
- new net: Q10.4 (S2), Q11.4 (S2), Q12.4 (S2), Q9.4 (S2), R42.2, R46.2, R50.2, R54.2, R55.1
- new net: RV6.2, U4.10 (VINC+)
- new net: C4.1, SW2.4
- new net: RV1.2, U1.3 (VINA+)
- new net: R62.1, R63.1, U3.1 (VOUTA), U3.2 (VINA-)
- new net: C2.1, SW2.2
- new net: C3.1, SW2.3
- new net: C5.1, SW2.5
- new net: C6.1, SW2.6
- new net: C7.1, SW2.7 (NC)
- new net: R33.2, R34.1, U3.10 (VINC+)
- new net: C18.2, R34.2, R35.1, RV4.1, RV4.2, U3.7 (VOUTB)
- new net: C19.1, R31.2, R32.1, U3.5 (VINB+)
- new net: R35.2, R36.1, U3.13 (VIND-)
- new net: Q10.2 (G1), Q10.5 (G2), R43.2, R44.2
- new net: Q12.2 (G1), Q12.5 (G2), R51.2, R52.2
- new net: Q12.3 (D2), Q12.6 (D1), R54.1
- new net: Q14.1 (B), R60.1
- new net: R58.2, R59.2, R60.2, R61.1, U5.13
- new net: Q8.1 (NG), U3.14 (VOUTD)
- new net: Q8.2 (PS), R37.2, U3.9 (VINC-)
- new net: Q8.3 (PG), U3.8 (VOUTC)
- new net: Q8.5 (NS), R38.1, U3.12 (VIND+)
- new net: R53.1, U4.1 (VOUTA), U4.2 (VINA-)
- new net: RV8.2, U4.3 (VINA+)
- new net: C15.1, C16.1, R22.2, R23.1, R24.1, R25.2
- new net: Q9.3 (D2), Q9.6 (D1), R42.1
- new net: Q9.1 (S1), R41.2
- new net: Q9.2 (G1), Q9.5 (G2), R39.2, R40.2
- new net: C17.2, R30.1
- new net: R45.1, U4.8 (VOUTC), U4.9 (VINC-)
- new net: R61.2, R62.2, U5.11 (+)
- new net: D2.2, R27.1, R28.2
- new net: R25.1, R27.2, U1.13 (VIND-)
- new net: Q12.1 (S1), R53.2
- new net: Q13.1 (B), R63.2
- new net: D3.1 (R-), Q13.3 (C)
- new net: D3.4 (+), R64.2
- new net: RV5.2, U4.5 (VINB+)
- new net: R41.1, U4.6 (VINB-), U4.7 (VOUTB)
- new net: RV7.2, U4.12 (VIND+)
- new net: C17.1, R29.2
- new net: Q10.1 (S1), R45.2
- new net: Q10.3 (D2), Q10.6 (D1), R46.1
- new net: D3.2 (G-), D3.3 (B-), Q14.3 (C)
- new net: R49.1, U4.13 (VIND-), U4.14 (VOUTD)
- new net: R24.2, R26.1, U1.12 (VIND+)
- new net: R26.2, RV3.1
- new net: R29.1, RV3.2, RV3.3, U1.14 (VOUTD)
- new net +0.375V: C10.1, R1.2, R2.1
- new net Rising_AP: C13.2, D1.2 (A), R10.1
- new net Syn4_Spike: J6.2, R51.1
- new net Syn4_Vm: J6.3
- new net V_Spike_Threshold: R56.2, R57.1, R58.1, U5.10 (-)
- no-connect marks 1 -> 19
Other:
- note added: "τ_membrane = RV2.w(1-w) x Cm, at gLeak default: τ = 6 ms τ = 12.5 ms τ = 25.0 ms τ = 37.5 ms τ = 62.5 ms τ = 125 ms τ = 250 ms"
- note removed: "τ_membrane = RV2.w(1-w) x Cm, at gLeak default: τ = 12.5 ms τ = 25.0 ms τ = 37.5 ms τ = 62.5 ms τ = 125 ms τ = 250 ms"
- moved on the sheet: BT1, U5E
