File: PCB/Spiky_Lui.kicad_pcb (KiCad board)
At the start: 2 copper layers, 98.5 x 59.8 mm, 90 parts, among them J1 Conn_02x01, J2 Conn_02x01, J3 Conn_02x01, J4 Conn_02x03, Q1 2sk3018, Q10 2sk3018, Q11 2sk3018, Q12 2sk3018, Q2 2sk3018, Q3 2sk3018, Q4 BSS84, Q5 BSS84, Q6 BSS84, Q7 SI2301, Q8 SI2302, Q9 2N7002, SW1 SW_SPDT, SW2 SW_SPDT, SW3 SW_SPDT, SW4 SW_SPDT_NO_PRONGS, U1 MCP6004, U2 LM339, U3 LM339

Commit message: update PCB
Parts:
- removed D3, D4, D5, D6, D7: LED_Small, LED_SMD:LED_0402_1005Metric
- removed REF** (x2): Testpad, Custom:Testpad
- removed SW3: SW_SPDT, Custom:K3-1296S-E1
- removed SW4: SW_SPDT_NO_PRONGS, Custom:SSAJ120100
- added .: Spikeling_neuron, Audio_Module:Spikeling_Neuron, F.Cu at (101.5, 83.0)
- added C10: 100nF, PCM_JLCPCB:C_0402, F.Cu at (152.1, 81.0)
- added C11: 100nF, PCM_JLCPCB:C_0402, F.Cu at (116.5, 93.2)
- added C12: 100nF, PCM_JLCPCB:C_0402, F.Cu at (106.7, 72.7)
- added C13: 10nF, PCM_JLCPCB:C_0402, F.Cu at (135.6, 81.5)
- added C14: 1uF, PCM_JLCPCB:C_0402, F.Cu at (110.8, 77.3)
- added C15: 100nF, PCM_JLCPCB:C_0402, F.Cu at (125.8, 92.3)
- added C16: 1uF, PCM_JLCPCB:C_0402, F.Cu at (125.8, 91.2)
- added C17: 1uF, PCM_JLCPCB:C_0402, F.Cu at (125.7, 96.2)
- added C18: 10uF, PCM_JLCPCB:C_0402, F.Cu at (126.5, 87.2)
- added C19: 100nF, PCM_JLCPCB:C_0402, F.Cu at (126.5, 86.1)
- added C8: 10uF, PCM_JLCPCB:C_0402, B.Cu at (94.5, 81.8)
- added J5: Syn3 Input, Maxime:AUDIO-SMD_PJ-320B, B.Cu at (73.4, 104.0)
- added J6: Syn4 Input, Maxime:AUDIO-SMD_PJ-320B, B.Cu at (93.6, 120.5)
- added R43: 100Ω, PCM_JLCPCB:R_0402, F.Cu at (80.6, 99.3)
- added R44: 100kΩ, PCM_JLCPCB:R_0402, F.Cu at (81.5, 97.8)
- added R46: 100Ω, PCM_JLCPCB:R_0402, F.Cu at (83.7, 96.7)
- added R47: 100Ω, PCM_JLCPCB:R_0402, F.Cu at (98.1, 109.6)
- added R48: 100kΩ, PCM_JLCPCB:R_0402, F.Cu at (86.1, 94.2)
- added R49: 100Ω, PCM_JLCPCB:R_0402, F.Cu at (97.6, 111.9)
- added R50: 100Ω, PCM_JLCPCB:R_0402, F.Cu at (94.5, 112.3)
- added R51: 100Ω, PCM_JLCPCB:R_0402, F.Cu at (121.1, 104.2)
- added R52: 100kΩ, PCM_JLCPCB:R_0402, F.Cu at (119.8, 101.8)
- added R53: 100Ω, PCM_JLCPCB:R_0402, F.Cu at (120.3, 103.0)
- added R54: 100Ω, PCM_JLCPCB:R_0402, F.Cu at (119.2, 100.7)
- added R55: 4.7kΩ, PCM_JLCPCB:R_0402, F.Cu at (101.3, 103.6)
- added RV7: 100kΩ, Maxime:RES-ADJ-SMD_G43BT, F.Cu at (93.5, 122.3)
- added RV8: 100kΩ, Maxime:RES-ADJ-SMD_G43BT, F.Cu at (121.9, 116.3)
- added U4: MCP6004T-I/ST, Maxime:TSSOP-14_L5.0-W4.4-P0.65-LS6.4-BL, F.Cu at (111.0, 73.2)
- added U5: LM339, Package_SO:TSSOP-14_4.4x5mm_P0.65mm, F.Cu at (120.3, 78.7)
- BT1: footprint Custom:CR2032_Holder -> Maxime:BAT-TH_CR2032-BS-6-1
- C1: value 100n -> 220nF; footprint Capacitor_SMD:C_0402_1005Metric -> PCM_JLCPCB:C_0603
- C2: value 10u -> 470nF; footprint Capacitor_SMD:C_0402_1005Metric -> PCM_JLCPCB:C_0402
- C3: value 100n -> 1uF; footprint Capacitor_SMD:C_0402_1005Metric -> PCM_JLCPCB:C_0402
- C4: value 100n -> 2.2uF; footprint Capacitor_SMD:C_0402_1005Metric -> PCM_JLCPCB:C_0402
- C5: value 22u ic=0.5 -> 4.7uF; footprint Capacitor_SMD:C_0402_1005Metric -> PCM_JLCPCB:C_0402
- C6: value 100n -> 10uF; footprint Capacitor_SMD:C_0402_1005Metric -> PCM_JLCPCB:C_0402
- C7: value 100n -> 22uF; footprint Capacitor_SMD:C_0402_1005Metric -> PCM_JLCPCB:C_0603
- C9: value 1u ic=2 -> 100nF; footprint Capacitor_SMD:C_0402_1005Metric -> PCM_JLCPCB:C_0402
- D1: value LED_Small -> 1N4148W; footprint LED_SMD:LED_0402_1005Metric -> Maxime:SOD-123_L2.8-W1.8-LS3.7-RD
- D2: value LED_Small -> 1SMA4728A; footprint LED_SMD:LED_0402_1005Metric -> PCM_JLCPCB:D_DO-214AC(SMA)
- J1: value Conn_02x01 -> Oscilloscope Jack; footprint Connector_PinHeader_2.54mm:PinHeader_1x02_P2.54mm_Vertical -> Maxime:AUDIO-SMD_PJ-320B; moved to B.Cu
- J2: value Conn_02x01 -> Axon Output; footprint Connector_PinHeader_2.54mm:PinHeader_1x02_P2.54mm_Vertical -> Maxime:AUDIO-SMD_PJ-320B; moved to B.Cu
- J3: value Conn_02x01 -> Syn1 Input; footprint Connector_PinHeader_2.54mm:PinHeader_1x02_P2.54mm_Vertical -> Maxime:AUDIO-SMD_PJ-320B; moved to B.Cu
- J4: value Conn_02x03 -> Syn2 Input; footprint Connector_PinHeader_2.54mm:PinHeader_2x03_P2.54mm_Vertical -> Maxime:AUDIO-SMD_PJ-320B; moved to B.Cu
- Q1, Q2, Q3: value 2sk3018 -> N_MOSFET
- Q10, Q11, Q12: value 2sk3018 -> SI1926DL-T1-E3; footprint Package_TO_SOT_SMD:SOT-23 -> Maxime:SOT-363-6_L2.0-W1.3-P0.65-LS2.1-BL
- Q4, Q5: value BSS84 -> P_MOSFET
- Q6: value BSS84 -> N_MOSFET
- Q7: value SI2301 -> N_MOSFET
- Q8: value SI2302 -> SI3552DV-T1-E3; footprint Package_TO_SOT_SMD:SOT-23 -> Maxime:TSOP-6_L3.0-W1.5-P0.95-BL
- Q9: value 2N7002 -> SI1926DL-T1-E3; footprint Package_TO_SOT_SMD:SOT-23 -> Maxime:SOT-363-6_L2.0-W1.3-P0.65-LS2.1-BL
- R1: value 100k -> 6.8kΩ; footprint Resistor_SMD:R_0402_1005Metric -> PCM_JLCPCB:R_0402
- R10, R23, R25, R27: value 22k -> 100kΩ; footprint Resistor_SMD:R_0402_1005Metric -> PCM_JLCPCB:R_0402
- R11: value 47k -> 1MΩ; footprint Resistor_SMD:R_0402_1005Metric -> PCM_JLCPCB:R_0402
- R12: value 47k -> 100kΩ; footprint Resistor_SMD:R_0402_1005Metric -> PCM_JLCPCB:R_0402
- R13: value 22k -> 1MΩ; footprint Resistor_SMD:R_0402_1005Metric -> PCM_JLCPCB:R_0402
- R14: value 2.2k -> 100kΩ; footprint Resistor_SMD:R_0402_1005Metric -> PCM_JLCPCB:R_0402
- R15: value 2.2k -> 22kΩ; footprint Resistor_SMD:R_0402_1005Metric -> PCM_JLCPCB:R_0402
- R16: value 470 -> 1Ω; footprint Resistor_SMD:R_0402_1005Metric -> PCM_JLCPCB:R_0402
- R17: value 100k -> 27kΩ; footprint Resistor_SMD:R_0402_1005Metric -> PCM_JLCPCB:R_0402
- R18, R31, R32, R33: value 56k -> 22kΩ; footprint Resistor_SMD:R_0402_1005Metric -> PCM_JLCPCB:R_0402
- R19: value 22 -> 100kΩ; footprint Resistor_SMD:R_0402_1005Metric -> PCM_JLCPCB:R_0402
- R2, R3: value 100k -> 1kΩ; footprint Resistor_SMD:R_0402_1005Metric -> PCM_JLCPCB:R_0402
- R20: value 4.7k -> 4.7kΩ; footprint Resistor_SMD:R_0402_1005Metric -> PCM_JLCPCB:R_0402
- R21: value 100k -> 100kΩ; footprint Resistor_SMD:R_0402_1005Metric -> PCM_JLCPCB:R_0402
- R22: value 27k -> 100kΩ; footprint Resistor_SMD:R_0402_1005Metric -> PCM_JLCPCB:R_0402
- R24, R4: value 10k -> 2kΩ; footprint Resistor_SMD:R_0402_1005Metric -> PCM_JLCPCB:R_0402
- R26: value 2.2 -> 1kΩ; footprint Resistor_SMD:R_0402_1005Metric -> PCM_JLCPCB:R_0402
- R28: value 470k -> 4.7kΩ; footprint Resistor_SMD:R_0402_1005Metric -> PCM_JLCPCB:R_0402
- R29, R30: value 56k -> 1kΩ; footprint Resistor_SMD:R_0402_1005Metric -> PCM_JLCPCB:R_0402
- R34: value 56k -> 47kΩ; footprint Resistor_SMD:R_0402_1005Metric -> PCM_JLCPCB:R_0402
- R35: value 150 -> 47kΩ; footprint Resistor_SMD:R_0402_1005Metric -> PCM_JLCPCB:R_0402
- R36: value 150 -> 22kΩ; footprint Resistor_SMD:R_0402_1005Metric -> PCM_JLCPCB:R_0402
- R37, R38: value 150 -> 2.4kΩ; footprint Resistor_SMD:R_0402_1005Metric -> PCM_JLCPCB:R_0402
- R39: value 150 -> 100Ω; footprint Resistor_SMD:R_0402_1005Metric -> PCM_JLCPCB:R_0402
- R40: value 150 -> 100kΩ; footprint Resistor_SMD:R_0402_1005Metric -> PCM_JLCPCB:R_0402
- R41: value 10 -> 100Ω; footprint Resistor_SMD:R_0402_1005Metric -> PCM_JLCPCB:R_0402
- R42: value 470 -> 100Ω; footprint Resistor_SMD:R_0402_1005Metric -> PCM_JLCPCB:R_0402
- R45: value 100k -> 100Ω; footprint Resistor_SMD:R_0402_1005Metric -> PCM_JLCPCB:R_0402
- R5: value 10k -> 220kΩ; footprint Resistor_SMD:R_0402_1005Metric -> PCM_JLCPCB:R_0402
- R6: value 10k -> 47kΩ; footprint Resistor_SMD:R_0402_1005Metric -> PCM_JLCPCB:R_0402
- R7: value 22k -> 220kΩ; footprint Resistor_SMD:R_0402_1005Metric -> PCM_JLCPCB:R_0402
- R8: value 22k -> 10kΩ; footprint Resistor_SMD:R_0402_1005Metric -> PCM_JLCPCB:R_0402
- R9: value 470 -> 22kΩ; footprint Resistor_SMD:R_0402_1005Metric -> PCM_JLCPCB:R_0402
- RV1, RV3: value 22k -> 100kΩ; footprint Custom:Potentiometer -> Maxime:RES-ADJ-SMD_G43BT
- RV2: value 22k -> 50kΩ; footprint Custom:Potentiometer -> Maxime:RES-ADJ-SMD_G43BT
- RV4: value 22k -> 10kΩ; footprint Custom:Potentiometer -> Maxime:RES-ADJ-SMD_G43BT
- RV5: value 100k -> 100kΩ; footprint Custom:Potentiometer -> Maxime:RES-ADJ-SMD_G43BT
- RV6: value 50k -> 100kΩ; footprint Custom:Potentiometer -> Maxime:RES-ADJ-SMD_G43BT
- SW1: footprint Custom:K3-1296S-E1 -> Maxime:SW-SMD_SSAJ120100; moved to B.Cu
- SW2: value SW_SPDT -> RS8160S; footprint Custom:K3-1296S-E1 -> Maxime:SW-SMD_RS8160S
- U1: value MCP6004 -> MCP6004T-I/ST; footprint Package_SO:TSSOP-14_4.4x5mm_P0.65mm -> Maxime:TSSOP-14_L5.0-W4.4-P0.65-LS6.4-BL
- U2, U3: value LM339 -> MCP6004T-I/ST; footprint Package_SO:TSSOP-14_4.4x5mm_P0.65mm -> Maxime:TSSOP-14_L5.0-W4.4-P0.65-LS6.4-BL
- moved J2 124.4 mm to (171.5, 82.5), turned to 90 degrees
- moved Q6 93.2 mm to (162.4, 81.5)
- moved Q7 87.4 mm to (166.4, 81.4), turned to 0 degrees
- moved Q5 84.2 mm to (148.5, 80.3), turned to 0 degrees
- moved Q3 80.1 mm to (140.7, 80.6), turned to 0 degrees
- moved Q4 75.3 mm to (144.6, 80.5)
- moved J3 70.0 mm to (121.9, 116.3), turned to 0 degrees
- moved J4 68.9 mm to (68.7, 71.6), turned to -90 degrees
- moved Q1 63.5 mm to (127.5, 78.8), turned to 0 degrees
- moved U2 63.2 mm to (156.5, 81.5), turned to -90 degrees
- moved R21 63.0 mm to (152.1, 82.9)
- moved Q2 57.5 mm to (107.7, 78.8), turned to 0 degrees
- moved R14 54.8 mm to (137.6, 80.6), turned to 0 degrees
- moved RV2 53.2 mm to (110.6, 89.0), turned to 0 degrees
- moved R5 52.7 mm to (115.2, 78.7)
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Connections:
- BT1 pad 1: VDD -> +BATT
- BT1 pad 2: GNDPWR -> GNDREF
- C1 pad 1: GND -> Net-(C1-Pad1)
- C1 pad 2: Net-(U1B-+) -> GNDREF
- C2 pad 1: Net-(U1B--) -> Net-(C2-Pad1)
- C2 pad 2: /VSYN -> GNDREF
- C3 pad 1: GND -> Net-(C3-Pad1)
- C3 pad 2: VDD -> GNDREF
- C4 pad 1: GND -> Net-(C4-Pad1)
- C4 pad 2: VDD -> GNDREF
- C5 pad 1: /MEM -> Net-(C5-Pad1)
- C5 pad 2: GND -> GNDREF
- C6 pad 1: GND -> Net-(C6-Pad1)
- C6 pad 2: VDD -> GNDREF
- C7 pad 1: GND -> Net-(SW2-NC)
- C7 pad 2: VDD -> GNDREF
- C9 pad 1: /REFR -> +2V
- C9 pad 2: GND -> GNDREF
- D1 pad 1: Net-(D1-K) -> Spike
- D1 pad 2: VDD -> /Rising_AP
- D2 pad 1: Net-(D2-K) -> VDD
- D2 pad 2: VDD -> Net-(D2-Pad2)
- J1 pad 1: GND -> GNDREF
- J1 pad 2: /INPUT_0 -> Stimulus_In
- J2 pad 1: GND -> GNDREF
- J2 pad 2: /INPUT_1 -> Spike
- J3 pad 1: GND -> GNDREF
- J3 pad 2: /INPUT_3 -> Syn1_Spike
- J4 pad 1: GND -> GNDREF
- J4 pad 2: /RESET -> Syn2_Spike
- J4 pad 3: GND -> Syn2_Vm
- Q1 pad 1: /INPUT_0 -> Net-(Q1-G)
- Q1 pad 2: GND -> AP
- Q10 pad 1: Net-(Q10-G) -> Net-(Q10-S1)
- Q10 pad 2: GND -> Net-(Q10-G1)
- Q10 pad 3: /SPK -> Net-(Q10-D1)
- Q11 pad 1: /SPK -> Net-(Q11-S1)
- Q11 pad 2: GND -> Net-(Q11-G1)
- Q11 pad 3: Net-(Q11-D) -> Net-(Q11-D1)
- Q12 pad 1: /RESET -> Net-(Q12-S1)
- Q12 pad 2: GND -> Net-(Q12-G1)
- Q12 pad 3: /VU7 -> Net-(Q12-D1)
- Q2 pad 1: /INPUT_1 -> AP
- Q2 pad 2: GND -> GNDREF
- Q3 pad 1: /INPUT_3 -> Spike
- Q3 pad 2: GND -> GNDREF
- Q4 pad 3: Net-(Q4-D) -> Vm
- Q5 pad 1: Net-(Q5-G) -> Net-(Q4-G)
- Q5 pad 2: VDD -> Peak
- Q5 pad 3: Net-(Q5-D) -> GNDREF
- Q6 pad 1: Net-(Q6-G) -> Peak
- Q6 pad 2: VDD -> /Reset_Current_Injection
- Q7 pad 1: Net-(Q7-G) -> Reset
- Q7 pad 2: Net-(Q7-S) -> Net-(Q6-D)
- Q7 pad 3: /MEM -> Net-(Q7-D)
- Q8 pad 1: Net-(Q8-G) -> Net-(Q8-NG)
- Q8 pad 2: Net-(Q8-S) -> Net-(Q8-PS)
- Q8 pad 3: /MEM -> Net-(Q8-PG)
- Q9 pad 1: /RESET -> Net-(Q9-S1)
- Q9 pad 2: GND -> Net-(Q9-G1)
- Q9 pad 3: Net-(Q9-D) -> Net-(Q9-D1)
- R1 pad 1: /INPUT_0 -> VDD
- R1 pad 2: GND -> +0.375V
- R10 pad 1: VDD -> /Rising_AP
- R10 pad 2: Net-(U1C-+) -> GNDREF
- R11 pad 1: Net-(U1C-+) -> Spike
- R11 pad 2: /VSYN -> GNDREF
- R12 pad 1: /VSYN -> Net-(Q3-D)
- R12 pad 2: Net-(U1D-+) -> Net-(Q4-G)
- R13 pad 1: Net-(U1D-+) -> Net-(Q4-G)
- R13 pad 2: GND -> VDD
- R14 pad 1: VDD -> Peak
- R14 pad 2: Net-(Q7-S) -> VDD
- R15 pad 1: Net-(Q8-S) -> VDD
- R15 pad 2: GND -> Net-(U5B--)
- R16 pad 1: Net-(R16-Pad1) -> Net-(U5B--)
- R16 pad 2: Net-(U1B--) -> Net-(Q2-D)
- R17 pad 1: Net-(U3B-+) -> VDD
- R17 pad 2: VDD -> Net-(U5B-+)
- R18 pad 1: GND -> Net-(U5B-+)
- R18 pad 2: Net-(U3B-+) -> GNDREF
- R19 pad 1: /MEM -> Net-(U5B-+)
- R19 pad 2: Net-(Q9-D) -> Reset
- R2 pad 1: /INPUT_1 -> +0.375V
- R2 pad 2: GND -> GNDREF
- R20 pad 1: /RESET -> VDD
- R20 pad 2: VDD -> Reset
- R21 pad 1: Net-(U3B-+) -> Net-(Q7-D)
- R21 pad 2: Net-(Q10-G) -> Vm
- R22 pad 2: Net-(U3A-+) -> Net-(C15-Pad1)
- R23 pad 1: Net-(U3A-+) -> Net-(C15-Pad1)
- R23 pad 2: GND -> GNDREF
- R24 pad 1: Net-(Q10-G) -> Net-(C15-Pad1)
- R24 pad 2: VDD -> Net-(U3D-VINA-)
- R25 pad 1: /SPK -> Net-(U3D-VINA+)
- R25 pad 2: VDD -> Net-(C15-Pad1)
- R26 pad 1: Net-(Q11-D) -> Net-(U3D-VINA-)
- R26 pad 2: /REFR -> Net-(R26-Pad2)
- R27 pad 1: /REFR -> Net-(D2-Pad2)
- R27 pad 2: VDD -> Net-(U3D-VINA+)
- R28 pad 2: Net-(U2D-+) -> Net-(D2-Pad2)
- R29 pad 1: Net-(U2D-+) -> Net-(U3D-VOUTA)
- R29 pad 2: Net-(U2C-+) -> Net-(C17-Pad1)
- R3 pad 1: /INPUT_3 -> VDD
- R3 pad 2: GND -> +2V
- R30 pad 1: Net-(U2C-+) -> Net-(C17-Pad2)
- R30 pad 2: Net-(U2B-+) -> Vm
- R31 pad 1: Net-(U2B-+) -> VDD
- R31 pad 2: Net-(U2A-+) -> Net-(U3A-VINB+)
- R32 pad 1: Net-(U2A-+) -> Net-(U3A-VINB+)
- R32 pad 2: Net-(U3C-+) -> GNDREF
- R33 pad 1: Net-(U3C-+) -> VDD
- R33 pad 2: Net-(U3D-+) -> Net-(U3B-VINC+)
- R34 pad 1: Net-(U3D-+) -> Net-(U3B-VINC+)
- R34 pad 2: GND -> Net-(U3A-VOUTB)
- R35 pad 1: /VU6 -> Net-(U3A-VOUTB)
- R35 pad 2: Net-(D2-K) -> Net-(U3C-VIND-)
- R36 pad 1: /VU5 -> Net-(U3C-VIND-)
- R36 pad 2: Net-(D3-K) -> GNDREF
- R37 pad 1: /VU4 -> VDD
- R37 pad 2: Net-(D4-K) -> Net-(Q8-PS)
- R38 pad 1: /VU3 -> Net-(Q8-NS)
- R38 pad 2: Net-(D5-K) -> GNDREF
- R39 pad 1: /VU2 -> Syn1_Spike
- R39 pad 2: Net-(D6-K) -> Net-(Q9-G1)
- R4 pad 1: VDD -> +2V
- R4 pad 2: Net-(Q4-G) -> GNDREF
- R40 pad 1: /VU1 -> GNDREF
- R40 pad 2: Net-(D7-K) -> Net-(Q9-G1)
- R41 pad 1: /VU7 -> Net-(U4A-VINB-)
- R41 pad 2: Net-(D1-K) -> Net-(Q9-S1)
- R42 pad 1: Net-(R42-Pad1) -> Net-(Q9-D1)
- R42 pad 2: Net-(U1B--) -> Net-(Q10-S2)
- R45 pad 1: /RESET -> Net-(U4B-VINC-)
- R45 pad 2: Net-(U3A-+) -> Net-(Q10-S1)
- R5 pad 2: Net-(Q5-G) -> /V_Threshold
- R6 pad 1: VDD -> /V_Threshold
- R6 pad 2: Net-(Q6-G) -> GNDREF
- R7 pad 1: VDD -> /V_Threshold
- R7 pad 2: Net-(U1B-+) -> Net-(Q1-G)
- R8 pad 1: Net-(U1B-+) -> VDD
- R8 pad 2: GND -> Net-(Q1-G)
- R9 pad 1: Net-(R9-Pad1) -> VDD
- R9 pad 2: Net-(U1B--) -> Net-(Q1-D)
- RV1 pad 1: Net-(Q4-D) -> GNDREF
- RV1 pad 2: Net-(R9-Pad1) -> Net-(U1D-VINA+)
- RV1 pad 3: Net-(R9-Pad1) -> +2V
- RV2 pad 1: Net-(Q5-D) -> Vm
- RV2 pad 2: Net-(R16-Pad1) -> Vm
- RV2 pad 3: Net-(R16-Pad1) -> /V_Leak
- RV3 pad 1: Net-(Q6-D) -> Net-(R26-Pad2)
- RV3 pad 2: Net-(R42-Pad1) -> Net-(U3D-VOUTA)
- RV3 pad 3: Net-(R42-Pad1) -> Net-(U3D-VOUTA)
- RV4 pad 1: /VSYN -> Net-(U3A-VOUTB)
- RV4 pad 2: /VSYN -> Net-(U3A-VOUTB)
- RV4 pad 3: Net-(U1B--) -> V_Synapses
- RV5 pad 1: VDD -> GNDREF
- RV5 pad 2: Net-(U1A-+) -> Net-(U4A-VINB+)
- RV5 pad 3: GND -> VDD
- RV6 pad 1: /MEM -> GNDREF
- RV6 pad 2: /MEM -> Net-(U4B-VINC+)
- RV6 pad 3: /VLEAK -> VDD
- SW1 pad 1: Net-(Q4-D) -> VDD
- SW1 pad 2: Net-(Q1-D) -> +BATT
- SW2 pad 1: Net-(Q5-G) -> Net-(C1-Pad1)
- SW2 pad 2: Net-(Q2-D) -> Net-(C2-Pad1)
- SW2 pad 3: Net-(Q5-D) -> Net-(C3-Pad1)
- U1 pad 1: /VLEAK -> /V_Leak
- U1 pad 10: Net-(U1C-+) -> unconnected-(U1B-VINC+-Pad10)
- U1 pad 11: GND -> GNDREF
- U1 pad 12: Net-(U1D-+) -> unconnected-(U1C-VIND+-Pad12)
- U1 pad 13: Net-(Q8-S) -> unconnected-(U1C-VIND--Pad13)
- U1 pad 14: Net-(Q8-G) -> unconnected-(U1C-VOUTD-Pad14)
- U1 pad 2: /VLEAK -> /V_Leak
- U1 pad 3: Net-(U1A-+) -> Net-(U1D-VINA+)
- U1 pad 4: VDD -> +2V
- U1 pad 5: Net-(U1B-+) -> unconnected-(U1A-VINB+-Pad5)
- U1 pad 6: Net-(U1B--) -> unconnected-(U1A-VINB--Pad6)
- U1 pad 7: /VSYN -> unconnected-(U1A-VOUTB-Pad7)
- U1 pad 8: Net-(Q7-G) -> unconnected-(U1B-VOUTC-Pad8)
- U1 pad 9: Net-(Q7-S) -> unconnected-(U1B-VINC--Pad9)
- U2 pad 1: /VU4 -> /Reset_Current_Injection
- U2 pad 10: /MEM -> unconnected-(U2B-VINC+-Pad10)
- U2 pad 11: Net-(U2C-+) -> GNDREF
- U2 pad 12: GND -> unconnected-(U2C-VIND+-Pad12)
- U2 pad 13: /VU5 -> unconnected-(U2C-VIND--Pad13)
- U2 pad 14: /VU6 -> unconnected-(U2C-VOUTD-Pad14)
- U2 pad 2: /VU3 -> +0.375
- U2 pad 3: VDD -> /Reset_Current_Injection
- U2 pad 4: /MEM -> +0.375
- U2 pad 5: Net-(U2A-+) -> unconnected-(U2A-VINB+-Pad5)
- U2 pad 6: /MEM -> unconnected-(U2A-VINB--Pad6)
- U2 pad 7: Net-(U2B-+) -> unconnected-(U2A-VOUTB-Pad7)
- U2 pad 8: /MEM -> unconnected-(U2B-VOUTC-Pad8)
- U2 pad 9: Net-(U2D-+) -> unconnected-(U2B-VINC--Pad9)
- U3 pad 1: Net-(Q10-G) -> Net-(U3D-VOUTA)
- U3 pad 10: /MEM -> Net-(U3B-VINC+)
- U3 pad 11: Net-(U3C-+) -> GNDREF
- U3 pad 12: GND -> Net-(Q8-NS)
- U3 pad 13: /VU2 -> Net-(U3C-VIND-)
- U3 pad 14: /VU1 -> Net-(Q8-NG)
- U3 pad 2: /RESET -> Net-(U3D-VINA-)
- U3 pad 3: VDD -> Net-(U3D-VINA+)
- U3 pad 4: /REFR -> VDD
- U3 pad 5: Net-(U3A-+) -> Net-(U3A-VINB+)
- U3 pad 6: /MEM -> V_Synapses
- U3 pad 7: Net-(U3B-+) -> Net-(U3A-VOUTB)
- U3 pad 8: /MEM -> Net-(Q8-PG)
- U3 pad 9: Net-(U3D-+) -> Net-(Q8-PS)
Routing:
- net /RESET: track 100.0 -> 0.00 mm, vias 6 -> 0
- net /MEM: track 81.2 -> 0.00 mm, vias 4 -> 0
- net Net-(U1B--): track 67.7 -> 0.00 mm, vias 5 -> 0
- net VDD: track 62.3 -> 0.00 mm, vias 18 -> 0
- net /VU6: track 49.5 -> 0.00 mm, vias 2 -> 0
- net /VU5: track 45.9 -> 0.00 mm, vias 2 -> 0
- net /VU7: track 43.4 -> 0.00 mm
- net /VU4: track 37.0 -> 0.00 mm, vias 2 -> 0
- net /VU3: track 34.3 -> 0.00 mm, vias 2 -> 0
- net /VU2: track 30.5 -> 0.00 mm, vias 2 -> 0
- net /VSYN: track 24.6 -> 0.00 mm, vias 2 -> 0
- net Net-(Q10-G): track 24.0 -> 0.00 mm, vias 2 -> 0
- net /VU1: track 21.4 -> 0.00 mm, vias 2 -> 0
- net /REFR: track 18.7 -> 0.00 mm, vias 2 -> 0
- net Net-(U3A-+): track 18.6 -> 0.00 mm, vias 3 -> 0
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- removed copper zone on B.Cu, net /MEM
- removed copper zone on F.Cu, net /MEM
- removed copper zone on B.Cu, net GND
- removed copper zone on F.Cu, net GND
- removed copper zone on B.Cu, net GNDPWR
- removed copper zone on F.Cu, net GNDPWR
- removed copper zone on B.Cu, net VDD
Other:
- board size 98.5 x 59.8 mm -> 6.2 x 4.7 mm
- board text removed: "+"
- board text removed: "-"
- board text removed: "1"
- board text removed: "2"
- board text removed: "3"
- board text removed: "Lu.i 03/2025 - giantaxon.org"
- board text removed: "V"
- board text removed: "from Heidelberg & Bern made with by YS, SB & JG"
- board text removed: "leak"
- board text removed: "mem"
- board text removed: "syn"
- board text removed: "w"
- board text removed: "τ"
- board text removed: "⎍"
- board text removed: "⏚"

Commit message: update PCB
Parts:
- removed .: Spikeling_neuron, Audio_Module:Spikeling_Neuron
- removed C1: 220nF, PCM_JLCPCB:C_0603
- removed C7: 22uF, PCM_JLCPCB:C_0603
- removed SW2: RS8160S, Maxime:SW-SMD_RS8160S
- added C20: 100nF, PCM_JLCPCB:C_0402, F.Cu at (89.7, 88.8)
- added D3: 1N4148WS, PCM_JLCPCB:D_SOD-323, F.Cu at (85.5, 89.4)
- added D4: 1N4148WS, PCM_JLCPCB:D_SOD-323, F.Cu at (85.5, 87.2)
- added D5: 1N4148WS, PCM_JLCPCB:D_SOD-323, F.Cu at (85.5, 85.0)
- added G***: LOGO, Maxime:spiky_pcb, F.Cu at (118.0, 100.4)
- added H1: MountingHole, MountingHole:MountingHole_2.2mm_M2, F.Cu at (75.1, 122.0)
- added H2: MountingHole, MountingHole:MountingHole_2.2mm_M2, F.Cu at (102.9, 131.1)
- added H3: MountingHole, MountingHole:MountingHole_2.2mm_M2, F.Cu at (127.1, 110.6)
- added H4: MountingHole, MountingHole:MountingHole_2.2mm_M2, F.Cu at (168.0, 66.4)
- added H5: MountingHole, MountingHole:MountingHole_2.2mm_M2, F.Cu at (95.4, 75.3)
- added H6: MountingHole, MountingHole:MountingHole_2.2mm_M2, F.Cu at (64.8, 84.3)
- added Q13: MMBT2222A, PCM_JLCPCB:Q_SOT-23, F.Cu at (115.8, 83.7)
- added Q14: MMBT2222A, PCM_JLCPCB:Q_SOT-23, F.Cu at (115.8, 79.9)
- added Q15: MMBT3904, Package_TO_SOT_SMD:SOT-23, F.Cu at (102.4, 75.2)
- added Q16: N_MOSFET, Package_TO_SOT_SMD:SOT-23, F.Cu at (91.1, 79.2)
- added Q17: N_MOSFET, Package_TO_SOT_SMD:SOT-23, F.Cu at (75.2, 115.8)
- added Q18: N_MOSFET, Package_TO_SOT_SMD:SOT-23, F.Cu at (97.5, 122.4)
- added Q19: N_MOSFET, Package_TO_SOT_SMD:SOT-23, F.Cu at (121.1, 111.0)
- added Q20: N_MOSFET, Package_TO_SOT_SMD:SOT-23, F.Cu at (97.7, 79.2)
- added R56: 220kΩ, PCM_JLCPCB:R_0402, F.Cu at (119.2, 83.8)
- added R57: 220kΩ, PCM_JLCPCB:R_0402, F.Cu at (119.2, 82.5)
- added R58: 220kΩ, PCM_JLCPCB:R_0402, F.Cu at (122.0, 80.9)
- added R59: 100kΩ, PCM_JLCPCB:R_0402, F.Cu at (119.2, 81.2)
- added R60: 10kΩ, PCM_JLCPCB:R_0402, F.Cu at (122.0, 79.6)
- added R61: 300kΩ, PCM_JLCPCB:R_0402, F.Cu at (122.0, 82.2)
- added R62: 10kΩ, PCM_JLCPCB:R_0402, F.Cu at (119.2, 79.9)
- added R63: 10kΩ, PCM_JLCPCB:R_0402, F.Cu at (112.3, 79.9)
- added R64: 220Ω, PCM_JLCPCB:R_0402, F.Cu at (112.4, 84.1)
- added R65: 100kΩ, PCM_JLCPCB:R_0402, F.Cu at (80.2, 85.8)
- added R66: 100kΩ, PCM_JLCPCB:R_0402, F.Cu at (82.5, 84.5)
- added R67: 1MΩ, PCM_JLCPCB:R_0402, F.Cu at (90.3, 76.8)
- added R68: 100kΩ, PCM_JLCPCB:R_0402, F.Cu at (90.3, 75.5)
- added R69: 1MΩ, PCM_JLCPCB:R_0402, F.Cu at (105.7, 79.8)
- added R70: 100kΩ, PCM_JLCPCB:R_0402, F.Cu at (105.7, 78.5)
- added R71: 1MΩ, PCM_JLCPCB:R_0402, F.Cu at (77.5, 113.2)
- added R72: 100kΩ, PCM_JLCPCB:R_0402, F.Cu at (76.4, 110.6)
- added R73: 1MΩ, PCM_JLCPCB:R_0402, F.Cu at (77.5, 111.9)
- added R74: 1MΩ, PCM_JLCPCB:R_0402, F.Cu at (91.9, 123.9)
- added R75: 1MΩ, PCM_JLCPCB:R_0402, F.Cu at (94.4, 122.8)
- added R76: 100kΩ, PCM_JLCPCB:R_0402, F.Cu at (91.9, 125.2)
- added R77: 1MΩ, PCM_JLCPCB:R_0402, F.Cu at (123.1, 109.7)
- added R78: 1MΩ, PCM_JLCPCB:R_0402, F.Cu at (117.1, 112.3)
- added R79: 100kΩ, PCM_JLCPCB:R_0402, F.Cu at (116.0, 109.7)
- added R80: 100kΩ, PCM_JLCPCB:R_0402, F.Cu at (88.0, 75.5)
- added R81: 1MΩ, PCM_JLCPCB:R_0402, F.Cu at (88.0, 76.8)
- added R82: 10Ω, PCM_JLCPCB:R_0402, F.Cu at (94.1, 79.2)
- added R83: 100kΩ, PCM_JLCPCB:R_0402, F.Cu at (77.5, 114.5)
- added R84: 1MΩ, PCM_JLCPCB:R_0402, F.Cu at (75.2, 113.2)
- added R85: 10Ω, PCM_JLCPCB:R_0402, F.Cu at (77.5, 117.1)
- added R86: 100kΩ, PCM_JLCPCB:R_0402, F.Cu at (94.4, 121.5)
- added R87: 1MΩ, PCM_JLCPCB:R_0402, F.Cu at (97.1, 119.8)
- added R88: 10Ω, PCM_JLCPCB:R_0402, F.Cu at (99.0, 120.8)
- added R89: 100kΩ, PCM_JLCPCB:R_0402, F.Cu at (117.1, 111.0)
- added R90: 1MΩ, PCM_JLCPCB:R_0402, F.Cu at (114.8, 112.3)
- added R91: 10Ω, PCM_JLCPCB:R_0402, F.Cu at (123.1, 112.3)
- added R92: 100kΩ, PCM_JLCPCB:R_0402, F.Cu at (103.3, 78.5)
- added R93: 1MΩ, PCM_JLCPCB:R_0402, F.Cu at (103.3, 79.8)
- added R94: 10Ω, PCM_JLCPCB:R_0402, F.Cu at (101.0, 78.5)
- added RV9: 50kΩ, Maxime:RES-ADJ-SMD_G43BT, F.Cu at (97.9, 96.9)
- added U6: LM339, Maxime:TSSOP-14_L5.0-W4.4-P0.65-LS6.4-BL, F.Cu at (93.9, 89.0)
- C8: moved to F.Cu
- D2: value 1SMA4728A -> 19-237/R6GHBHC-A01/2T; footprint PCM_JLCPCB:D_DO-214AC(SMA) -> Maxime:LED-SMD_4P-L1.6-W1.6-19-237A-BHR6GHC-A01-2T
- R22, R23: value 100kΩ -> 22kΩ
- R24: value 2kΩ -> 100kΩ
- R25, R27: value 100kΩ -> 100Ω
- R26: value 1kΩ -> 100Ω
- R28: value 4.7kΩ -> 100kΩ
- R29, R30: value 1kΩ -> 100kΩ
- RV3: value 100kΩ -> 50kΩ
- U4: value MCP6004T-I/ST -> LM339
- U5: footprint Package_SO:TSSOP-14_4.4x5mm_P0.65mm -> Maxime:TSSOP-14_L5.0-W4.4-P0.65-LS6.4-BL
- moved J3 61.9 mm to (66.5, 88.6), turned to -70 degrees
- moved R28 50.5 mm to (77.9, 84.5)
- moved R29 50.2 mm to (77.9, 85.8)
- moved R30 49.0 mm to (80.2, 84.5)
- moved J4 48.0 mm to (69.1, 119.6), turned to -50 degrees
- moved R22 44.3 mm to (82.5, 85.8), turned to 180 degrees
- moved C17 44.0 mm to (82.5, 88.4)
- moved C16 43.5 mm to (82.5, 87.1)
- moved C10 43.2 mm to (116.3, 105.2), turned to -90 degrees
- moved U2 42.7 mm to (120.7, 104.7)
- moved R48 42.0 mm to (91.2, 135.9), turned to 90 degrees
- moved C11 41.4 mm to (92.9, 127.1), turned to -90 degrees
- moved U3 40.6 mm to (97.2, 126.6)
- moved R26 39.2 mm to (90.6, 106.7), turned to 180 degrees
- moved C15 37.3 mm to (89.5, 83.4), turned to -90 degrees
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Connections:
- net Net-(U1D-VINA+) renamed /V_ref
- C10 pad 1: +0.375V -> VDD
- C14 pad 1: Net-(U5B--) -> Net-(U4B--)
- C15 pad 1: Net-(C15-Pad1) -> VDD
- C16 pad 1: Net-(C15-Pad1) -> Net-(U1B-VINC-)
- C16 pad 2: GNDREF -> /Vkick
- C17 pad 1: Net-(C17-Pad1) -> GNDREF
- C17 pad 2: Net-(C17-Pad2) -> /Vw
- C18 pad 2: Net-(U3A-VOUTB) -> Net-(U2A-VOUTB)
- C19 pad 1: Net-(U3A-VINB+) -> Net-(U2A-VINB+)
- C9 pad 1: +2V -> VDD
- D2 pad 1: VDD -> Net-(D2-R-)
- D2 pad 2: Net-(D2-Pad2) -> Net-(D2-B-)
- Q1 pad 1: Net-(Q1-G) -> SP
- Q1 pad 2: AP -> GNDREF
- Q1 pad 3: Net-(Q1-D) -> AP
- R13 pad 1: Net-(Q4-G) -> VDD
- R13 pad 2: VDD -> Net-(Q4-G)
- R14 pad 1: Peak -> VDD
- R14 pad 2: VDD -> Peak
- R15 pad 2: Net-(U5B--) -> Net-(U4B--)
- R16 pad 1: Net-(U5B--) -> Net-(U4B--)
- R17 pad 2: Net-(U5B-+) -> Net-(U4B-+)
- R18 pad 1: Net-(U5B-+) -> Net-(U4B-+)
- R19 pad 1: Net-(U5B-+) -> Net-(U4B-+)
- R22 pad 1: VDD -> /Vkick
- R22 pad 2: Net-(C15-Pad1) -> GNDREF
- R23 pad 1: Net-(C15-Pad1) -> /Vw_buf
- R23 pad 2: GNDREF -> Net-(Q15-B)
- R24 pad 1: Net-(C15-Pad1) -> GNDREF
- R24 pad 2: Net-(U3D-VINA-) -> Net-(Q15-B)
- R25 pad 1: Net-(U3D-VINA+) -> Net-(Q15-C)
- R25 pad 2: Net-(C15-Pad1) -> Vm
- R26 pad 1: Net-(U3D-VINA-) -> Net-(R26-Pad1)
- R26 pad 2: Net-(R26-Pad2) -> GNDREF
- R27 pad 1: Net-(D2-Pad2) -> Vm
- R27 pad 2: Net-(U3D-VINA+) -> Stimulus_In
- R28 pad 2: Net-(D2-Pad2) -> T4
- R29 pad 1: Net-(U3D-VOUTA) -> T4
- R29 pad 2: Net-(C17-Pad1) -> T3
- R30 pad 1: Net-(C17-Pad2) -> T3
- R30 pad 2: Vm -> T2
- R31 pad 2: Net-(U3A-VINB+) -> Net-(U2A-VINB+)
- R32 pad 1: Net-(U3A-VINB+) -> Net-(U2A-VINB+)
- R33 pad 2: Net-(U3B-VINC+) -> Net-(U2B-VINC+)
- R34 pad 1: Net-(U3B-VINC+) -> Net-(U2B-VINC+)
- R34 pad 2: Net-(U3A-VOUTB) -> Net-(U2A-VOUTB)
- R35 pad 1: Net-(U3A-VOUTB) -> Net-(U2A-VOUTB)
- R35 pad 2: Net-(U3C-VIND-) -> Net-(U2C-VIND-)
- R36 pad 1: Net-(U3C-VIND-) -> Net-(U2C-VIND-)
- R41 pad 1: Net-(U4A-VINB-) -> Net-(U3A-VINB-)
- R45 pad 1: Net-(U4B-VINC-) -> Net-(U3B-VINC-)
- R49 pad 1: Net-(U4C-VIND-) -> Net-(U3C-VIND-)
- R53 pad 1: Net-(U4D-VINA-) -> Net-(U3D-VINA-)
- R7 pad 2: Net-(Q1-G) -> SP
- R8 pad 2: Net-(Q1-G) -> SP
- R9 pad 2: Net-(Q1-D) -> AP
- RV3 pad 1: Net-(R26-Pad2) -> /Vw
- RV3 pad 2: Net-(U3D-VOUTA) -> /Vw
- RV3 pad 3: Net-(U3D-VOUTA) -> Net-(R26-Pad1)
- RV4 pad 1: Net-(U3A-VOUTB) -> Net-(U2A-VOUTB)
- RV4 pad 2: Net-(U3A-VOUTB) -> Net-(U2A-VOUTB)
- RV5 pad 2: Net-(U4A-VINB+) -> Net-(U3A-VINB+)
- RV6 pad 2: Net-(U4B-VINC+) -> Net-(U3B-VINC+)
- RV7 pad 2: Net-(U4C-VIND+) -> Net-(U3C-VIND+)
- RV8 pad 2: Net-(U4D-VINA+) -> Net-(U3D-VINA+)
- U1 pad 10: unconnected-(U1B-VINC+-Pad10) -> SP
- U1 pad 12: unconnected-(U1C-VIND+-Pad12) -> /Vw
- U1 pad 13: unconnected-(U1C-VIND--Pad13) -> /Vw_buf
- U1 pad 14: unconnected-(U1C-VOUTD-Pad14) -> /Vw_buf
- U1 pad 4: +2V -> VDD
- U1 pad 5: unconnected-(U1A-VINB+-Pad5) -> +0.375V
- U1 pad 6: unconnected-(U1A-VINB--Pad6) -> /Reset_Current_Injection
- U1 pad 7: unconnected-(U1A-VOUTB-Pad7) -> /Reset_Current_Injection
- U1 pad 8: unconnected-(U1B-VOUTC-Pad8) -> Net-(U1B-VINC-)
- U1 pad 9: unconnected-(U1B-VINC--Pad9) -> Net-(U1B-VINC-)
- U2 pad 1: /Reset_Current_Injection -> Net-(U2D-VINA-)
- U2 pad 10: unconnected-(U2B-VINC+-Pad10) -> Net-(U2B-VINC+)
- U2 pad 12: unconnected-(U2C-VIND+-Pad12) -> Net-(Q8-NS)
- U2 pad 13: unconnected-(U2C-VIND--Pad13) -> Net-(U2C-VIND-)
- U2 pad 14: unconnected-(U2C-VOUTD-Pad14) -> Net-(Q8-NG)
- U2 pad 2: +0.375 -> Net-(U2D-VINA-)
- U2 pad 3: /Reset_Current_Injection -> Vm
- U2 pad 4: +0.375 -> VDD
- U2 pad 5: unconnected-(U2A-VINB+-Pad5) -> Net-(U2A-VINB+)
- U2 pad 6: unconnected-(U2A-VINB--Pad6) -> V_Synapses
- U2 pad 7: unconnected-(U2A-VOUTB-Pad7) -> Net-(U2A-VOUTB)
- U2 pad 8: unconnected-(U2B-VOUTC-Pad8) -> Net-(Q8-PG)
- U2 pad 9: unconnected-(U2B-VINC--Pad9) -> Net-(Q8-PS)
- U3 pad 1: Net-(U3D-VOUTA) -> Net-(U3D-VINA-)
- U3 pad 12: Net-(Q8-NS) -> Net-(U3C-VIND+)
- U3 pad 14: Net-(Q8-NG) -> Net-(U3C-VIND-)
- U3 pad 6: V_Synapses -> Net-(U3A-VINB-)
- U3 pad 7: Net-(U3A-VOUTB) -> Net-(U3A-VINB-)
- U3 pad 8: Net-(Q8-PG) -> Net-(U3B-VINC-)
- U3 pad 9: Net-(Q8-PS) -> Net-(U3B-VINC-)
- U4 pad 1: Net-(U4D-VINA-) -> Reset
- U4 pad 10: Net-(U4B-VINC+) -> /V_Spike_Threshold
- U4 pad 11: GNDREF -> Net-(U4C-+)
- U4 pad 12: Net-(U4C-VIND+) -> GNDREF
- U4 pad 13: Net-(U4C-VIND-) -> Net-(R58-Pad2)
- U4 pad 14: Net-(U4C-VIND-) -> unconnected-(U4-Pad14)
- U4 pad 2: Net-(U4D-VINA-) -> SP
- U4 pad 3: Net-(U4D-VINA+) -> VDD
- U4 pad 4: VDD -> Vm
- U4 pad 5: Net-(U4A-VINB+) -> /V_Threshold
- U4 pad 6: Net-(U4A-VINB-) -> Net-(U4B--)
- U4 pad 7: Net-(U4A-VINB-) -> Net-(U4B-+)
- U4 pad 8: Net-(U4B-VINC-) -> unconnected-(U4D---Pad8)
- U4 pad 9: Net-(U4B-VINC-) -> unconnected-(U4D-+-Pad9)
- U5 pad 1: Reset -> S4
- U5 pad 10: unconnected-(U5C---Pad10) -> Vsel
- U5 pad 11: unconnected-(U5C-+-Pad11) -> T3
- U5 pad 13: unconnected-(U5-Pad13) -> S1
- U5 pad 14: unconnected-(U5-Pad14) -> S1
- U5 pad 2: Net-(Q1-G) -> S0
- U5 pad 4: Vm -> Vsel
- U5 pad 5: /V_Threshold -> T4
- U5 pad 6: Net-(U5B--) -> Vsel
- U5 pad 7: Net-(U5B-+) -> T1
- U5 pad 8: unconnected-(U5D---Pad8) -> T4
- U5 pad 9: unconnected-(U5D-+-Pad9) -> Vsel
Routing:
- net VDD: track 0.00 -> 365.9 mm, vias 0 -> 32
- net Vm: track 0.00 -> 274.4 mm, vias 0 -> 17
- net Net-(Q10-S2): track 0.00 -> 162.5 mm, vias 0 -> 10
- net Vsel: track 0.00 -> 149.8 mm, vias 0 -> 9
- net Reset: track 0.00 -> 93.7 mm, vias 0 -> 2
- net Net-(U3B-VINC-): track 0.00 -> 81.9 mm, vias 0 -> 4
- net T1: track 0.00 -> 81.9 mm, vias 0 -> 5
- net Net-(U3A-VINB+): track 0.00 -> 79.0 mm, vias 0 -> 2
- net Net-(U3A-VINB-): track 0.00 -> 75.9 mm
- net /Reset_Current_Injection: track 0.00 -> 75.8 mm, vias 0 -> 2
- net T2: track 0.00 -> 75.6 mm, vias 0 -> 5
- net +0.375V: track 0.00 -> 71.4 mm, vias 0 -> 4
- net Net-(U3B-VINC+): track 0.00 -> 68.1 mm, vias 0 -> 4
- net /Vw: track 0.00 -> 62.6 mm, vias 0 -> 7
- net T3: track 0.00 -> 61.1 mm, vias 0 -> 4
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- added copper zone on B.Cu, net GNDREF
- added copper zone on F.Cu, net GNDREF
Other:
- board size 6.2 x 4.7 mm -> 119.7 x 79.7 mm
- board text added: "C"
- board text added: "G"
- board text added: "V"
- board text added: "adapt"
- board text added: "leak"
- board text added: "m"
- board text added: "syn"
- board text added: "τ"
