File: PCBs/LIFeling/LIFeling.kicad_sch (KiCad schematic)
At the start: 203 parts, among them J1 Oscilloscope Jack, J2 Axon Output, J3 Syn1 Input, J4 Syn2 Input, J5 Syn3 Input, J6 Syn4 Input, Q1 BSS138, Q2 MMBT3904, Q3 BSS138, Q4 BSS138, Q5 BSS138, Q6 BSS138, Q7 BSS138, Q8 MMBT3904, SW1 SW_SPDT, U1 MCP6004T-I/ST, U10 TS5A3166DCKR, U11 TS5A3166DCKR, U12 TS5A3166DCKR, U13 TS5A3166DCKR, U14 TS5A3166DCKR, U15 TS5A3166DCKR, U16 TS5A3166DCKR, U17 TS5A3166DCKR, U18 TS5A3166DCKR, U19 MCP6004T-I/ST, U2 MCP6004T-I/ST, U20 TS5A3166DCKR, U3 MCP6004T-I/ST, U4 TLV7044PWR, U5 TLV7044PWR, U6 TLV7044PWR, U7 TPS610995DRVR, U8 TLV9001IDBVR, U9 TS5A3166DCKR

Commit message: update LIFelingPCB
Parts:
- added C40, C41, C9: 100nF, C0402, symbol CL05B104KO5NNNC1_CL05B104KO5NNNC (1)-altium-import:root_0_CL05B104KO5NNNC_
- added C42, C43: 1uF, C0402, symbol CL05A105KA5NQNC1_CL05A105KA5NQNC-altium-import:root_0_CL05A105KA5NQNC_
- added R92: 100Ω, R0402, symbol RC0402FR-07100RL1_RC0402FR-07100RL-altium-import:root_0_RC0402FR-07100RL_
- added R93: 1MΩ, R0402, symbol RC0402FR-071ML1_RC0402FR-071ML-altium-import:root_0_RC0402FR-071ML_
- added U21: REF35102QDBVR, SOT-23-6_L2.9-W1.6-P0.95-LS2.8-BR, symbol 1_P1-altium-import:root_0_REF35102QDBVR_
- R88: value 47kΩ -> 100kΩ
Connections:
- net GNDREF: now also C40.1, C41.1, C42.2, C43.1, C9.1, U21.1 (GND), U21.2 (GND)
- net VDD: now also R92.2
- net V_Leak: no longer R86.1
- net V_Stim_Cmd: now also R93.2
- new net: C40.2, U21.5 (NR)
- new net: C43.2, C9.2, R92.1, U21.3 (EN), U21.4 (VIN)
- new net V_Stim_Zero_1V024: C41.2, C42.1, R86.1, R93.1, U21.6 (VREF)
Other:
- note added: "Servoed Stimulus Driver V_Stim_Drive = Vm_Int + 0.5 × (V_Stim_Cmd - V_Stim_Zero_1V024)"
- note added: "Stimulus injection strength I_inj = (V_Stim_Drive - Vm_Int) / R88 I_inj = (V_Stim_Cmd - 1.024 V) / (2 × R88)"
- note added: "Stimulus_Ext is converted into a local current command: The external analog stimulus is ESD-protected and lightly filtered intoV_Stim_Cmd V_Stim_Zero_1V024 is used as the zero-current reference. Stimulus_Ext is a command voltage: → 1.024 V = zero injected current → above 1.024 V = depolarising → below 1.024 V = hyperpolarising Produces an approximate current-clamp style stimulus current into the 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"
- note removed: "Servoed Stimulus Driver"
- note removed: "Stimulus injection strength"
- note removed: "Stimulus_Ext is converted into a local current command: The external analog stimulus is ESD-protected and lightly filtered intoV_Stim_Cmd V_Leak is used as the zero-current reference, → Commands above V_Leak are depolarising → Commands below V_Leak are hyperpolarising Produces an approximate current-clamp style stimulus current into the membrane"
