File: PCBs/LIFeling/LIFeling.kicad_sch (KiCad schematic)
At the start: 211 parts, among them J1 Oscilloscope Jack, J2 Axon Output, J3 Syn1 Input, J4 Syn2 Input, J5 Syn3 Input, J6 Syn4 Input, Q1 BSS138, Q2 MMBT3904, Q3 BSS138, Q4 BSS138, Q5 BSS138, Q6 BSS138, Q7 BSS138, Q8 MMBT3904, SW1 SW_SPDT, U1 MCP6004T-I/ST, U10 TS5A3166DCKR, U11 TS5A3166DCKR, U12 TS5A3166DCKR, U13 TS5A3166DCKR, U14 TS5A3166DCKR, U15 TS5A3166DCKR, U16 TS5A3166DCKR, U17 TS5A3166DCKR, U18 TS5A3166DCKR, U19 MCP6004T-I/ST, U2 MCP6004T-I/ST, U20 TS5A3166DCKR, U21 REF35102QDBVR, U3 MCP6004T-I/ST, U4 TLV7044PWR, U5 TLV7044PWR, U6 TLV7044PWR, U7 TPS610995DRVR, U8 TLV9001IDBVR, U9 TS5A3166DCKR

Commit message: update pcb
Parts:
- removed C42, C43: 1uF, C0402, symbol CL05A105KA5NQNC1_CL05A105KA5NQNC-altium-import:root_0_CL05A105KA5NQNC_
- removed J1: Oscilloscope Jack, Maxime:AUDIO-SMD_PJ-320B, symbol PJ-320B1_PJ-320B-altium-import:root_0_PJ-320B贴片_
- removed J2: Axon Output, Maxime:AUDIO-SMD_PJ-320B, symbol PJ-320B1_PJ-320B-altium-import:root_0_PJ-320B贴片_
- removed J3: Syn1 Input, Maxime:AUDIO-SMD_PJ-320B, symbol PJ-320B1_PJ-320B-altium-import:root_0_PJ-320B贴片_
- removed J4: Syn2 Input, Maxime:AUDIO-SMD_PJ-320B, symbol PJ-320B1_PJ-320B-altium-import:root_0_PJ-320B贴片_
- removed J5: Syn3 Input, Maxime:AUDIO-SMD_PJ-320B, symbol PJ-320B1_PJ-320B-altium-import:root_0_PJ-320B贴片_
- removed J6: Syn4 Input, Maxime:AUDIO-SMD_PJ-320B, symbol PJ-320B1_PJ-320B-altium-import:root_0_PJ-320B贴片_
- removed R10: 69.8kΩ, R0402, symbol Spiky_Lui-altium-import:root_0_0402WGF6982TCE_
- removed R12, R13, R5, R54: 100kΩ, R0402, symbol Spiky_Lui-altium-import:root_0_RC0402FR-07100KL_
- removed R33: 220kΩ, R0402, symbol RC0402FR-07220KL1_RC0402FR-07220KL-altium-import:root_0_RC0402FR-07220KL_
- removed R35, R55: 22kΩ, R0402, symbol RC0402FR-0722KL1_RC0402FR-0722KL-altium-import:root_0_RC0402FR-0722KL_
- removed R4: 49.9kΩ, R0402, symbol Spiky_Lui-altium-import:root_0_RC0402FR-0749K9L_
- removed R53: 27kΩ, R0402, symbol RC0402FR-0727KL1_RC0402FR-0727KL-altium-import:root_0_RC0402FR-0727KL_
- removed R7, R8: 10kΩ, R0402, symbol Spiky_Lui-altium-import:root_0_RC0402FR-0710KL_
- removed R92: 100Ω, R0402, symbol RC0402FR-07100RL1_RC0402FR-07100RL-altium-import:root_0_RC0402FR-07100RL_
- removed RV1, RV4: 50kΩ, Maxime:RES-ADJ-SMD_G43BT, symbol G43BT-B5031_G43BT-B503-altium-import:root_0_G43BT-B503_
- removed RV6, RV7, RV8, RV9: 100kΩ, Maxime:RES-ADJ-SMD_G43BT, symbol G43BT-B1041_G43BT-B104-altium-import:root_0_G43BT-B104_
- removed SW1: SW_SPDT, Maxime:SW-SMD_SSAJ120100, symbol Switch:SW_SPDT
- removed U19: MCP6004T-I/ST, Maxime:TSSOP-14_L5.0-W4.4-P0.65-LS6.4-BL, symbol MCP6004T-I_ST1_MCP6004T-I_ST-altium-import:root_0_MCP6004T-I/ST_
- removed U21: REF35102QDBVR, SOT-23-6_L2.9-W1.6-P0.95-LS2.8-BR, symbol 1_P1-altium-import:root_0_REF35102QDBVR_
- added C42: 100nF, JLCPCB:C_0402, symbol CL05B104KO5NNNC1_CL05B104KO5NNNC (1)-altium-import:root_0_CL05B104KO5NNNC_
- added J1: Stim_Ext, AUDIO-SMD_HX-PJ-320A-3P-DIP, symbol 1_P1-altium-import:root_0_HX PJ-320A-3P DIP_
- added J2: Axon_Output, AUDIO-SMD_HX-PJ-320A-3P-DIP, symbol 1_P1-altium-import:root_0_HX PJ-320A-3P DIP_
- added J3: Syn1_Input, AUDIO-SMD_HX-PJ-320A-3P-DIP, symbol 1_P1-altium-import:root_0_HX PJ-320A-3P DIP_
- added J4: Syn2_Input, AUDIO-SMD_HX-PJ-320A-3P-DIP, symbol 1_P1-altium-import:root_0_HX PJ-320A-3P DIP_
- added J5: Syn3_Input, AUDIO-SMD_HX-PJ-320A-3P-DIP, symbol 1_P1-altium-import:root_0_HX PJ-320A-3P DIP_
- added J6: Syn4_Input, AUDIO-SMD_HX-PJ-320A-3P-DIP, symbol 1_P1-altium-import:root_0_HX PJ-320A-3P DIP_
- added R11, R38, R8, R96: 100kΩ, JLCPCB:R_0402, symbol Spiky_Lui-altium-import:root_0_RC0402FR-07100KL_
- added R12, R57, R83, R84, R85, R86: 1MΩ, JLCPCB:R_0402, symbol RC0402FR-071ML1_RC0402FR-071ML-altium-import:root_0_RC0402FR-071ML_
- added R13, R14, R5, R6: 220kΩ, JLCPCB:R_0402, symbol RC0402FR-07220KL1_RC0402FR-07220KL-altium-import:root_0_RC0402FR-07220KL_
- added R36: 2.2MΩ, JLCPCB:R_0402, symbol 1_P1-altium-import:root_0_RC0402FR-072M2L_
- added R56: 270kΩ, JLCPCB:R_0402, symbol 1_P1-altium-import:root_0_CR0402F270KQ10Z_
- added R58: 220kΩ, JLCPCB:R_0402, symbol 1_P1-altium-import:root_0_1RC0402F2203_
- added RV1, RV4: 100kΩ, Maxime:RES-ADJ-SMD_G43BT, symbol G43BT-B1041_G43BT-B104-altium-import:root_0_G43BT-B104_
- added RV6, RV7, RV8, RV9: 1MΩ, RES-ADJ-SMD_G43BT, symbol 1_P1-altium-import:root_0_G43BT-B105_
- added SW1: K3-1260D-L1, Maxime:SW-TH_K3-1260D-L1, symbol K3-1260D-L11_K3-1260D-L1-altium-import:root_0_K3-1260D-L1_
- added U19: TLV7031DCKR, Maxime:SC-70-5_L2.1-W1.3-P0.65-LS2.2-BR, symbol 1_P1-altium-import:root_0_TLV7031DCKR_
- added U21: REF3020AIDBZR, SOT-23-3_L3.0-W1.7-P0.95-LS2.9-BR, symbol 1_P1-altium-import:root_0_REF3020AIDBZR_
- added U22: TLV9001IDBVR, SOT-23-5_L3.0-W1.7-P0.95-LS2.8-BR, symbol 1_P1-altium-import:root_0_TLV9001IDBVR_
- C1, C2: footprint C0402 -> JLCPCB:C_0805; LCSC Part # (none) -> C15850; SUPPLIER PART C315248 -> (none)
- C10: renamed from C11; footprint C0402 -> JLCPCB:C_0805; LCSC Part # (none) -> C602037; SUPPLIER PART C385994 -> (none)
- C11: renamed from C12; footprint C0402 -> JLCPCB:C_0402; LCSC Part # (none) -> C52923; SUPPLIER PART C52923 -> (none)
- C12: renamed from C13; footprint C0402 -> JLCPCB:C_0402; LCSC Part # (none) -> C1525; SUPPLIER PART C1525 -> (none)
- C13: renamed from C14; footprint C0402 -> JLCPCB:C_0402; LCSC Part # (none) -> C2167113; SUPPLIER PART C1546 -> (none)
- C14: renamed from C15; footprint C0402 -> JLCPCB:C_0402; LCSC Part # (none) -> C1525; SUPPLIER PART C1525 -> (none)
- C15: renamed from C9; footprint C0402 -> JLCPCB:C_0402
- C16: renamed from C38; footprint C0402 -> JLCPCB:C_0402; LCSC Part # (none) -> C1532; SUPPLIER PART C1525 -> (none)
- C17: renamed from C39; footprint C0402 -> JLCPCB:C_0402; LCSC Part # (none) -> C1525; SUPPLIER PART C1525 -> (none)
- C18: renamed from C16; footprint C0603 -> JLCPCB:C_0603; LCSC Part # (none) -> C376839; SUPPLIER PART C376839 -> (none)
- C19: renamed from C17; footprint C0402 -> JLCPCB:C_0402; LCSC Part # (none) -> C1525; SUPPLIER PART C1525 -> (none)
- C20: renamed from C18; footprint C0603 -> JLCPCB:C_0603; LCSC Part # (none) -> C29936; SUPPLIER PART C86020 -> (none)
- C21: renamed from C19; footprint C0402 -> JLCPCB:C_0402; LCSC Part # (none) -> C1525; SUPPLIER PART C1525 -> (none)
- C22: renamed from C20; footprint C0603 -> JLCPCB:C_0603; LCSC Part # (none) -> C57895; SUPPLIER PART C57895 -> (none)
- C23: renamed from C21; footprint C0402 -> JLCPCB:C_0402; LCSC Part # (none) -> C1525; SUPPLIER PART C1525 -> (none)
- C24: renamed from C22; footprint C0805 -> JLCPCB:C_0805; LCSC Part # (none) -> C1779; SUPPLIER PART C1779 -> (none)
- C25: renamed from C23; footprint C0402 -> JLCPCB:C_0402; LCSC Part # (none) -> C1525; SUPPLIER PART C1525 -> (none)
- C26: renamed from C24; footprint C0805 -> JLCPCB:C_0805; LCSC Part # (none) -> C40894; SUPPLIER PART C6119932 -> (none)
- C27: renamed from C25; footprint C0402 -> JLCPCB:C_0402; LCSC Part # (none) -> C1525; SUPPLIER PART C1525 -> (none)
- C28: renamed from C26; footprint C0402 -> JLCPCB:C_0402; LCSC Part # (none) -> C2167113; SUPPLIER PART C1546 -> (none)
- C29: renamed from C27; footprint C0603 -> JLCPCB:C_0603; LCSC Part # (none) -> C29936; SUPPLIER PART C86020 -> (none)
- C3, C4, C5, C6, C7, C8: footprint C0402 -> JLCPCB:C_0402; LCSC Part # (none) -> C1525; SUPPLIER PART C1525 -> (none)
- C30: renamed from C28; footprint C0402 -> JLCPCB:C_0805; LCSC Part # (none) -> C15850; SUPPLIER PART C315248 -> (none)
- C31: renamed from C29; footprint PCM_JLCPCB:C_0402 -> JLCPCB:C_0402; LCSC C15195 -> (none); LCSC Part # (none) -> C15195
- C32: renamed from C30; footprint C0402 -> JLCPCB:C_0402; LCSC Part # (none) -> C1525; SUPPLIER PART C1525 -> (none)
- C33: renamed from C31; footprint C0402 -> JLCPCB:C_0402; LCSC Part # (none) -> C52923; SUPPLIER PART C52923 -> (none)
- C34: renamed from C32; footprint C0402 -> JLCPCB:C_0402; LCSC Part # (none) -> C1525; SUPPLIER PART C1525 -> (none)
- C35: renamed from C33; footprint C0402 -> JLCPCB:C_0402; LCSC Part # (none) -> C1525; SUPPLIER PART C1525 -> (none)
- C36: renamed from C34; footprint C0402 -> JLCPCB:C_0402; LCSC Part # (none) -> C1525; SUPPLIER PART C1525 -> (none)
- C37: renamed from C35; footprint C0402 -> JLCPCB:C_0402; LCSC Part # (none) -> C1525; SUPPLIER PART C1525 -> (none)
- C38: renamed from C36; footprint C0603 -> JLCPCB:C_0603; LCSC Part # (none) -> C106249; SUPPLIER PART C106249 -> (none)
- C39: renamed from C37; footprint C0402 -> JLCPCB:C_0402; LCSC Part # (none) -> C2167113; SUPPLIER PART C1546 -> (none)
- C40, C41: footprint C0402 -> JLCPCB:C_0402
- C9: renamed from C10; footprint C0402 -> JLCPCB:C_0805; LCSC Part # (none) -> C15850; SUPPLIER PART C315248 -> (none)
- D1, D19: footprint X1SON-2_L1.0-W0.6-P0.65-RD -> Maxime:X1SON-2_L1.0-W0.6-P0.65-RD-1; LCSC Part # (none) -> C1847651; SUPPLIER PART C1847651 -> (none)
- D10, D11, D12, D13, D14, D15, D16, D17, D2, D21, D22, D3: LCSC Part # (none) -> C22629; SUPPLIER PART C22629 -> (none)
- D18: LCSC Part # (none) -> C1847651; SUPPLIER PART C1847651 -> (none)
- D20, D6, D8: footprint SOD-523_L1.2-W0.8-LS1.6-RD -> Maxime:SOD-523_L1.2-W0.8-LS1.6-RD; LCSC Part # (none) -> C145179; SUPPLIER PART C145179 -> (none)
- D4, D5, D7: footprint SOD-323_L1.8-W1.3-LS2.5-RD-1 -> Maxime:SOD-323_L1.8-W1.3-LS2.5-RD-1; LCSC Part # (none) -> C57759; SUPPLIER PART C57759 -> (none)
- D9: LCSC Part # (none) -> C60105; SUPPLIER PART C60105 -> (none)
- L1: footprint IND-SMD_L3.0-W3.0_SMNR3015 -> Maxime:IND-SMD_L3.0-W3.0_SMNR3015; LCSC Part # (none) -> C6364793; SUPPLIER PART C6364793 -> (none)
- Q1, Q3, Q4, Q5, Q6, Q7: LCSC Part # (none) -> C52895; SUPPLIER PART C52895 -> (none)
- Q2, Q8: LCSC Part # (none) -> C181119; SUPPLIER PART C181119 -> (none)
- R1: renamed from R89; footprint R0402 -> JLCPCB:R_0402; LCSC Part # (none) -> C2906862; SUPPLIER PART C2906862 -> (none)
- R10: renamed from R11; value 10kΩ -> 56kΩ; footprint R0402 -> JLCPCB:R_0402; LCSC PART NAME 厚膜电阻 10kΩ ±1% 62.5mW -> 56kΩ ±1% 62.5mW 0402; LCSC Part # (none) -> C2906875; MANUFACTURER YAGEO(国巨) -> FOJAN; MANUFACTURER PART RC0402FR-0710KL -> FRC0402F5602TS; SUPPLIER PART C60490 -> (none)
- R15: renamed from R90; footprint R0402 -> JLCPCB:R_0402; LCSC Part # (none) -> C60491; SUPPLIER PART C60491 -> (none)
- R16: renamed from R91; footprint R0402 -> JLCPCB:R_0402; LCSC Part # (none) -> C60490; SUPPLIER PART C60490 -> (none)
- R17: renamed from R14; footprint R0402 -> JLCPCB:R_0402; LCSC Part # (none) -> C60491; SUPPLIER PART C60491 -> (none)
- R18: renamed from R15; footprint R0402 -> JLCPCB:R_0402; LCSC Part # (none) -> C60491; SUPPLIER PART C60491 -> (none)
- R19: renamed from R16; footprint R0402 -> JLCPCB:R_0402; LCSC Part # (none) -> C60491; SUPPLIER PART C60491 -> (none)
- R2: renamed from R1; footprint R0402 -> JLCPCB:R_0402; LCSC Part # (none) -> C112291; SUPPLIER PART C112291 -> (none)
- R20: renamed from R17; footprint R0402 -> JLCPCB:R_0402; LCSC Part # (none) -> C60491; SUPPLIER PART C60491 -> (none)
- R21: renamed from R18; footprint R0402 -> JLCPCB:R_0402; LCSC Part # (none) -> C60491; SUPPLIER PART C60491 -> (none)
- R22: renamed from R19; footprint R0402 -> JLCPCB:R_0402; LCSC Part # (none) -> C60491; SUPPLIER PART C60491 -> (none)
- R23: renamed from R20; footprint R0402 -> JLCPCB:R_0402; LCSC Part # (none) -> C138033; SUPPLIER PART C138033 -> (none)
- R24: renamed from R21; footprint R0402 -> JLCPCB:R_0402; LCSC Part # (none) -> C60491; SUPPLIER PART C60491 -> (none)
- R25: renamed from R22; footprint R0402 -> JLCPCB:R_0402; LCSC Part # (none) -> C138033; SUPPLIER PART C138033 -> (none)
- R26: renamed from R23; footprint R0402 -> JLCPCB:R_0402; LCSC Part # (none) -> C138033; SUPPLIER PART C138033 -> (none)
- R27: renamed from R24; footprint R0402 -> JLCPCB:R_0402; LCSC Part # (none) -> C60491; SUPPLIER PART C60491 -> (none)
- R28: renamed from R25; footprint R0402 -> JLCPCB:R_0402; LCSC Part # (none) -> C138033; SUPPLIER PART C138033 -> (none)
- R29: renamed from R26; footprint R0402 -> JLCPCB:R_0402; LCSC Part # (none) -> C138033; SUPPLIER PART C138033 -> (none)
- R3: renamed from R2; footprint R0402 -> JLCPCB:R_0402; LCSC Part # (none) -> C60490; SUPPLIER PART C60490 -> (none)
- R30: renamed from R27; footprint R0402 -> JLCPCB:R_0402; LCSC Part # (none) -> C60491; SUPPLIER PART C60491 -> (none)
- R31: renamed from R28; footprint R0402 -> JLCPCB:R_0402; LCSC Part # (none) -> C138033; SUPPLIER PART C138033 -> (none)
- R32: renamed from R29; footprint R0402 -> JLCPCB:R_0402; LCSC Part # (none) -> C138033; SUPPLIER PART C138033 -> (none)
- R33: renamed from R30; footprint R0402 -> JLCPCB:R_0402; LCSC Part # (none) -> C60491; SUPPLIER PART C60491 -> (none)
- R34: renamed from R31; footprint R0402 -> JLCPCB:R_0402; LCSC Part # (none) -> C138033; SUPPLIER PART C138033 -> (none)
- R35: renamed from R32; footprint R0402 -> JLCPCB:R_0402; LCSC Part # (none) -> C106235; SUPPLIER PART C106235 -> (none)
- R37: renamed from R34; footprint R0402 -> JLCPCB:R_0402; LCSC Part # (none) -> C60490; SUPPLIER PART C60490 -> (none)
- R39: renamed from R36; footprint R0402 -> JLCPCB:R_0402; LCSC Part # (none) -> C82868; SUPPLIER PART C82868 -> (none)
- R4: renamed from R3; footprint R0402 -> JLCPCB:R_0402; LCSC Part # (none) -> C60491; SUPPLIER PART C60491 -> (none)
- R40: renamed from R42; footprint R0402 -> JLCPCB:R_0402; LCSC Part # (none) -> C106232; SUPPLIER PART C106232 -> (none)
- R41: renamed from R37; footprint R0402 -> JLCPCB:R_0402; LCSC Part # (none) -> C114763; SUPPLIER PART C114763 -> (none)
- R42: renamed from R38; footprint R0402 -> JLCPCB:R_0402; LCSC Part # (none) -> C60491; SUPPLIER PART C60491 -> (none)
- R43: renamed from R39; footprint R0402 -> JLCPCB:R_0402; LCSC Part # (none) -> C60491; SUPPLIER PART C60491 -> (none)
- R44: renamed from R40; footprint R0402 -> JLCPCB:R_0402; LCSC Part # (none) -> C114763; SUPPLIER PART C114763 -> (none)
- R45: renamed from R41; footprint R0402 -> JLCPCB:R_0402; LCSC Part # (none) -> C138006; SUPPLIER PART C138006 -> (none)
- R46: renamed from R43; footprint R0402 -> JLCPCB:R_0402; LCSC Part # (none) -> C60490; SUPPLIER PART C60490 -> (none)
- R47: renamed from R44; footprint R0402 -> JLCPCB:R_0402; LCSC Part # (none) -> C82868; SUPPLIER PART C82868 -> (none)
- R48: renamed from R45; footprint R0402 -> JLCPCB:R_0402; LCSC Part # (none) -> C60491; SUPPLIER PART C60491 -> (none)
- R49: renamed from R46; footprint R0402 -> JLCPCB:R_0402; LCSC Part # (none) -> C60491; SUPPLIER PART C60491 -> (none)
- R50: renamed from R47; footprint R0402 -> JLCPCB:R_0402; LCSC Part # (none) -> C138033; SUPPLIER PART C138033 -> (none)
- R51: renamed from R48; footprint R0402 -> JLCPCB:R_0402; LCSC Part # (none) -> C60491; SUPPLIER PART C60491 -> (none)
- R52: renamed from R49; footprint R0402 -> JLCPCB:R_0402; LCSC Part # (none) -> C60490; SUPPLIER PART C60490 -> (none)
- R53: renamed from R50; footprint R0402 -> JLCPCB:R_0402; LCSC Part # (none) -> C82868; SUPPLIER PART C82868 -> (none)
- R54: renamed from R51; footprint R0402 -> JLCPCB:R_0402; LCSC Part # (none) -> C106232; SUPPLIER PART C106232 -> (none)
- R55: renamed from R52; footprint R0402 -> JLCPCB:R_0402; LCSC Part # (none) -> C60491; SUPPLIER PART C60491 -> (none)
- R59: renamed from R56; footprint R0402 -> JLCPCB:R_0402
- R60: renamed from R57; footprint R0402 -> JLCPCB:R_0402; LCSC Part # (none) -> C60490; SUPPLIER PART C60490 -> (none)
- R61: renamed from R58; value 1kΩ -> 2kΩ; footprint R0402 -> JLCPCB:R_0402; LCSC Part # (none) -> C4109; SUPPLIER PART C106235 -> (none)
- R62: renamed from R59; value 1kΩ -> 2kΩ; footprint R0402 -> JLCPCB:R_0402; LCSC Part # (none) -> C4109; SUPPLIER PART C106235 -> (none)
- R63: renamed from R60; value 1kΩ -> 2kΩ; footprint R0402 -> JLCPCB:R_0402; LCSC Part # (none) -> C4109; SUPPLIER PART C106235 -> (none)
- R64: renamed from R61; footprint R0402 -> JLCPCB:R_0402; LCSC Part # (none) -> C60490; SUPPLIER PART C60490 -> (none)
- R65: renamed from R62; footprint R0402 -> JLCPCB:R_0402; LCSC Part # (none) -> C60491; SUPPLIER PART C60491 -> (none)
- R66: renamed from R63; footprint R0402 -> JLCPCB:R_0402; LCSC Part # (none) -> C82868; SUPPLIER PART C82868 -> (none)
- R67: renamed from R64; footprint R0402 -> JLCPCB:R_0402; LCSC Part # (none) -> C106235; SUPPLIER PART C106235 -> (none)
- R68: renamed from R65; footprint R0402 -> JLCPCB:R_0402; LCSC Part # (none) -> C60491; SUPPLIER PART C60491 -> (none)
- R69: renamed from R66; footprint R0402 -> JLCPCB:R_0402; LCSC Part # (none) -> C82868; SUPPLIER PART C82868 -> (none)
- R7: renamed from R6; value 24.3kΩ -> 20kΩ; footprint R0402 -> JLCPCB:R_0402; LCSC PART NAME 24.3kΩ ±1% 62.5mW 厚膜电阻 -> 20kΩ ±1% 62.5mW 厚膜电阻; LCSC Part # (none) -> C25765; SUPPLIER PART C26969 -> (none)
- R70: renamed from R67; footprint R0402 -> JLCPCB:R_0402; LCSC Part # (none) -> C82868; SUPPLIER PART C82868 -> (none)
- R71: renamed from R68; footprint R0402 -> JLCPCB:R_0402; LCSC Part # (none) -> C106235; SUPPLIER PART C106235 -> (none)
- R72: renamed from R69; footprint R0402 -> JLCPCB:R_0402; LCSC Part # (none) -> C60491; SUPPLIER PART C60491 -> (none)
- R73: renamed from R70; footprint R0402 -> JLCPCB:R_0402; LCSC Part # (none) -> C82868; SUPPLIER PART C82868 -> (none)
- R74: renamed from R71; footprint R0402 -> JLCPCB:R_0402; LCSC Part # (none) -> C82868; SUPPLIER PART C82868 -> (none)
- R75: renamed from R72; footprint R0402 -> JLCPCB:R_0402; LCSC Part # (none) -> C106235; SUPPLIER PART C106235 -> (none)
- R76: renamed from R73; footprint R0402 -> JLCPCB:R_0402; LCSC Part # (none) -> C60491; SUPPLIER PART C60491 -> (none)
- R77: renamed from R74; footprint R0402 -> JLCPCB:R_0402; LCSC Part # (none) -> C82868; SUPPLIER PART C82868 -> (none)
- R78: renamed from R75; footprint R0402 -> JLCPCB:R_0402; LCSC Part # (none) -> C82868; SUPPLIER PART C82868 -> (none)
- R79: renamed from R76; footprint R0402 -> JLCPCB:R_0402; LCSC Part # (none) -> C106235; SUPPLIER PART C106235 -> (none)
- R80: renamed from R77; footprint R0402 -> JLCPCB:R_0402; LCSC Part # (none) -> C60491; SUPPLIER PART C60491 -> (none)
- R81: renamed from R78; footprint R0402 -> JLCPCB:R_0402; LCSC Part # (none) -> C82868; SUPPLIER PART C82868 -> (none)
- R82: renamed from R79; footprint R0402 -> JLCPCB:R_0402; LCSC Part # (none) -> C60490; SUPPLIER PART C60490 -> (none)
- R87: renamed from R80; footprint R0402 -> JLCPCB:R_0402; LCSC Part # (none) -> C93943; SUPPLIER PART C93943 -> (none)
- R88: renamed from R81; footprint R0402 -> JLCPCB:R_0402; LCSC Part # (none) -> C60491; SUPPLIER PART C60491 -> (none)
- R89: renamed from R82; footprint R0402 -> JLCPCB:R_0402; LCSC Part # (none) -> C106232; SUPPLIER PART C106232 -> (none)
- R9: footprint R0402 -> JLCPCB:R_0402; LCSC Part # (none) -> C60491; SUPPLIER PART C60491 -> (none)
- R90: renamed from R93; footprint R0402 -> JLCPCB:R_0402
- R91: renamed from R83; footprint R0402 -> JLCPCB:R_0402; LCSC Part # (none) -> C106235; SUPPLIER PART C106235 -> (none)
- R92: renamed from R84; footprint R0402 -> JLCPCB:R_0402; LCSC Part # (none) -> C60491; SUPPLIER PART C60491 -> (none)
- R93: renamed from R85; footprint R0402 -> JLCPCB:R_0402; LCSC Part # (none) -> C114763; SUPPLIER PART C114763 -> (none)
- R94: renamed from R86; footprint R0402 -> JLCPCB:R_0402; LCSC Part # (none) -> C114763; SUPPLIER PART C114763 -> (none)
- R95: renamed from R87; footprint R0402 -> JLCPCB:R_0402; LCSC Part # (none) -> C60491; SUPPLIER PART C60491 -> (none)
- R97: renamed from R88; footprint R0402 -> JLCPCB:R_0402; LCSC Part # (none) -> C93943; SUPPLIER PART C93943 -> (none)
- U1, U2, U3: LCSC Part # (none) -> C50282; SUPPLIER PART C50282 -> (none)
- U10, U11, U12, U13, U14, U20, U9: LCSC Part # (none) -> C133819; SUPPLIER PART C133819 -> (none)
- U15, U16, U17, U18: footprint SC-70-5_L2.1-W1.3-P0.65-LS2.1-BR -> Maxime:SC-70-5_L2.1-W1.3-P0.65-LS2.1-BR; LCSC Part # (none) -> C133819; SUPPLIER PART C133819 -> (none)
- U4, U5, U6: LCSC Part # (none) -> C3658877; SUPPLIER PART C3658877 -> (none)
- U4: renamed from U5; LCSC Part # (none) -> C3658877; SUPPLIER PART C3658877 -> (none)
- U5: renamed from U4; LCSC Part # (none) -> C3658877; SUPPLIER PART C3658877 -> (none)
- U7: footprint WSON-6_L2.0-W2.0-P0.65-TL-EP -> Maxime:WSON-6_L2.0-W2.0-P0.65-TL-EP; LCSC Part # (none) -> C2071098; SUPPLIER PART C2071098 -> (none)
- U8: LCSC Part # (none) -> C398363; SUPPLIER PART C398363 -> (none)
Connections:
- net +BATT: now also SW1.1
- net AP: now also R38.2
- net AP_Gate: now also U6.14 (OUTD), R36.2; no longer U6.7 (OUTB)
- net GNDREF: now also C15.2, C40.2, U5.11 (VEE), C42.1, J1.3, J2.3, J3.3, J4.3, J5.3, J6.3, R12.1, R14.1, R58.1, R6.1, R8.2, RV1.1, RV4.1, RV6.1, RV7.1, RV8.1, RV9.1, U19.2 (GND), U21.3 (GND), U22.2 (V-); no longer C15.1, C40.1, R9.2, U4.11 (VEE)
- net Peak_Window: now also U19.3 (IN+); no longer U6.12 (IND+)
- net Reset_Window: now also R57.2
- net S2: now also U5.1 (OUTA), U5.7 (OUTB); no longer U5.14 (OUTD), U5.14 (OUTD)
- net S3: now also U5.14 (OUTD), U5.8 (OUTC); no longer U5.7 (OUTB), U5.8 (OUTC)
- net S4: now also U4.14 (OUTD); no longer U4.1 (OUTA)
- net Spike_Out: now also J2.2
- net Stimulus_Ext: now also J1.2
- net Syn1_Spike: now also J3.2
- net Syn2_Spike: now also J4.2
- net Syn3_Spike: now also J5.2
- net Syn4_Spike: now also J6.2
- net T2: now also U5.3 (INA-); no longer U5.13 (IND−)
- net T3: now also U5.5 (INB+), U5.9 (INC-); no longer U5.12 (IND+), U5.6 (INB-)
- net T4: now also U4.13 (IND−), U5.12 (IND+); no longer U4.3 (INA-), U5.10 (INC+)
- net VDD: now also C40.1, C41.2, U5.4 (VCC), C42.2, R11.1, R13.2, R38.1, R56.2, R96.1, RV4.3, SW1.2, U19.5 (VCC), U21.1 (IN), U22.5 (V+); no longer R7.2, U4.4 (VCC)
- net V_Leak: no longer RV5.3
- net V_Leak_Ref_Max: now also RV1.3
- net V_Leak_ref: now also RV1.2
- net V_Logic_Mid: now also R13.1, R14.2, U19.4 (IN-); no longer U6.13 (IND−)
- net V_Peak_Ref: now also R11.2, R12.2; no longer R9.1
- net V_Reset_Ref: now also R9.2
- net V_Stim_Drive: now also U6.7 (OUTB), R96.2
- net V_Syn_State: now also R83.1; no longer U2.12 (VIND+)
- net V_Threshold: now also U6.12 (IND+), R36.1, R8.1; no longer U6.5 (INB+)
- net Vm_Ext: now also J1.1, J2.1
- net Vm_Int: now also U6.13 (IND−), R84.1; no longer U6.6 (INB-)
- net Vsel: now also U4.12 (IND+), U5.10 (INC+), U5.13 (IND−), U5.2 (INA+), U5.6 (INB-), RV4.2; no longer U4.2 (INA+), U5.12 (IND+), U5.13 (IND−), U5.5 (INB+), U5.9 (INC-)
- net V_Syn_Drive: now reaches R87.1, U2.14 (VOUTD)
- net V_Syn_Drive: now also R86.2; no longer U2.13 (VIND-)
- net at U6.10 (INC+): now also R56.1, R57.1, R58.2
- net at R88.2, R89.1: now also U19.1 (OUT); no longer U6.14 (OUTD)
- net at R92.2, R93.2: now also U6.5 (INB+)
- net at R94.2, R95.2: now also U6.6 (INB-)
- net at U3.12 (VIND+): now also RV8.2
- net at U3.10 (VINC+): now also RV7.2
- net at U3.5 (VINB+): now also RV6.2
- net at U3.3 (VINA+): now also RV9.2
- net V_Leak_Ref_Max_Raw renamed VREF_2V048
- net VREF_2V048: now also C15.1, R5.2, RV6.3, RV7.3, RV8.3, RV9.3, U21.2 (OUT)
- net V_Stim_Zero_1V024 renamed VREF_1V024
- net VREF_1V024: now also R7.2, R9.1, RV5.3, R85.1, U22.1 (OUT), U22.4 (IN-); no longer C41.2
- net Vm_DRV renamed Vm_Out_DRV
- new net: R85.2, R86.1, U2.13 (VIND-)
- new net: R83.2, R84.2, U2.12 (VIND+)
- new net VREF_1V024_RAW: R5.1, R6.2, U22.3 (IN+)
- no-connect marks 1 -> 5
Other:
- note added: "0.368V (-75mV)"
- note added: "0.853V (-55mV)"
- note added: "90% VDD"
- note added: "MCP6004_U6"
- note added: "TLV7031_U19"
- note added: "Threshold voltage (incl. hysteresis): 0.853 V corresponds to -55mV"
- note removed: "12.5% VDD (-75mV)"
- note removed: "29.17% VDD (-55mV)"
- note removed: "66% VDD (-10mV)"
- note removed: "90% VDD (+20mV)"
- note removed: "TLV7044_U6"
- note removed: "Threshold voltage (incl. hysteresis): 0.865 V corresponds to -55mV"
- moved on the sheet: C15, C16, C17, C2, C3, C4, C41, C5, C6, C7, C8, D21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

Commit message: update PCB
Parts:
- removed R96: 100kΩ, JLCPCB:R_0402, symbol Spiky_Lui-altium-import:root_0_RC0402FR-07100KL_
- added C43: 100nF, JLCPCB:C_0402, symbol CL05B104KO5NNNC1_CL05B104KO5NNNC (1)-altium-import:root_0_CL05B104KO5NNNC_
- added U23: TLV9041IDBVR, SOT-23-5_L2.9-W1.6-P0.95-LS2.8-BR, symbol SpikyOscilloscopce-altium-import:root_0_TLV9041IDBVR_
- renumbered R97 to R96, U3 to U1, U2 to U1, U1 to U2, U1 to U3, U2 to U3
Connections:
- net AP: now also U2.3 (VINA+); no longer U2.10 (VINC+)
- net Adapt_Kick_Drive: now also U2.1 (VOUTA), U2.2 (VINA-); no longer U2.8 (VOUTC), U2.9 (VINC-)
- net GNDREF: now also U1.11 (VSS), U2.11 (VSS), U6.6 (INB-), C43.1, U23.2 (V-); no longer U3.11 (VSS), U3.11 (VSS)
- net Spike_Pulse: now also U6.3 (INA+); no longer U6.2 (INA+)
- net T1: now also U4.3 (INA+); no longer U4.2 (INA+)
- net T2: now also U5.2 (INA-); no longer U5.3 (INA-)
- net VDD: now also U1.4 (VDD), U2.4 (VDD), U6.5 (INB+), C43.2, U23.5 (V+); no longer U3.4 (VDD), U3.4 (VDD)
- net VREF_2V048: now also U3.5 (VINB+); no longer U3.3 (VINA+)
- net V_Leak_Ref_Max: now also U3.6 (VINB-), U3.7 (VOUTB); no longer U3.1 (VOUTA), U3.2 (VINA-)
- net V_Stim_Drive: now also U23.1 (OUT); no longer U6.7 (OUTB)
- net V_Syn1_Set: now also U1.1 (VOUTA), U1.2 (VINA-); no longer U1.6 (VINB-), U1.7 (VOUTB)
- net V_Syn2_Set: now also U1.6 (VINB-), U1.7 (VOUTB); no longer U1.8 (VOUTC), U1.9 (VINC-)
- net V_Syn3_Set: now also U3.8 (VOUTC), U3.9 (VINC-); no longer U3.13 (VIND-), U3.14 (VOUTD)
- net V_Syn4_Set: now also U3.13 (VIND-), U3.14 (VOUTD); no longer U3.1 (VOUTA), U3.2 (VINA-)
- net V_Threshold: now also U6.2 (INA-); no longer U6.3 (INA-)
- net Vsel: now also U4.2 (INA-), U5.3 (INA+); no longer U4.3 (INA-), U5.2 (INA+)
- net Vw: now also U1.10 (VINC+); no longer U1.12 (VIND+)
- net Vw_buff: now also U1.8 (VOUTC), U1.9 (VINC-); no longer U1.13 (VIND-), U1.14 (VOUTD)
- net at R41.2, R42.1: now also U2.12 (VIND+); no longer U2.5 (VINB+)
- net at R43.1, R44.1: now also U2.13 (VIND-); no longer U2.6 (VINB-)
- net Adapt: now reaches R44.2, R45.1
- net Adapt: now also U2.14 (VOUTD); no longer U2.7 (VOUTB)
- net at R92.2, R93.2: now also U23.3 (IN+); no longer U6.5 (INB+)
- net at RV7.2: now also U1.5 (VINB+); no longer U1.10 (VINC+)
- net at R94.2, R95.2: now also U23.4 (IN-); no longer U6.6 (INB-)
- net at RV9.2: now also U3.12 (VIND+); no longer U3.3 (VINA+)
- net at RV8.2: now also U3.10 (VINC+); no longer U3.12 (VIND+)
- net at RV6.2: now also U1.3 (VINA+); no longer U1.5 (VINB+)
- no-connect marks 5 -> 6
Other:
- note added: "TLV9041_U23"
- moved on the sheet: R92, R93, R94, R95, R96, U6B
