File: PCBs/LIFeling/LIFeling.kicad_pcb (KiCad board)
At the start: 2 copper layers, 119.7 x 79.7 mm, 167 parts, among them J1 Oscilloscope Jack, J2 Axon Output, J3 Syn1 Input, J4 Syn2 Input, J5 Syn3 Input, J6 Syn4 Input, Q1 N_MOSFET, Q10 SI1926DL-T1-E3, Q11 SI1926DL-T1-E3, Q12 SI1926DL-T1-E3, Q13 MMBT2222A, Q14 MMBT2222A, Q15 MMBT3904, Q16 N_MOSFET, Q17 N_MOSFET, Q18 N_MOSFET, Q19 N_MOSFET, Q2 N_MOSFET, Q20 N_MOSFET, Q3 N_MOSFET, Q4 P_MOSFET, Q5 P_MOSFET, Q6 N_MOSFET, Q7 N_MOSFET, Q8 SI3552DV-T1-E3, Q9 SI1926DL-T1-E3, SW1 SW_SPDT, U1 MCP6004T-I/ST, U2 MCP6004T-I/ST, U3 MCP6004T-I/ST, U4 LM339, U5 LM339, U6 LM339

Commit message: update pcb
Parts:
- removed the G*** at (118.0, 100.4)
- removed Q10, Q11, Q12, Q9: SI1926DL-T1-E3, Maxime:SOT-363-6_L2.0-W1.3-P0.65-LS2.1-BL
- removed Q13, Q14: MMBT2222A, PCM_JLCPCB:Q_SOT-23
- removed Q15: MMBT3904, Package_TO_SOT_SMD:SOT-23
- removed Q16, Q17, Q18, Q19, Q20: N_MOSFET, Package_TO_SOT_SMD:SOT-23
- added C1: 10uF, JLCPCB:C_0805, F.Cu at (84.5, 27.8)
- added C21: 100nF, JLCPCB:C_0402, F.Cu at (106.2, 91.4)
- added C22: 2.2uF, JLCPCB:C_0603, F.Cu at (103.9, 126.4)
- added C23: 100nF, JLCPCB:C_0402, F.Cu at (101.2, 126.3)
- added C24: 4.7uF, JLCPCB:C_0805, F.Cu at (103.5, 118.9)
- added C25: 100nF, JLCPCB:C_0402, F.Cu at (100.7, 118.3)
- added C26: 10uF, JLCPCB:C_0805, F.Cu at (113.0, 92.9)
- added C27: 100nF, JLCPCB:C_0402, F.Cu at (110.7, 91.6)
- added C28: 100pF, JLCPCB:C_0402, F.Cu at (86.4, 82.1)
- added C29: 1uF, JLCPCB:C_0603, F.Cu at (116.8, 71.4)
- added C30: 10uF, JLCPCB:C_0805, F.Cu at (140.3, 67.2)
- added C31: 10nF, JLCPCB:C_0402, F.Cu at (120.0, 76.0)
- added C32: 100nF, JLCPCB:C_0402, F.Cu at (142.9, 78.2)
- added C33: 1uF, JLCPCB:C_0402, F.Cu at (101.7, 78.3)
- added C34: 100nF, JLCPCB:C_0402, F.Cu at (66.3, 76.2)
- added C35: 100nF, JLCPCB:C_0402, F.Cu at (65.2, 100.3)
- added C36: 100nF, JLCPCB:C_0402, F.Cu at (81.1, 116.9)
- added C37: 100nF, JLCPCB:C_0402, F.Cu at (105.8, 103.0)
- added C38: 220nF, JLCPCB:C_0603, F.Cu at (96.7, 98.7)
- added C39: 100pF, JLCPCB:C_0402, F.Cu at (94.7, 51.0)
- added C40: 100nF, JLCPCB:C_0402, F.Cu at (41.1, 56.6)
- added C41: 100nF, JLCPCB:C_0402, F.Cu at (25.4, 55.7)
- added C42: 100nF, JLCPCB:C_0402, F.Cu at (162.0, 56.1)
- added C7: 100nF, JLCPCB:C_0402, F.Cu at (84.7, 109.1)
- added D10: BAT54WS L9, Maxime:SOD-323_L1.8-W1.3-LS2.5-RD, F.Cu at (55.3, 76.8)
- added D11: BAT54WS L9, Maxime:SOD-323_L1.8-W1.3-LS2.5-RD, F.Cu at (55.3, 78.7)
- added D12: BAT54WS L9, Maxime:SOD-323_L1.8-W1.3-LS2.5-RD, F.Cu at (58.5, 109.3)
- added D13: BAT54WS L9, Maxime:SOD-323_L1.8-W1.3-LS2.5-RD, F.Cu at (58.5, 111.2)
- added D14: BAT54WS L9, Maxime:SOD-323_L1.8-W1.3-LS2.5-RD, F.Cu at (82.8, 123.6)
- added D15: BAT54WS L9, Maxime:SOD-323_L1.8-W1.3-LS2.5-RD, F.Cu at (82.8, 125.4)
- added D16: BAT54WS L9, Maxime:SOD-323_L1.8-W1.3-LS2.5-RD, F.Cu at (113.3, 109.0)
- added D17: BAT54WS L9, Maxime:SOD-323_L1.8-W1.3-LS2.5-RD, F.Cu at (113.3, 110.8)
- added D18: TPD1E05U06DPYT, Maxime:X1SON-2_L1.0-W0.6-P0.65-RD, F.Cu at (165.3, 56.4)
- added D19: TPD1E05U06DPYT, Maxime:X1SON-2_L1.0-W0.6-P0.65-RD-1, F.Cu at (92.5, 51.1)
- added D20: RB521S30T1G, Maxime:SOD-523_L1.2-W0.8-LS1.6-RD, F.Cu at (133.3, 77.1)
- added D21: BAT54WS L9, Maxime:SOD-323_L1.8-W1.3-LS2.5-RD, F.Cu at (66.0, 88.0)
- added D22: BAT54WS L9, Maxime:SOD-323_L1.8-W1.3-LS2.5-RD, F.Cu at (66.0, 90.6)
- added D6: RB521S30T1G, Maxime:SOD-523_L1.2-W0.8-LS1.6-RD, F.Cu at (134.7, 69.9)
- added D7: 1N4148WS, Maxime:SOD-323_L1.8-W1.3-LS2.5-RD-1, F.Cu at (145.9, 65.5)
- added D8: RB521S30T1G, Maxime:SOD-523_L1.2-W0.8-LS1.6-RD, F.Cu at (126.3, 76.8)
- added D9: 19-237/R6GHBHC-A01/2T, Maxime:LED-SMD_4P-L1.6-W1.6-19-237A-BHR6GHC-A01-2T, F.Cu at (106.5, 51.5)
- added G***: LOGO, Maxime:LIFeling, F.Cu at (154.5, 161.5)
- added L1: 2.2uH, Maxime:IND-SMD_L3.0-W3.0_SMNR3015, F.Cu at (85.0, 64.2)
- added R95: 100kΩ, JLCPCB:R_0402, F.Cu at (90.9, 79.5)
- added R96: 100kΩ, JLCPCB:R_0402, F.Cu at (90.7, 76.8)
- added R97: 100kΩ, JLCPCB:R_0402, F.Cu at (89.8, 68.7)
- added U10: TS5A3166DCKR, Maxime:SC-70-5_L2.1-W1.3-P0.65-LS2.1-BR, F.Cu at (106.8, 89.5)
- added U11: TS5A3166DCKR, Maxime:SC-70-5_L2.1-W1.3-P0.65-LS2.1-BR, F.Cu at (101.8, 124.4)
- added U12: TS5A3166DCKR, Maxime:SC-70-5_L2.1-W1.3-P0.65-LS2.1-BR, F.Cu at (101.3, 116.3)
- added U13: TS5A3166DCKR, Maxime:SC-70-5_L2.1-W1.3-P0.65-LS2.1-BR, F.Cu at (111.2, 89.6)
- added U14: TS5A3166DCKR, Maxime:SC-70-5_L2.1-W1.3-P0.65-LS2.1-BR, F.Cu at (139.7, 78.9)
- added U15: TS5A3166DCKR, Maxime:SC-70-5_L2.1-W1.3-P0.65-LS2.1-BR, F.Cu at (69.2, 75.5)
- added U16: TS5A3166DCKR, Maxime:SC-70-5_L2.1-W1.3-P0.65-LS2.1-BR, F.Cu at (68.0, 99.6)
- added U17: TS5A3166DCKR, Maxime:SC-70-5_L2.1-W1.3-P0.65-LS2.1-BR, F.Cu at (83.9, 116.3)
- added U18: TS5A3166DCKR, Maxime:SC-70-5_L2.1-W1.3-P0.65-LS2.1-BR, F.Cu at (108.7, 102.3)
- added U19: TLV7031DCKR, Maxime:SC-70-5_L2.1-W1.3-P0.65-LS2.2-BR, F.Cu at (162.1, 53.8)
- added U20: TS5A3166DCKR, Maxime:SC-70-5_L2.1-W1.3-P0.65-LS2.1-BR, F.Cu at (115.2, 81.9)
- added U21: REF3020AIDBZR, JLCPCB:SOT-23-3_L3.0-W1.7-P0.95-LS2.9-BR, F.Cu at (28.4, 56.7)
- added U22: TLV9001IDBVR, Maxime:SOT-23-5_L3.0-W1.7-P0.95-LS2.8-BR, F.Cu at (37.3, 57.5)
- added U7: TPS610995DRVR, Maxime:WSON-6_L2.0-W2.0-P0.65-TL-EP, F.Cu at (81.1, 63.0)
- added U8: TLV9001IDBVR, Maxime:SOT-23-5_L3.0-W1.7-P0.95-LS2.8-BR, F.Cu at (91.5, 65.0)
- added U9: TS5A3166DCKR, Maxime:SC-70-5_L2.1-W1.3-P0.65-LS2.1-BR, F.Cu at (102.5, 89.4)
- C10: value 100nF -> 22uF; footprint PCM_JLCPCB:C_0402 -> JLCPCB:C_0805
- C11: value 100nF -> 1uF; footprint PCM_JLCPCB:C_0402 -> JLCPCB:C_0402
- C12, C15, C19: footprint PCM_JLCPCB:C_0402 -> JLCPCB:C_0402
- C13: value 10nF -> 100pF; footprint PCM_JLCPCB:C_0402 -> JLCPCB:C_0402
- C14, C17, C3: value 1uF -> 100nF; footprint PCM_JLCPCB:C_0402 -> JLCPCB:C_0402
- C16: value 1uF -> 22nF; footprint PCM_JLCPCB:C_0402 -> JLCPCB:C_0402
- C18: value 10uF -> 470nF; footprint PCM_JLCPCB:C_0402 -> JLCPCB:C_0603
- C2: value 470nF -> 10uF; footprint PCM_JLCPCB:C_0402 -> JLCPCB:C_0805
- C20: value 100nF -> 1uF; footprint PCM_JLCPCB:C_0402 -> JLCPCB:C_0603
- C4: value 2.2uF -> 100nF; footprint PCM_JLCPCB:C_0402 -> JLCPCB:C_0402
- C5: value 4.7uF -> 100nF; footprint PCM_JLCPCB:C_0402 -> JLCPCB:C_0402
- C6, C8: value 10uF -> 100nF; footprint PCM_JLCPCB:C_0402 -> JLCPCB:C_0402
- C9: value 100nF -> 10uF; footprint PCM_JLCPCB:C_0402 -> JLCPCB:C_0805
- D1: value 1N4148W -> TPD1E05U06DPYT; footprint Maxime:SOD-123_L2.8-W1.8-LS3.7-RD -> Maxime:X1SON-2_L1.0-W0.6-P0.65-RD-1
- D2: value 19-237/R6GHBHC-A01/2T -> BAT54WS L9; footprint Maxime:LED-SMD_4P-L1.6-W1.6-19-237A-BHR6GHC-A01-2T -> Maxime:SOD-323_L1.8-W1.3-LS2.5-RD
- D3: value 1N4148WS -> BAT54WS L9; footprint PCM_JLCPCB:D_SOD-323 -> Maxime:SOD-323_L1.8-W1.3-LS2.5-RD
- D4, D5: footprint PCM_JLCPCB:D_SOD-323 -> Maxime:SOD-323_L1.8-W1.3-LS2.5-RD-1
- J1: value Oscilloscope Jack -> Stim_Ext; footprint Maxime:AUDIO-SMD_PJ-320B -> Maxime:AUDIO-SMD_HX-PJ-320A-3P-DIP
- J2: value Axon Output -> Axon_Output; footprint Maxime:AUDIO-SMD_PJ-320B -> Maxime:AUDIO-SMD_HX-PJ-320A-3P-DIP
- J3: value Syn1 Input -> Syn1_Input; footprint Maxime:AUDIO-SMD_PJ-320B -> Maxime:AUDIO-SMD_HX-PJ-320A-3P-DIP
- J4: value Syn2 Input -> Syn2_Input; footprint Maxime:AUDIO-SMD_PJ-320B -> Maxime:AUDIO-SMD_HX-PJ-320A-3P-DIP
- J5: value Syn3 Input -> Syn3_Input; footprint Maxime:AUDIO-SMD_PJ-320B -> Maxime:AUDIO-SMD_HX-PJ-320A-3P-DIP
- J6: value Syn4 Input -> Syn4_Input; footprint Maxime:AUDIO-SMD_PJ-320B -> Maxime:AUDIO-SMD_HX-PJ-320A-3P-DIP
- Q1, Q3, Q6, Q7: value N_MOSFET -> BSS138; footprint Package_TO_SOT_SMD:SOT-23 -> JLCPCB:SOT-23-3_L2.9-W1.6-P1.90-LS2.8-BR
- Q2: value N_MOSFET -> MMBT3904; footprint Package_TO_SOT_SMD:SOT-23 -> JLCPCB:SOT-23-3_L2.9-W1.6-P1.90-LS2.8-BR
- Q4, Q5: value P_MOSFET -> BSS138; footprint Package_TO_SOT_SMD:SOT-23 -> JLCPCB:SOT-23-3_L2.9-W1.6-P1.90-LS2.8-BR
- Q8: value SI3552DV-T1-E3 -> MMBT3904; footprint Maxime:TSOP-6_L3.0-W1.5-P0.95-BL -> JLCPCB:SOT-23-3_L2.9-W1.6-P1.90-LS2.8-BR
- R1: value 6.8kΩ -> 10Ω; footprint PCM_JLCPCB:R_0402 -> JLCPCB:R_0402
- R10: value 100kΩ -> 56kΩ; footprint PCM_JLCPCB:R_0402 -> JLCPCB:R_0402
- R11: value 1MΩ -> 100kΩ; footprint PCM_JLCPCB:R_0402 -> JLCPCB:R_0402
- R12, R28, R29, R83, R86: value 100kΩ -> 1MΩ; footprint PCM_JLCPCB:R_0402 -> JLCPCB:R_0402
- R13: value 1MΩ -> 220kΩ; footprint PCM_JLCPCB:R_0402 -> JLCPCB:R_0402
- R14: value 100kΩ -> 220kΩ; footprint PCM_JLCPCB:R_0402 -> JLCPCB:R_0402
- R15, R18, R22, R33, R9: value 22kΩ -> 100kΩ; footprint PCM_JLCPCB:R_0402 -> JLCPCB:R_0402
- R16: value 1Ω -> 10kΩ; footprint PCM_JLCPCB:R_0402 -> JLCPCB:R_0402
- R17: value 27kΩ -> 100kΩ; footprint PCM_JLCPCB:R_0402 -> JLCPCB:R_0402
- R19, R21, R24, R30, R48, R5, R54, R58, R59, R60, R65, R68, R72, R76, R80, R84, R90, R92: footprint PCM_JLCPCB:R_0402 -> JLCPCB:R_0402
- R2: value 1kΩ -> 220Ω; footprint PCM_JLCPCB:R_0402 -> JLCPCB:R_0402
- R20, R55: value 4.7kΩ -> 100kΩ; footprint PCM_JLCPCB:R_0402 -> JLCPCB:R_0402
- R23, R31, R32: value 22kΩ -> 1MΩ; footprint PCM_JLCPCB:R_0402 -> JLCPCB:R_0402
- R25, R26, R50: value 100Ω -> 1MΩ; footprint PCM_JLCPCB:R_0402 -> JLCPCB:R_0402
- R27, R42, R43, R49, R51: value 100Ω -> 100kΩ; footprint PCM_JLCPCB:R_0402 -> JLCPCB:R_0402
- R3: value 1kΩ -> 10kΩ; footprint PCM_JLCPCB:R_0402 -> JLCPCB:R_0402
- R34: value 47kΩ -> 1MΩ; footprint PCM_JLCPCB:R_0402 -> JLCPCB:R_0402
- R35: value 47kΩ -> 1kΩ; footprint PCM_JLCPCB:R_0402 -> JLCPCB:R_0402
- R36: value 22kΩ -> 2.2MΩ; footprint PCM_JLCPCB:R_0402 -> JLCPCB:R_0402
- R37: value 2.4kΩ -> 10kΩ; footprint PCM_JLCPCB:R_0402 -> JLCPCB:R_0402
- R38: value 2.4kΩ -> 100kΩ; footprint PCM_JLCPCB:R_0402 -> JLCPCB:R_0402
- R39, R47, R53: value 100Ω -> 22kΩ; footprint PCM_JLCPCB:R_0402 -> JLCPCB:R_0402
- R4: value 2kΩ -> 100kΩ; footprint PCM_JLCPCB:R_0402 -> JLCPCB:R_0402
- R40, R89: value 100kΩ -> 100Ω; footprint PCM_JLCPCB:R_0402 -> JLCPCB:R_0402
- R41: value 100Ω -> 200kΩ; footprint PCM_JLCPCB:R_0402 -> JLCPCB:R_0402
- R44: value 100kΩ -> 200kΩ; footprint PCM_JLCPCB:R_0402 -> JLCPCB:R_0402
- R45: value 100Ω -> 330kΩ; footprint PCM_JLCPCB:R_0402 -> JLCPCB:R_0402
- R46: value 100Ω -> 10kΩ; footprint PCM_JLCPCB:R_0402 -> JLCPCB:R_0402
- R52: value 100kΩ -> 10kΩ; footprint PCM_JLCPCB:R_0402 -> JLCPCB:R_0402
- R56: value 220kΩ -> 270kΩ; footprint PCM_JLCPCB:R_0402 -> JLCPCB:R_0402
- R57: value 220kΩ -> 1MΩ; footprint PCM_JLCPCB:R_0402 -> JLCPCB:R_0402
- R6: value 47kΩ -> 220kΩ; footprint PCM_JLCPCB:R_0402 -> JLCPCB:R_0402
- R61: value 300kΩ -> 2kΩ; footprint PCM_JLCPCB:R_0402 -> JLCPCB:R_0402
- R62, R63: value 10kΩ -> 2kΩ; footprint PCM_JLCPCB:R_0402 -> JLCPCB:R_0402
- R64: value 220Ω -> 10kΩ; footprint PCM_JLCPCB:R_0402 -> JLCPCB:R_0402
- R66, R70: value 100kΩ -> 22kΩ; footprint PCM_JLCPCB:R_0402 -> JLCPCB:R_0402
- R67, R71, R75: value 1MΩ -> 1kΩ; footprint PCM_JLCPCB:R_0402 -> JLCPCB:R_0402
- R69, R73, R74, R77, R78, R81: value 1MΩ -> 22kΩ; footprint PCM_JLCPCB:R_0402 -> JLCPCB:R_0402
- R7: value 220kΩ -> 20kΩ; footprint PCM_JLCPCB:R_0402 -> JLCPCB:R_0402
- R79: value 100kΩ -> 1kΩ; footprint PCM_JLCPCB:R_0402 -> JLCPCB:R_0402
- R8: value 10kΩ -> 100kΩ; footprint PCM_JLCPCB:R_0402 -> JLCPCB:R_0402
- R82: value 10Ω -> 10kΩ; footprint PCM_JLCPCB:R_0402 -> JLCPCB:R_0402
- R85: value 10Ω -> 1MΩ; footprint PCM_JLCPCB:R_0402 -> JLCPCB:R_0402
- R87: value 1MΩ -> 47kΩ; footprint PCM_JLCPCB:R_0402 -> JLCPCB:R_0402
- R88: value 10Ω -> 100kΩ; footprint PCM_JLCPCB:R_0402 -> JLCPCB:R_0402
- R91: value 10Ω -> 1kΩ; footprint PCM_JLCPCB:R_0402 -> JLCPCB:R_0402
- R93: value 1MΩ -> 200kΩ; footprint PCM_JLCPCB:R_0402 -> JLCPCB:R_0402
- R94: value 10Ω -> 200kΩ; footprint PCM_JLCPCB:R_0402 -> JLCPCB:R_0402
- RV3: value 50kΩ -> 100kΩ
- RV4: value 10kΩ -> 100kΩ
- RV6, RV7, RV8: value 100kΩ -> 1MΩ
- RV9: value 50kΩ -> 1MΩ
- SW1: value SW_SPDT -> K3-1260D-L1; footprint Maxime:SW-SMD_SSAJ120100 -> Maxime:SW-TH_K3-1260D-L1
- U4, U5, U6: value LM339 -> TLV7044PWR
- moved H6 211.2 mm to (264.0, 14.1)
- moved H1 210.4 mm to (252.1, 8.18)
- moved H2 189.6 mm to (252.1, 14.1)
- moved H5 181.4 mm to (264.0, 8.18)
- moved H3 166.3 mm to (258.0, 8.18)
- moved R14 117.9 mm to (43.7, 63.9)
- moved R12 116.7 mm to (39.0, 63.7)
- moved R10 114.1 mm to (32.8, 63.9), turned to 0 degrees
- moved R13 112.4 mm to (43.8, 61.8)
- moved R11 108.3 mm to (39.1, 61.6)
- moved R8 104.2 mm to (27.8, 63.9), turned to 0 degrees
- moved H4 104.1 mm to (258.0, 14.1)
- moved R9 99.8 mm to (33.0, 61.7), turned to 0 degrees
- moved R7 99.0 mm to (28.0, 61.5), turned to 0 degrees
- moved R21 98.6 mm to (80.6, 95.1)
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Connections:
- net /V_ref renamed /V_Leak_ref
- C10 pad 1: VDD -> GNDREF
- C10 pad 2: GNDREF -> Net-(U7-VOUT)
- C11 pad 1: VDD -> V_Boost
- C12 pad 1: VDD -> V_Boost
- C13 pad 1: AP -> Vm_Ext
- C13 pad 2: /Rising_AP -> GNDREF
- C14 pad 1: Net-(U4B--) -> V_Boost
- C15 pad 1: VDD -> VREF_2V048
- C16 pad 1: Net-(U1B-VINC-) -> GNDREF
- C16 pad 2: /Vkick -> Vm_Display_In
- C17 pad 1: GNDREF -> VDD
- C17 pad 2: /Vw -> GNDREF
- C18 pad 1: V_Synapses -> Net-(U9-NO)
- C18 pad 2: Net-(U2A-VOUTB) -> GNDREF
- C19 pad 1: Net-(U2A-VINB+) -> VDD
- C2 pad 1: Net-(Q16-S) -> VDD
- C20 pad 1: VDD -> Net-(U10-NO)
- C3 pad 1: Net-(Q17-S) -> GNDREF
- C3 pad 2: GNDREF -> VDD
- C4 pad 1: Net-(Q18-S) -> GNDREF
- C4 pad 2: GNDREF -> VDD
- C5 pad 1: Net-(Q19-S) -> GNDREF
- C5 pad 2: GNDREF -> VDD
- C6 pad 1: Net-(Q20-S) -> GNDREF
- C6 pad 2: GNDREF -> VDD
- C8 pad 1: +BATT -> GNDREF
- C8 pad 2: GNDREF -> VDD
- D1 pad 1: Spike -> Vm_Ext
- D1 pad 2: /Rising_AP -> GNDREF
- D2 pad 1: Net-(D2-R-) -> VDD
- D2 pad 2: Net-(D2-B-) -> Vm_Int
- D3 pad 1: /Vkick -> Vm_Int
- D4 pad 1: /Vw -> /Vkick
- D4 pad 2: /Vkick -> GNDREF
- D5 pad 1: /Vw -> Vw
- D5 pad 2: GNDREF -> /Vkick
- J1 pad 1: GNDREF -> Vm_Ext
- J1 pad 2: Stimulus_In -> Stimulus_Ext
- J1 pad 3: Vm -> GNDREF
- J2 pad 1: GNDREF -> Vm_Ext
- J2 pad 2: Spike -> Spike_Out
- J2 pad 3: Vm -> GNDREF
- J3 pad 1: GNDREF -> unconnected-(J3-Pad1)
- J3 pad 3: Syn1_Vm -> GNDREF
- J4 pad 1: GNDREF -> unconnected-(J4-Pad1)
- J4 pad 3: Syn2_Vm -> GNDREF
- J5 pad 1: GNDREF -> unconnected-(J5-Pad1)
- J5 pad 3: Syn3_Vm -> GNDREF
- J6 pad 1: GNDREF -> unconnected-(J6-Pad1)
- J6 pad 3: Syn4_Vm -> GNDREF
- Q1 pad 1: SP -> /AP_Gate
- Q2 pad 1: AP -> /Adapt_Base
- Q2 pad 3: Net-(Q2-D) -> /Adapt_Current_Sink
- Q3 pad 1: Spike -> AP
- Q3 pad 3: Net-(Q3-D) -> /Reset_Timer_Discharge
- Q4 pad 1: Net-(Q4-G) -> Peak_Window
- Q4 pad 2: VDD -> GNDREF
- Q4 pad 3: Vm -> /Reset_Injection_Enable
- Q5 pad 1: Net-(Q4-G) -> /Reset_Injection_Enable
- Q5 pad 2: Peak -> /Reset_Injection_Drive
- Q5 pad 3: GNDREF -> /Reset_Switch_Mid
- Q6 pad 1: Peak -> Reset_Window
- Q6 pad 2: /Reset_Current_Injection -> /Reset_Switch_Mid
- Q6 pad 3: Net-(Q6-D) -> /Reset_Gated_Drive
- Q7 pad 1: Reset -> Reset_Window
- Q7 pad 2: Net-(Q6-D) -> GNDREF
- Q8 pad 1: Net-(Q8-NG) -> Net-(Q8-Pad1)
- Q8 pad 2: Net-(Q8-PS) -> GNDREF
- Q8 pad 3: Net-(Q8-PG) -> Net-(Q8-Pad3)
- R1 pad 1: VDD -> Net-(U7-VOUT)
- R1 pad 2: +0.375V -> V_Boost
- R10 pad 1: /Rising_AP -> GNDREF
- R10 pad 2: GNDREF -> V_Reset_Ref
- R11 pad 1: Spike -> VDD
- R11 pad 2: GNDREF -> V_Peak_Ref
- R12 pad 1: Net-(Q3-D) -> GNDREF
- R12 pad 2: Net-(Q4-G) -> V_Peak_Ref
- R13 pad 1: VDD -> V_Logic_Mid
- R13 pad 2: Net-(Q4-G) -> VDD
- R14 pad 1: VDD -> GNDREF
- R14 pad 2: Peak -> V_Logic_Mid
- R15 pad 1: VDD -> Vm_Display_In
- R15 pad 2: Net-(U4B--) -> Vm_Int
- R16 pad 1: Net-(U4B--) -> Net-(U20-NO)
- R16 pad 2: Net-(Q2-D) -> V_Peak_Drive
- R17 pad 2: Net-(U4B-+) -> T4
- R18 pad 1: Net-(U4B-+) -> T4
- R18 pad 2: GNDREF -> T3
- R19 pad 1: Net-(U4B-+) -> T3
- R19 pad 2: Reset -> T2
- R2 pad 1: +0.375V -> Vm_Out_DRV
- R2 pad 2: GNDREF -> Vm_Ext
- R20 pad 1: VDD -> T2
- R20 pad 2: Reset -> T1
- R21 pad 1: Net-(Q7-D) -> T1
- R21 pad 2: Vm -> GNDREF
- R22 pad 1: /Vkick -> VDD
- R22 pad 2: GNDREF -> S0
- R23 pad 1: /Vw_buf -> T1
- R23 pad 2: Net-(Q15-B) -> S0
- R24 pad 1: GNDREF -> VDD
- R24 pad 2: Net-(Q15-B) -> S1
- R25 pad 1: Net-(Q15-C) -> T1
- R25 pad 2: Vm -> S1
- R26 pad 1: Net-(R26-Pad1) -> T2
- R26 pad 2: GNDREF -> S1
- R27 pad 1: Vm -> VDD
- R27 pad 2: Stimulus_In -> S2
- R28 pad 1: VDD -> T2
- R28 pad 2: T4 -> S2
- R29 pad 1: T4 -> T3
- R29 pad 2: T3 -> S2
- R3 pad 1: VDD -> Vm_FB
- R3 pad 2: +2V -> Vm_Out_DRV
- R30 pad 1: T3 -> VDD
- R30 pad 2: T2 -> S3
- R31 pad 1: VDD -> T3
- R31 pad 2: Net-(U2A-VINB+) -> S3
- R32 pad 1: Net-(U2A-VINB+) -> T4
- R32 pad 2: GNDREF -> S3
- R33 pad 2: Net-(U2B-VINC+) -> S4
- R34 pad 1: Net-(U2B-VINC+) -> T4
- R34 pad 2: Net-(U2A-VOUTB) -> S4
- R35 pad 1: Net-(U2A-VOUTB) -> Net-(R35-Pad1)
- R35 pad 2: Net-(U2C-VIND-) -> Vm_Int
- R36 pad 1: Net-(U2C-VIND-) -> V_Threshold
- R36 pad 2: GNDREF -> /AP_Gate
- R37 pad 2: Net-(Q8-PS) -> /AP_Gate
- R38 pad 1: Net-(Q8-NS) -> VDD
- R38 pad 2: GNDREF -> AP
- R39 pad 1: Syn1_Spike -> GNDREF
- R39 pad 2: Net-(Q9-G1) -> /Vkick
- R4 pad 1: +2V -> GNDREF
- R4 pad 2: GNDREF -> Vm_FB
- R40 pad 1: GNDREF -> Net-(R40-Pad1)
- R40 pad 2: Net-(Q9-G1) -> GNDREF
- R41 pad 1: Net-(U3A-VINB-) -> GNDREF
- R41 pad 2: Net-(Q9-S1) -> Net-(U1A-VINB+)
- R42 pad 1: Net-(Q9-D1) -> Net-(U1A-VINB+)
- R42 pad 2: Net-(Q10-S2) -> Vm_Int
- R43 pad 1: Syn2_Spike -> Net-(U1A-VINB-)
- R43 pad 2: Net-(Q10-G1) -> V_Leak
- R44 pad 1: GNDREF -> Net-(U1A-VINB-)
- R44 pad 2: Net-(Q10-G1) -> Net-(U1A-VOUTB)
- R45 pad 1: Net-(U3B-VINC-) -> Net-(U1A-VOUTB)
- R46 pad 1: Net-(Q10-D1) -> Vm_Int
- R46 pad 2: Net-(Q10-S2) -> /Adapt_Current_Sink
- R47 pad 1: Syn3_Spike -> /Adapt_Base
- R47 pad 2: Net-(Q11-G1) -> Vw_buff
- R48 pad 1: GNDREF -> /Adapt_Base
- R48 pad 2: Net-(Q11-G1) -> GNDREF
- R49 pad 1: Net-(U3C-VIND-) -> /Rising_AP
- R49 pad 2: Net-(Q11-S1) -> GNDREF
- R5 pad 1: VDD -> VREF_1V024_RAW
- R5 pad 2: /V_Threshold -> VREF_2V048
- R50 pad 1: Net-(Q11-D1) -> GNDREF
- R50 pad 2: Net-(Q10-S2) -> Spike_Pulse
- R51 pad 1: Syn4_Spike -> VDD
- R51 pad 2: Net-(Q12-G1) -> Peak_Window
- R52 pad 1: GNDREF -> Net-(U14-NO)
- R52 pad 2: Net-(Q12-G1) -> V_Peak_Drive
- R53 pad 1: Net-(U3D-VINA-) -> VDD
- R53 pad 2: Net-(Q12-S1) -> Net-(U6C-INC-)
- R54 pad 1: Net-(Q12-D1) -> /Reset_Timer_Discharge
- R54 pad 2: Net-(Q10-S2) -> Net-(U6C-INC-)
- R55 pad 1: Net-(Q10-S2) -> VDD
- R55 pad 2: V_Synapses -> Reset_Window
- R56 pad 1: VDD -> Net-(U6C-INC+)
- R56 pad 2: /V_Spike_Threshold -> VDD
- R57 pad 1: /V_Spike_Threshold -> Net-(U6C-INC+)
- R57 pad 2: GNDREF -> Reset_Window
- R58 pad 1: /V_Spike_Threshold -> GNDREF
- R58 pad 2: Net-(R58-Pad2) -> Net-(U6C-INC+)
- R59 pad 2: Net-(R58-Pad2) -> /Reset_Injection_Enable
- R6 pad 1: /V_Threshold -> GNDREF
- R6 pad 2: GNDREF -> VREF_1V024_RAW
- R60 pad 1: Net-(Q14-B) -> /Reset_Gated_Drive
- R60 pad 2: Net-(R58-Pad2) -> Vm_Int
- R61 pad 1: Net-(R58-Pad2) -> Net-(Q7-D)
- R61 pad 2: Net-(U4C-+) -> Net-(D9-B-)
- R62 pad 1: Net-(U2D-VINA-) -> Net-(Q7-D)
- R62 pad 2: Net-(U4C-+) -> Net-(D9-G-)
- R63 pad 1: Net-(U2D-VINA-) -> Net-(Q8-Pad3)
- R64 pad 1: VDD -> Net-(Q8-Pad1)
- R64 pad 2: Net-(D2-+) -> Vm_Int
- R65 pad 1: T2 -> Net-(Q8-Pad1)
- R65 pad 2: T1 -> GNDREF
- R66 pad 1: T1 -> Net-(U15-NO)
- R66 pad 2: GNDREF -> V_Syn_State
- R67 pad 1: T4 -> Net-(U15-IN)
- R67 pad 2: S0 -> Net-(D10-A)
- R68 pad 1: S0 -> GNDREF
- R68 pad 2: VDD -> Net-(D10-A)
- R69 pad 1: T1 -> Syn1_Spike
- R69 pad 2: S4 -> Net-(D10-A)
- R7 pad 1: /V_Threshold -> V_Threshold
- R7 pad 2: SP -> VREF_1V024
- R70 pad 1: S4 -> Net-(U16-NO)
- R70 pad 2: VDD -> V_Syn_State
- R71 pad 1: Vsel -> Net-(U16-IN)
- R71 pad 2: S1 -> Net-(D12-A)
- R72 pad 1: S1 -> GNDREF
- R72 pad 2: VDD -> Net-(D12-A)
- R73 pad 1: T3 -> Syn2_Spike
- R73 pad 2: S1 -> Net-(D12-A)
- R74 pad 1: Vsel -> Net-(U17-NO)
- R74 pad 2: S2 -> V_Syn_State
- R75 pad 1: T2 -> Net-(U17-IN)
- R75 pad 2: S2 -> Net-(D14-A)
- R76 pad 1: S2 -> GNDREF
- R76 pad 2: VDD -> Net-(D14-A)
- R77 pad 1: Vsel -> Syn3_Spike
- R77 pad 2: S3 -> Net-(D14-A)
- R78 pad 1: T1 -> Net-(U18-NO)
- R78 pad 2: S3 -> V_Syn_State
- R79 pad 1: S3 -> Net-(U18-IN)
- R79 pad 2: VDD -> Net-(D16-A)
- R8 pad 1: VDD -> V_Threshold
- R8 pad 2: SP -> GNDREF
- R80 pad 1: S0 -> GNDREF
- R80 pad 2: Net-(Q16-G) -> Net-(D16-A)
- R81 pad 1: Net-(Q16-G) -> Syn4_Spike
- R81 pad 2: Net-(Q16-S) -> Net-(D16-A)
- R82 pad 1: Vm -> V_Syn_State
- R82 pad 2: Net-(Q16-D) -> Net-(R82-Pad2)
- R83 pad 1: S1 -> V_Syn_State
- R83 pad 2: Net-(Q17-G) -> Net-(U2C-VIND+)
- R84 pad 1: Net-(Q17-G) -> Vm_Int
- R84 pad 2: Net-(Q17-S) -> Net-(U2C-VIND+)
- R85 pad 1: Vm -> VREF_1V024
- R85 pad 2: Net-(Q17-D) -> Net-(U2C-VIND-)
- R86 pad 1: S2 -> Net-(U2C-VIND-)
- R86 pad 2: Net-(Q18-G) -> /V_Syn_Drive
- R87 pad 1: Net-(Q18-G) -> /V_Syn_Drive
- R87 pad 2: Net-(Q18-S) -> Vm_Int
- R88 pad 1: Vm -> VDD
- R88 pad 2: Net-(Q18-D) -> Net-(U19-OUT)
- R89 pad 1: S3 -> Net-(U19-OUT)
- R89 pad 2: Net-(Q19-G) -> Spike_Out
- R9 pad 1: VDD -> VREF_1V024
- R9 pad 2: AP -> V_Reset_Ref
- R90 pad 1: Net-(Q19-G) -> VREF_1V024
- R90 pad 2: Net-(Q19-S) -> V_Stim_Cmd
- R91 pad 1: Vm -> Stimulus_Ext
- R91 pad 2: Net-(Q19-D) -> V_Stim_Cmd
- R92 pad 1: S4 -> Vm_Int
- R92 pad 2: Net-(Q20-G) -> Net-(U6B-INB+)
- R93 pad 1: Net-(Q20-G) -> V_Stim_Cmd
- R93 pad 2: Net-(Q20-S) -> Net-(U6B-INB+)
- R94 pad 1: Vm -> VREF_1V024
- R94 pad 2: Net-(Q20-D) -> Net-(U6B-INB-)
- RV1 pad 3: +2V -> V_Leak_Ref_Max
- RV2 pad 1: Vm -> Net-(R35-Pad1)
- RV2 pad 2: Vm -> Vm_Int
- RV2 pad 3: /V_Leak -> V_Leak
- RV3 pad 1: /Vw -> Vw
- RV3 pad 2: /Vw -> Vw
- RV3 pad 3: Net-(R26-Pad1) -> Net-(R40-Pad1)
- RV4 pad 1: Net-(U2A-VOUTB) -> GNDREF
- RV4 pad 2: Net-(U2A-VOUTB) -> Vsel
- RV4 pad 3: V_Synapses -> VDD
- RV5 pad 1: GNDREF -> Net-(R82-Pad2)
- RV5 pad 2: Net-(U3A-VINB+) -> Net-(R82-Pad2)
- RV5 pad 3: VDD -> VREF_1V024
- RV6 pad 2: Net-(U3B-VINC+) -> Net-(U3A-VINB+)
- RV6 pad 3: VDD -> VREF_2V048
- RV7 pad 2: Net-(U3C-VIND+) -> Net-(U3B-VINC+)
- RV7 pad 3: VDD -> VREF_2V048
- RV8 pad 2: Net-(U3D-VINA+) -> Net-(U3C-VIND+)
- RV8 pad 3: VDD -> VREF_2V048
- RV9 pad 2: Vsel -> Net-(U3D-VINA+)
- RV9 pad 3: VDD -> VREF_2V048
- SW1 pad 1: VDD -> +BATT
- SW1 pad 2: +BATT -> VDD
- U1 pad 1: /V_Leak -> V_Leak
- U1 pad 10: SP -> AP
- U1 pad 12: /Vw -> Vw
- U1 pad 13: /Vw_buf -> Vw_buff
- U1 pad 14: /Vw_buf -> Vw_buff
- U1 pad 2: /V_Leak -> V_Leak
- U1 pad 5: +0.375V -> Net-(U1A-VINB+)
- U1 pad 6: /Reset_Current_Injection -> Net-(U1A-VINB-)
- U1 pad 7: /Reset_Current_Injection -> Net-(U1A-VOUTB)
- U1 pad 8: Net-(U1B-VINC-) -> /Adapt_Kick_Drive
- U1 pad 9: Net-(U1B-VINC-) -> /Adapt_Kick_Drive
- U2 pad 1: Net-(U2D-VINA-) -> V_Leak_Ref_Max
- U2 pad 10: Net-(U2B-VINC+) -> V_Peak_Ref
- U2 pad 12: Net-(Q8-NS) -> Net-(U2C-VIND+)
- U2 pad 14: Net-(Q8-NG) -> /V_Syn_Drive
- U2 pad 2: Net-(U2D-VINA-) -> V_Leak_Ref_Max
- U2 pad 3: Vm -> VREF_2V048
- U2 pad 5: Net-(U2A-VINB+) -> V_Reset_Ref
- U2 pad 6: V_Synapses -> /Reset_Injection_Drive
- U2 pad 7: Net-(U2A-VOUTB) -> /Reset_Injection_Drive
- U2 pad 8: Net-(Q8-PG) -> V_Peak_Drive
- U2 pad 9: Net-(Q8-PS) -> V_Peak_Drive
- U3 pad 1: Net-(U3D-VINA-) -> V_Syn4_Set
- U3 pad 13: Net-(U3C-VIND-) -> V_Syn3_Set
- U3 pad 14: Net-(U3C-VIND-) -> V_Syn3_Set
- U3 pad 2: Net-(U3D-VINA-) -> V_Syn4_Set
- U3 pad 6: Net-(U3A-VINB-) -> V_Syn1_Set
- U3 pad 7: Net-(U3A-VINB-) -> V_Syn1_Set
- U3 pad 8: Net-(U3B-VINC-) -> V_Syn2_Set
- U3 pad 9: Net-(U3B-VINC-) -> V_Syn2_Set
- U4 pad 1: Reset -> S0
- U4 pad 10: /V_Spike_Threshold -> T2
- U4 pad 11: Net-(U4C-+) -> GNDREF
- U4 pad 12: GNDREF -> Vsel
- U4 pad 13: Net-(R58-Pad2) -> T4
- U4 pad 14: unconnected-(U4-Pad14) -> S4
- U4 pad 2: SP -> T1
- U4 pad 3: VDD -> Vsel
- U4 pad 4: Vm -> VDD
- U4 pad 5: /V_Threshold -> Vsel
- U4 pad 6: Net-(U4B--) -> T1
- U4 pad 7: Net-(U4B-+) -> S1
- U4 pad 8: unconnected-(U4D---Pad8) -> S1
- U4 pad 9: unconnected-(U4D-+-Pad9) -> Vsel
- U5 pad 1: S4 -> S2
- U5 pad 11: T3 -> GNDREF
- U5 pad 12: GNDREF -> T4
- U5 pad 13: S1 -> Vsel
- U5 pad 14: S1 -> S3
- U5 pad 2: S0 -> Vsel
- U5 pad 3: VDD -> T2
- U5 pad 4: Vsel -> VDD
- U5 pad 5: T4 -> T3
- U5 pad 7: T1 -> S2
- U5 pad 8: T4 -> S3
- U5 pad 9: Vsel -> T3
- U6 pad 1: S2 -> Peak_Window
- U6 pad 10: Vsel -> Net-(U6C-INC+)
- U6 pad 11: T1 -> GNDREF
- U6 pad 12: GNDREF -> V_Threshold
- U6 pad 13: S3 -> Vm_Int
- U6 pad 14: S3 -> /AP_Gate
- U6 pad 2: S2 -> Spike_Pulse
- U6 pad 3: VDD -> V_Threshold
- U6 pad 4: Vsel -> VDD
- U6 pad 5: T2 -> Net-(U6B-INB+)
- U6 pad 6: T3 -> Net-(U6B-INB-)
- U6 pad 7: Vsel -> V_Stim_Drive
- U6 pad 8: T2 -> Reset_Window
- U6 pad 9: Vsel -> Net-(U6C-INC-)
Routing:
- net VDD: track 365.9 -> 14.6 mm, vias 32 -> 0
- net Vm: track 274.4 -> 0.00 mm, vias 17 -> 0
- net Net-(Q10-S2): track 162.5 -> 0.00 mm, vias 10 -> 0
- net Vsel: track 149.8 -> 0.00 mm, vias 9 -> 0
- net Reset: track 93.7 -> 0.00 mm, vias 2 -> 0
- net Net-(U3B-VINC-): track 81.9 -> 0.00 mm, vias 4 -> 0
- net Net-(U3A-VINB+): track 79.0 -> 0.00 mm, vias 2 -> 0
- net Net-(U3A-VINB-): track 75.9 -> 0.00 mm
- net /Reset_Current_Injection: track 75.8 -> 0.00 mm, vias 2 -> 0
- net T1: track 81.9 -> 9.99 mm, vias 5 -> 0
- net +0.375V: track 71.4 -> 0.00 mm, vias 4 -> 0
- net Net-(U3B-VINC+): track 68.1 -> 0.00 mm, vias 4 -> 0
- net T2: track 75.6 -> 8.26 mm, vias 5 -> 0
- net /Vw: track 62.6 -> 0.00 mm, vias 7 -> 0
- net S3: track 60.6 -> 0.00 mm, vias 3 -> 0
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- removed copper zone on B.Cu, net GNDREF
- removed copper zone on F.Cu, net GNDREF
Other:
- board size 119.7 x 79.7 mm -> 119.2 x 79.8 mm
- board text removed: "C"
- board text removed: "G"
- board text removed: "V"
- board text removed: "adapt"
- board text removed: "leak"
- board text removed: "m"
- board text removed: "syn"
- board text removed: "τ"

Commit message: update PCB
Parts:
- moved R14 120.7 mm to (164.3, 56.8)
- moved R13 120.6 mm to (164.3, 55.8), turned to 180 degrees
- moved R15 91.7 mm to (151.1, 67.3), turned to 90 degrees
- moved C16 87.6 mm to (146.3, 67.3), turned to -90 degrees
- moved D22 85.5 mm to (148.7, 68.7)
- moved D21 85.3 mm to (148.7, 67.0), turned to 180 degrees
- moved G*** 81.0 mm to (112.6, 92.1)
- moved BT1 69.0 mm to (91.5, 83.8), turned to 90 degrees
- moved C41 67.3 mm to (72.4, 103.9), turned to 90 degrees
- moved R11 64.4 mm to (102.5, 72.9), turned to 180 degrees
- moved R12 64.3 mm to (102.5, 74.0), turned to 180 degrees
- moved R8 63.5 mm to (90.9, 70.7), turned to 180 degrees
- moved R7 63.5 mm to (90.9, 69.7), turned to 180 degrees
- moved U21 62.0 mm to (71.3, 101.5)
- moved C15 60.3 mm to (74.1, 100.5)
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Connections:
- R41 pad 2: Net-(U1A-VINB+) -> Net-(U2C-VIND+)
- R42 pad 1: Net-(U1A-VINB+) -> Net-(U2C-VIND+)
- R43 pad 1: Net-(U1A-VINB-) -> Net-(U2C-VIND-)
- R44 pad 1: Net-(U1A-VINB-) -> Net-(U2C-VIND-)
- R44 pad 2: Net-(U1A-VOUTB) -> /Adapt
- R45 pad 1: Net-(U1A-VOUTB) -> /Adapt
- R83 pad 2: Net-(U2C-VIND+) -> Net-(U1C-VIND+)
- R84 pad 2: Net-(U2C-VIND+) -> Net-(U1C-VIND+)
- R85 pad 2: Net-(U2C-VIND-) -> Net-(U1C-VIND-)
- R86 pad 1: Net-(U2C-VIND-) -> Net-(U1C-VIND-)
- RV6 pad 2: Net-(U3A-VINB+) -> Net-(U1D-VINA+)
- RV7 pad 2: Net-(U3B-VINC+) -> Net-(U1A-VINB+)
- RV8 pad 2: Net-(U3C-VIND+) -> Net-(U3B-VINC+)
- RV9 pad 2: Net-(U3D-VINA+) -> Net-(U3C-VIND+)
- U1 pad 1: V_Leak -> V_Syn1_Set
- U1 pad 10: AP -> Vw
- U1 pad 12: Vw -> Net-(U1C-VIND+)
- U1 pad 13: Vw_buff -> Net-(U1C-VIND-)
- U1 pad 14: Vw_buff -> /V_Syn_Drive
- U1 pad 2: V_Leak -> V_Syn1_Set
- U1 pad 3: /V_Leak_ref -> Net-(U1D-VINA+)
- U1 pad 6: Net-(U1A-VINB-) -> V_Syn2_Set
- U1 pad 7: Net-(U1A-VOUTB) -> V_Syn2_Set
- U1 pad 8: /Adapt_Kick_Drive -> Vw_buff
- U1 pad 9: /Adapt_Kick_Drive -> Vw_buff
- U2 pad 1: V_Leak_Ref_Max -> /Adapt_Kick_Drive
- U2 pad 14: /V_Syn_Drive -> /Adapt
- U2 pad 2: V_Leak_Ref_Max -> /Adapt_Kick_Drive
- U2 pad 3: VREF_2V048 -> AP
- U3 pad 1: V_Syn4_Set -> V_Leak
- U3 pad 13: V_Syn3_Set -> V_Syn4_Set
- U3 pad 14: V_Syn3_Set -> V_Syn4_Set
- U3 pad 2: V_Syn4_Set -> V_Leak
- U3 pad 3: Net-(U3D-VINA+) -> /V_Leak_ref
- U3 pad 5: Net-(U3A-VINB+) -> VREF_2V048
- U3 pad 6: V_Syn1_Set -> V_Leak_Ref_Max
- U3 pad 7: V_Syn1_Set -> V_Leak_Ref_Max
- U3 pad 8: V_Syn2_Set -> V_Syn3_Set
- U3 pad 9: V_Syn2_Set -> V_Syn3_Set
Routing:
- net VDD: track 14.6 -> 515.5 mm, vias 0 -> 28
- net Vm_Int: track 0.00 -> 228.9 mm, vias 0 -> 12
- net V_Syn_State: track 0.00 -> 181.6 mm, vias 0 -> 9
- net VREF_2V048: track 0.00 -> 166.7 mm, vias 0 -> 10
- net Vm_Ext: track 0.00 -> 147.6 mm, vias 0 -> 1
- net Vm_Display_In: track 0.00 -> 125.1 mm, vias 0 -> 2
- net Peak_Window: track 0.00 -> 104.3 mm, vias 0 -> 5
- net GNDREF: track 0.00 -> 93.8 mm, vias 0 -> 110
- net Reset_Window: track 0.00 -> 90.7 mm, vias 0 -> 5
- net Vsel: track 0.00 -> 79.7 mm, vias 0 -> 7
- net Vw_buff: track 0.00 -> 79.1 mm, vias 0 -> 2
- net /Reset_Injection_Drive: track 0.00 -> 77.6 mm, vias 0 -> 2
- net VREF_1V024: track 0.00 -> 71.2 mm, vias 0 -> 4
- net Vw: track 0.00 -> 69.6 mm, vias 0 -> 4
- net V_Boost: track 0.00 -> 66.7 mm, vias 0 -> 2
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- added copper zone on B.Cu, net GNDREF
- added copper zone on F.Cu, net GNDREF
Other:
- board size 119.2 x 79.8 mm -> 124.1 x 83 mm
- board text added: "Adapt"
- board text added: "C"
- board text added: "G"
- board text added: "V"
- board text added: "leak"
- board text added: "m"
- board text added: "syn"
- board text added: "τ"
