File: PCBs/Oscilloscope/SpikyOscilloscopce.kicad_sch (KiCad schematic)
At the start: 557 parts, among them J1 Channel 1, J10 SSD1963, J11 SparkFun SD/MMC Card Breakout, J2 Channel 5, J3 Rotary Encoder, J4 Channel 2, J5 Channel 6, J6 Channel 3, J7 Channel 7, J8 Channel 4, J9 Channel 8, K1 G5V-1, K2 G5V-1, K3 G5V-1, K4 G5V-1, K5 G5V-1, K6 G5V-1, K7 G5V-1, K8 G5V-1, Q1 FQP27P06, Q2 2N3904, Q3 2N3904, Q4 2N3904, Q5 2N3904, Q6 2N3904, Q7 2N3904, Q8 2N3904, Q9 2N3904, SW1 Power_Switch, SW10 SW_SPST, SW11 SW_Rotary_1x4_MP, SW12 SW_Rotary_1x4_MP, SW13 SW_Rotary_1x4_MP, SW14 SW_Rotary_1x4_MP, SW15 SW_Rotary_1x4_MP, SW16 SW_Rotary_1x4_MP, SW17 SW_Rotary_1x4_MP, SW18 SW_Rotary_1x4_MP, SW2 SW_Push, SW3 SW_SPST, SW4 SW_SPST, SW5 SW_SPST, SW6 SW_SPST, SW7 SW_SPST, SW8 SW_SPST, SW9 SW_SPST, U1 MCP3208, U10 MCP6022, U11 NE5532, U12 NE5532, U13 ULN2803A, U14 MCP3208, U15 NE5532, U16 NE5532, U17 AD780ANZ, U18 MCP23S17_SP, U19 ULN2803A, U2 MCP6004, U20 ESP32-S3-DevKitC, U22 TC7660HCPA, U23 MCP4922, U24 TC7660HCPA, U25 MCP4922, U26 TC7660HCPA, U27 MCP4922, U28 TC7660HCPA, U29 MCP4922, U3 NE5532, U4 NE5532, U5 MCP23S17_SP, U6 MCP6004, U7 NE5532, U8 NE5532, U9 LM2587T

Commit message: update Oscilloscope PCB
Parts:
- added C178: 10μF, Capacitor_THT:CP_Radial_D5.0mm_P2.50mm, symbol Device:C_US
- added C179: 100nF, Capacitor_THT:C_Disc_D4.7mm_W2.5mm_P5.00mm, symbol Device:C
- added U21: ADR420ABRZ, Package_SO:MSOP-8_3x3mm_P0.65mm, symbol Reference_Voltage:ADR420ARMZ
- J1, J2, J4, J5, J6, J7, J8, J9: DATASHEET https://atta.szlcsc.com/upload/public/pdf/source/20180120/C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 -> (none)
Connections:
- net +5VA: now also C178.1, C179.2, U21.2 (VIN)
- net ADC_Stim1: now also U14.1 (CH0); no longer U1.5 (CH4)
- net ADC_Stim2: now also U14.2 (CH1); no longer U1.6 (CH5)
- net ADC_Stim3: now also U14.3 (CH2); no longer U1.7 (CH6)
- net ADC_Stim4: now also U14.4 (CH3); no longer U1.8 (CH7)
- net ADC_Vm5: now also U1.5 (CH4); no longer U14.1 (CH0)
- net ADC_Vm6: now also U1.6 (CH5); no longer U14.2 (CH1)
- net ADC_Vm7: now also U1.7 (CH6); no longer U14.3 (CH2)
- net ADC_Vm8: now also U1.8 (CH7); no longer U14.4 (CH3)
- net GNDA: now also C178.2, C179.1, U21.4 (GND)
- net Vref_2V5: no longer C1.1, C2.2, C28.1, C29.2, U1.15 (Vref), U14.15 (Vref)
- new net Vref_2V048: C1.1, C2.2, C28.1, C29.2, U1.15 (Vref), U14.15 (Vref), U21.6 (OUT)
- no-connect marks 52 -> 53
Other:
- note removed: "Route VREF_2V5 short/wide to MCP3208.VREF and MCP4921.VREF; cap grounds land in ADC AGND region (Kelvin-ish)."
- note removed: "Single stitch: tie AGND ↔ DGND at one short, low-impedance point near the ADC/REF cluster."
- note removed: "analog and digital grounds are stitched once near the ADC/REF cluster"
- moved on the sheet: BT1, C1, C10, C100, C101, C102, C103, C104, C105, C106, C107, C108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

Commit message: update PCB for oscilloscope
Parts:
- removed BT1: Keystone 2477 (PC-pin 4×AA), Battery:BatteryHolder_Keystone_2479_3xAAA, symbol Device:Battery
- removed C1, C10, C102, C103, C104, C105, C15, C156, C157, C158, C161, C162, C165, C166, C169, C170, C173, C174, C177, C178, C19, C23, C28, C3, C31, C35, C37, C38, C40, C43, C48, C49, C50, C60, C78, C79, C80, C81, C9: 10μF, Capacitor_THT:CP_Radial_D5.0mm_P2.50mm, symbol Device:C_US
- removed C100, C106, C107, C108, C109, C11, C110, C111, C112, C113, C13, C14, C154, C155, C159, C160, C163, C164, C167, C168, C171, C172, C175, C176, C179, C2, C21, C22, C24, C26, C29, C30, C32, C33, C34, C39, C4, C41, C42, C44, C45, C46, C47, C5, C51, C61, C7, C8, C82, C83, C84, C85, C86, C87, C88, C89, C94, C96, C98: 100nF, Capacitor_THT:C_Disc_D4.7mm_W2.5mm_P5.00mm, symbol Device:C
- removed C101, C95, C97, C99: 10μF, Capacitor_THT:C_Rect_L7.0mm_W2.5mm_P5.00mm, symbol Device:C
- removed C114, C115, C116, C117, C118, C119, C120, C121, C70, C71, C72, C73, C74, C75, C76, C77: 2.2nF, Capacitor_THT:C_Disc_D3.8mm_W2.6mm_P2.50mm, symbol Device:C
- removed C12, C36, C6: 470μF, Capacitor_THT:CP_Radial_D8.0mm_P3.50mm, symbol Device:C_US
- removed C122, C123, C124, C125, C126, C127, C128, C129, C146, C147, C148, C149, C150, C151, C152, C153, C62, C63, C64, C65, C66, C67, C68, C69: 100pF, Capacitor_THT:C_Disc_D3.8mm_W2.6mm_P2.50mm, symbol Device:C
- removed C130, C131, C132, C133, C134, C135, C136, C137: 150pF, Capacitor_THT:C_Rect_L4.0mm_W2.5mm_P2.50mm, symbol Device:C
- removed C138, C139, C140, C141, C142, C143, C144, C145, C17, C18, C20, C25, C52, C53, C54, C55, C56, C57, C58, C59: 10nF, Capacitor_THT:C_Rect_L4.6mm_W2.0mm_P2.50mm_MKS02_FKP02, symbol Device:C
- removed C16: 220μF, Capacitor_THT:CP_Radial_D10.0mm_P5.00mm, symbol Device:C_US
- removed C27: 680μF, Capacitor_THT:CP_Radial_D10.0mm_P5.00mm, symbol Device:C_US
- removed C90, C91, C92, C93: 4.7μF, Capacitor_THT:CP_Radial_D5.0mm_P2.00mm, symbol Device:C_US
- removed D1: BZX55C10, Diode_THT:D_DO-35_SOD27_P7.62mm_Horizontal, symbol Device:D_Zener
- removed D10, D11, D12, D5, D6, D7, D8, D9: LED, Connector_JST:JST_XH_B2B-XH-A_1x02_P2.50mm_Vertical, symbol Device:LED
- removed D13, D14, D15, D16, D17, D18, D19, D20, D21, D22, D23, D24, D25, D26, D27, D28, D37, D38, D39, D40, D41, D42, D43, D44, D45, D46, D47, D48, D49, D50, D51, D52: BAT41, Diode_THT:D_DO-35_SOD27_P7.62mm_Horizontal, symbol Diode:BAT41
- removed D2: P6KE6.8CA, Diode_THT:D_DO-15_P10.16mm_Horizontal, symbol Diode:1N62xxCA
- removed D29, D30, D31, D32, D33, D34, D35, D36: 1N4148, Diode_THT:D_DO-35_SOD27_P7.62mm_Horizontal, symbol Diode:1N4148
- removed D3: 1N5819, Diode_THT:D_DO-41_SOD81_P7.62mm_Horizontal, symbol Device:D_Schottky
- removed D4: MBR360G, Diode_THT:D_DO-27_P12.70mm_Horizontal, symbol Device:D_Schottky
- removed D53, D54, D55, D56, D57, D58, D59, D60: P6kE6.8ca, Diode_THT:D_DO-15_P10.16mm_Horizontal, symbol Diode:1N62xxCA
- removed F1: MF-R185, Fuse:Fuse_Bourns_MF-RG300, symbol Device:Fuse
- removed F2: MF-R110, Fuse:Fuse_Bourns_MF-RG300, symbol Device:Fuse
- removed FB1, FB2, FB3, FB4: 2944666651, Ferrite_THT:LairdTech_28C0236-0JW-10, symbol Device:FerriteBead
- removed H1, H2, H3, H4: MountingHole, MountingHole:MountingHole_3mm, symbol Mechanical:MountingHole
- removed J1: Channel 1, Maxime:Spikeling Audio Jack 3.5mm, symbol PJ-320B1_PJ-320B-altium-import:root_0_PJ-320B贴片_
- removed J10: SSD1963, Connector_JST:JST_PUD_B40B-PUDSS_2x20_P2.00mm_Vertical, symbol Connector_Generic:Conn_02x20_Top_Bottom
- removed J11: SparkFun SD/MMC Card Breakout, Connector_JST:JST_XH_B13B-XH-A_1x13_P2.50mm_Vertical, symbol Connector:SD_Card_Receptacle
- removed J2: Channel 5, Maxime:Spikeling Audio Jack 3.5mm, symbol PJ-320B1_PJ-320B-altium-import:root_0_PJ-320B贴片_
- removed J4: Channel 2, Maxime:Spikeling Audio Jack 3.5mm, symbol PJ-320B1_PJ-320B-altium-import:root_0_PJ-320B贴片_
- removed J5: Channel 6, Maxime:Spikeling Audio Jack 3.5mm, symbol PJ-320B1_PJ-320B-altium-import:root_0_PJ-320B贴片_
- removed J6: Channel 3, Maxime:Spikeling Audio Jack 3.5mm, symbol PJ-320B1_PJ-320B-altium-import:root_0_PJ-320B贴片_
- removed J7: Channel 7, Maxime:Spikeling Audio Jack 3.5mm, symbol PJ-320B1_PJ-320B-altium-import:root_0_PJ-320B贴片_
- removed J8: Channel 4, Maxime:Spikeling Audio Jack 3.5mm, symbol PJ-320B1_PJ-320B-altium-import:root_0_PJ-320B贴片_
- removed J9: Channel 8, Maxime:Spikeling Audio Jack 3.5mm, symbol PJ-320B1_PJ-320B-altium-import:root_0_PJ-320B贴片_
- removed K1, K2, K3, K4, K5, K6, K7, K8: G5V-1, Relay_THT:Relay_SPDT_Omron_G5V-1, symbol Relay:G5V-1
- removed L1, L2: 100μH, Inductor_THT:L_Radial_D8.7mm_P5.00mm_Fastron_07HCP, symbol Device:L
- removed Q1: FQP27P06, Package_TO_SOT_THT:TO-220-3_Vertical, symbol Simulation_SPICE:PMOS
- removed Q2, Q3, Q4, Q5, Q6, Q7, Q8, Q9: 2N3904, Package_TO_SOT_THT:TO-92_Inline, symbol Transistor_BJT:2N3904
- removed R1, R14, R15, R210, R211, R212, R213, R214, R215, R216, R217: 10k, Resistor_THT:R_Axial_DIN0207_L6.3mm_D2.5mm_P7.62mm_Horizontal, symbol Device:R
- removed R10, R11: 10k (0.1%), Resistor_THT:R_Axial_DIN0207_L6.3mm_D2.5mm_P7.62mm_Horizontal, symbol Device:R
- removed R100, R101, R102, R103, R104, R105, R98, R99: 10k 1%, Resistor_THT:R_Axial_DIN0207_L6.3mm_D2.5mm_P7.62mm_Horizontal, symbol Device:R
- removed R106, R108, R110, R112, R114, R116, R118, R120: 20k 1%, Resistor_THT:R_Axial_DIN0207_L6.3mm_D2.5mm_P7.62mm_Horizontal, symbol Device:R
- removed R107, R109, R111, R113, R115, R117, R119, R121, R186, R187, R188, R189, R190, R191, R192, R193, R218, R219, R220, R221, R222, R223, R224, R225, R226, R227, R228, R229, R230, R231, R232, R233, R74, R75, R76, R77, R78, R79, R80, R81, R90, R91, R92, R93, R94, R95, R96, R97: 100, Resistor_THT:R_Axial_DIN0207_L6.3mm_D2.5mm_P7.62mm_Horizontal, symbol Device:R
- removed R12: 10k, Resistor_THT:R_Axial_DIN0207_L6.3mm_D2.5mm_P10.16mm_Horizontal, symbol Device:R
- removed R122, R123, R124, R125, R126, R127, R128, R129, R130, R131, R132, R133, R134, R135, R136, R137, R138, R139, R140, R141, R142, R143, R144, R145, R170, R171, R172, R173, R174, R175, R176, R177: 5k 1%, Resistor_THT:R_Axial_DIN0207_L6.3mm_D2.5mm_P7.62mm_Horizontal, symbol Device:R
- removed R13, R41, R42: 100k, Resistor_THT:R_Axial_DIN0207_L6.3mm_D2.5mm_P10.16mm_Horizontal, symbol Device:R
- removed R146, R147, R148, R149, R150, R151, R152, R153: 4.7k, Resistor_THT:R_Axial_DIN0207_L6.3mm_D2.5mm_P7.62mm_Horizontal, symbol Device:R
- removed R154, R155, R156, R157, R158, R159, R16, R160, R161, R2: 100k, Resistor_THT:R_Axial_DIN0207_L6.3mm_D2.5mm_P7.62mm_Horizontal, symbol Device:R
- removed R162, R163, R164, R165, R166, R167, R168, R169: 68, Resistor_THT:R_Axial_DIN0207_L6.3mm_D2.5mm_P7.62mm_Horizontal, symbol Device:R
- removed R17, R18, R19, R20, R21, R22, R23, R24, R4, R7, R8, R9: 220, Resistor_THT:R_Axial_DIN0207_L6.3mm_D2.5mm_P7.62mm_Horizontal, symbol Device:R
- removed R178, R179, R180, R181, R182, R183, R184, R185, R25, R26, R27, R28, R29, R30, R31, R32, R66, R67, R68, R69, R70, R71, R72, R73: 1k, Resistor_THT:R_Axial_DIN0207_L6.3mm_D2.5mm_P7.62mm_Horizontal, symbol Device:R
- removed R194, R195, R196, R197, R198, R199, R200, R201: 2k, Resistor_THT:R_Axial_DIN0207_L6.3mm_D2.5mm_P7.62mm_Horizontal, symbol Device:R
- removed R202, R203, R204, R205, R206, R207, R208, R209: 5k, Resistor_THT:R_Axial_DIN0207_L6.3mm_D2.5mm_P7.62mm_Horizontal, symbol Device:R
- removed R3: 3k, Resistor_THT:R_Axial_DIN0207_L6.3mm_D2.5mm_P7.62mm_Horizontal, symbol Device:R
- removed R33, R40, R63: 47k, Resistor_THT:R_Axial_DIN0207_L6.3mm_D2.5mm_P7.62mm_Horizontal, symbol Device:R
- removed R34, R35, R36, R37, R38, R39, R43, R44, R45, R46, R47, R48, R49, R50, R51, R52, R53, R54, R55, R56, R57, R58, R59, R60, R61, R62, R64, R65: 47, Resistor_THT:R_Axial_DIN0207_L6.3mm_D2.5mm_P10.16mm_Horizontal, symbol Device:R
- removed R5: 3.4k, Resistor_THT:R_Axial_DIN0207_L6.3mm_D2.5mm_P7.62mm_Horizontal, symbol Device:R
- removed R6: 1.1k, Resistor_THT:R_Axial_DIN0207_L6.3mm_D2.5mm_P7.62mm_Horizontal, symbol Device:R
- removed R82, R83, R84, R85, R86, R87, R88, R89: 22, Resistor_THT:R_Axial_DIN0207_L6.3mm_D2.5mm_P7.62mm_Horizontal, symbol Device:R
- removed SW1: Power_Switch, Connector_JST:JST_XH_B3B-XH-A_1x03_P2.50mm_Vertical, symbol Switch:SW_SPDT
- removed SW10, SW3, SW4, SW5, SW6, SW7, SW8, SW9: SW_SPST, Connector_JST:JST_XH_B2B-XH-A_1x02_P2.50mm_Vertical, symbol Switch:SW_SPST
- removed SW11, SW12, SW13, SW14, SW15, SW16, SW17, SW18: SW_Rotary_1x4_MP, Connector_JST:JST_XH_B5B-XH-A_1x05_P2.50mm_Vertical, symbol Switch:SW_Rotary_1x4_MP
- removed SW2: SW_Push, Connector_JST:JST_XH_B2B-XH-A_1x02_P2.50mm_Vertical, symbol Switch:SW_Push
- removed U1, U14: MCP3208, Package_DIP:DIP-16_W7.62mm, symbol Analog_ADC:MCP3208
- removed U10: MCP6022, Package_DIP:DIP-8_W7.62mm, symbol Amplifier_Operational:MCP6022
- removed U11, U12, U15, U16, U3, U4, U7, U8: NE5532, Package_DIP:DIP-8_W7.62mm, symbol Amplifier_Operational:NE5532
- removed U13, U19: ULN2803A, Package_DIP:DIP-18_W7.62mm, symbol Transistor_Array:ULN2803A
- removed U17: AD780ANZ, Package_DIP:DIP-8_W7.62mm, symbol Reference_Voltage:REF02CP
- removed U18, U5: MCP23S17_SP, Package_DIP:DIP-28_W7.62mm, symbol Interface_Expansion:MCP23S17_SP
- removed U2, U6: MCP6004, Package_DIP:DIP-14_W7.62mm, symbol Amplifier_Operational:MCP6004
- removed U20: ESP32-S3-DevKitC, PCM_Espressif:ESP32-S3-DevKitC, symbol PCM_Espressif:ESP32-S3-DevKitC
- removed U21: ADR420ABRZ, Package_SO:MSOP-8_3x3mm_P0.65mm, symbol Reference_Voltage:ADR420ARMZ
- removed U22, U24, U26, U28: TC7660HCPA, Package_DIP:DIP-8_W7.62mm_Socket, symbol Regulator_SwitchedCapacitor:ICL7660
- removed U23, U25, U27, U29: MCP4922, Package_DIP:DIP-14_W7.62mm, symbol Analog_DAC:MCP4922
- removed U9: LM2587T, Package_TO_SOT_THT:TO-220-5_Vertical, symbol Regulator_Switching:LM2575-3.3BT
- added C1, C2, C34, C37, C38, C39, C7, C9: 2.2nF, C0603, symbol 1_P1-altium-import:root_0_C1608C0G1H222JT000N_
- added C10, C11, C17, C18, C20, C25, C28, C29: 22nF, C0603, symbol 1_P1-altium-import:root_0_0603B223K500NT_
- added C101, C126, C128, C134, C144, C145, C160, C41, C50, C52: 10uF, JLCPCB:C_0805, symbol CL21A106KBYQNNE1_CL21A106KBYQNNE-altium-import:root_0_CL21A106KBYQNNE_
- added C102, C104, C116, C124, C127, C129, C135, C138, C146, C147, C152, C153, C161, C42, C51, C53, C84, C85, C86, C90, C91, C92, C94, C96: 100nF, JLCPCB:C_0603, symbol CL10B104KB8NNNC1_CL10B104KB8NNNC (2)-altium-import:root_0_CL10B104KB8NNNC_
- added C103: 4.7nF, JLCPCB:C_0603, symbol 0603B472K500NT1_0603B472K500NT-altium-import:root_0_0603B472K500NT_
- added C105, C136, C137, C148, C149, C150, C151, C49: 4.7nF, C0603, symbol 1_P1-altium-import:root_0_CC0603KRX7R9BB472_
- added C106, C139, C158, C159, C83, C87, C93: 1uF, JLCPCB:C_0805, symbol CL21B105KBFNNNE1_CL21B105KBFNNNE-altium-import:root_0_CL21B105KBFNNNE_
- added C113, C114, C132, C133, C140, C141, C142, C143, C162, C163, C164, C165, C166, C167, C168, C169, C172, C173: 10nF, JLCPCB:C_0603, symbol CC0603KRX7R9BB1031_CC0603KRX7R9BB103 (1)-altium-import:root_0_CC0603KRX7R9BB103_
- added C23: 1nF, JLCPCB:C_0603, symbol CC0603KRX7R9BB1021_CC0603KRX7R9BB102 (1)-altium-import:root_0_CC0603KRX7R9BB102_
- added C3: 220uF, CAP-SMD_BD6.3-L6.6-W6.6-FD, symbol 1_P1-altium-import:root_0_RST220UF10V018_
- added C4: 10uF, C1206, symbol 1_P1-altium-import:root_0_1206B106K100NT_
- added C40, C82, C95: 10uF, JLCPCB:C_1206, symbol TCC1206X7R106K250HT1_TCC1206X7R106K250HT-altium-import:root_0_TCC1206X7R106K250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
- added C44, C47, C48: 1uF, C0402, symbol CL05A105KA5NQNC1_CL05A105KA5NQNC-altium-import:root_0_CL05A105KA5NQNC_
- added C5: 1uF, C0805, symbol 1_P1-altium-import:root_0_0805B105K500NT_C215803_
- added C6: 100nF, C0603, symbol 1_P1-altium-import:root_0_C0603C104J5RAC7867_C490602_
- added C88: 22uF, JLCPCB:C_1206, symbol CL31A226KAHNNNE1_CL31A226KAHNNNE-altium-import:root_0_CL31A226KAHNNNE_
- added C89: 4.7uF, JLCPCB:C_0805, symbol CS2012X7R475K350NRE1_CS2012X7R475K350NRE-altium-import:root_0_CS2012X7R475K350N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
- added D29: SMF6.0A, JLCPCB:D_SOD-123FL, symbol SMF6.0A_C1782601_SMF6.0A_C178260-altium-import:root_0_SMF6.0A_C178260_
- added D31, D32, D49, D50, D51, D52, D53, D54, D55, D56: Red, JLCPCB:D_0603, symbol PCM_JLCPCB-Diodes:LED,0603,Red
- added D33, D35, D37, D38, D41, D42, D43, D44: BAT54S, JLCPCB:SOT-23-3_L2.9-W1.3-P1.90-LS2.4-BR, symbol BAT54S_C9164251_BAT54S_C916425 (1)-altium-import:root_0_BAT54S_C916425_
- added D34, D36, D39, D40, D45, D46, D47, D48: TPD2E2U06DCKR, Maxime:SC-70-3_L2.0-W1.3-P0.65-LS2.1-BL, symbol Spikeling_V2.5-altium-import:root_0_TPD2E2U06DCKR_
- added H10, H11, H12, H5, H6, H7, H8, H9: MountingHole_Pad, MountingHole:MountingHole_3.2mm_M3_DIN965_Pad, symbol Mechanical:MountingHole_Pad
- added J1: Conn_02x20_Top_Bottom, Connector_PinHeader_2.54mm:PinHeader_2x20_P2.54mm_Vertical, symbol Connector_Generic:Conn_02x20_Top_Bottom
- added J12: Connector, USB-TYPE-C-16P, JLCPCB:TYPE-C-SMD_HX-TYPE-C-16PIN, symbol PCM_JLCPCB-Extended:Connector, USB-TYPE-C-16P
- added J13: Channel 1, Maxime:AUDIO-SMD_PJ-320B, symbol PJ-320B1_PJ-320B-altium-import:root_0_PJ-320B贴片_
- added J14: Channel 2, Maxime:AUDIO-SMD_PJ-320B, symbol PJ-320B1_PJ-320B-altium-import:root_0_PJ-320B贴片_
- added J15: Channel 3, Maxime:AUDIO-SMD_PJ-320B, symbol PJ-320B1_PJ-320B-altium-import:root_0_PJ-320B贴片_
- added J16: Channel 4, Maxime:AUDIO-SMD_PJ-320B, symbol PJ-320B1_PJ-320B-altium-import:root_0_PJ-320B贴片_
- added J17: Channel 5, Maxime:AUDIO-SMD_PJ-320B, symbol PJ-320B1_PJ-320B-altium-import:root_0_PJ-320B贴片_
- added J18: Channel 6, Maxime:AUDIO-SMD_PJ-320B, symbol PJ-320B1_PJ-320B-altium-import:root_0_PJ-320B贴片_
- added J19: Channel 7, Maxime:AUDIO-SMD_PJ-320B, symbol PJ-320B1_PJ-320B-altium-import:root_0_PJ-320B贴片_
- added J20: Channel 8, Maxime:AUDIO-SMD_PJ-320B, symbol PJ-320B1_PJ-320B-altium-import:root_0_PJ-320B贴片_
- added L4: MPZ2012S601, JLCPCB:L_0805, symbol SpikyOscilloscopce-altium-import:root_0_MPZ2012S601AT000_
- added L6: 2.2uH, Maxime:IND-SMD_L3.0-W3.0_XFL3012, symbol SpikyOscilloscopce-altium-import:root_0_XFL3012-222MEC_
- added R1: 249kΩ, R0603, symbol 1_P1-altium-import:root_0_0603WAF2493T5E_
- added R10: 1Ω, R0603, symbol 1_P1-altium-import:root_0_AC0603JR-071RL_
- added R106, R107: 22Ω, JLCPCB:R_0603, symbol 0603WAF220JT5E1_0603WAF220JT5E-altium-import:root_0_0603WAF220JT5E_
- added R111, R112, R113, R117, R118, R119, R120, R121, R122, R123, R124, R125, R126, R128, R163, R164, R165, R166, R167, R168, R169, R170, R171, R174, R175, R176, R186, R187: 47Ω, JLCPCB:R_0603, symbol 0603WAF470JT5E1_0603WAF470JT5E-altium-import:root_0_0603WAF470JT5E_
- added R114, R115, R161, R189, R190, R191, R192, R193, R194, R195, R196, R197, R213, R214, R215, R222, R223, R224, R225, R226, R227, R228, R229, R230, R231, R232, R233, R234, R250, R251, R252, R253: 10kΩ, JLCPCB:R_0603, symbol FRC0603F1002TS1_FRC0603F1002TS-altium-import:root_0_FRC0603F1002TS_
- added R116, R127, R177, R180, R181, R205, R206, R207, R208, R209, R210, R211, R212, R43, R44, R45, R46: 100Ω, JLCPCB:R_0603, symbol RC0603FR-07100RL1_RC0603FR-07100RL (4)-altium-import:root_0_RC0603FR-07100RL_
- added R13, R14, R15, R16, R17, R18, R19, R20, R21, R22, R23, R24, R25, R26, R27, R28: 4.7kΩ, R0603, symbol 1_P1-altium-import:root_0_0603WAF4701T5E_
- added R136, R139, R142, R143, R148, R149, R150, R151, R90, R91: 5.1kΩ, JLCPCB:R_0603, symbol 0603WAF5101T5E1_0603WAF5101T5E-altium-import:root_0_0603WAF5101T5E_
- added R137, R138, R140, R141, R144, R145, R146, R147, R152, R153, R154, R155, R156, R157, R158, R159, R160, R172, R173, R184, R185, R188, R199, R200, R201, R202, R203, R204: 100kΩ, JLCPCB:R_0603, symbol RC0603FR-07100KL1_RC0603FR-07100KL (1)-altium-import:root_0_RC0603FR-07100KL_
- added R2: 900kΩ, R0805, symbol 1_P1-altium-import:root_0_0805W8F9003T5E_
- added R216, R217, R218, R219, R220, R221, R235, R236, R237, R238, R239, R240, R241, R242, R243, R244, R245, R246, R247, R248, R249: 1kΩ, JLCPCB:R_0603, symbol FRC0603F1001TS1_FRC0603F1001TS (2)-altium-import:root_0_FRC0603F1001TS_
- added R3: 820Ω, R0603, symbol 1_P1-altium-import:root_0_RC0603FR-07820RL_
- added R82: 1MΩ, JLCPCB:R_0603, symbol RC0603FR-071ML1_RC0603FR-071ML (1)-altium-import:root_0_RC0603FR-071ML_
- added R89: 0Ω, JLCPCB:R_0603, symbol 0603WAF0000T5E1_0603WAF0000T5E-altium-import:root_0_0603WAF0000T5E_
- added SW12: SKHHLVA010, Maxime:KEY-TH_4P-L7.5-W6.8-P4.50-LS7.2, symbol SKHHLVA0101_SKHHLVA010-altium-import:root_0_SKHHLVA010_
- added SW13: Tactile Button, 160gf, JLCPCB:SW_TS-1088-AR02016, symbol PCM_JLCPCB-Connectors_Buttons:Tactile Button, 160gf, 12V, 50mA, 4.0mm
- added SW14: Stimulus 1 Arm / Enable, Maxime:maxi_DPDT_Angled, symbol Switch:SW_Push_DPDT
- added SW15: Stimulus 2 Arm / Enable, Maxime:maxi_DPDT_Angled, symbol Switch:SW_Push_DPDT
- added SW16: Stimulus 3 Arm / Enable, Maxime:maxi_DPDT_Angled, symbol Switch:SW_Push_DPDT
- added SW17: Stimulus 4 Arm / Enable, Maxime:maxi_DPDT_Angled, symbol Switch:SW_Push_DPDT
- added SW18: Stimulus 5 Arm / Enable, Maxime:maxi_DPDT_Angled, symbol Switch:SW_Push_DPDT
- added SW19: Stimulus 7 Arm / Enable, Maxime:maxi_DPDT_Angled, symbol Switch:SW_Push_DPDT
- added SW20: Stimulus 6 Arm / Enable, Maxime:maxi_DPDT_Angled, symbol Switch:SW_Push_DPDT
- added SW21: Stimulus 8 Arm / Enable, Maxime:maxi_DPDT_Angled, symbol Switch:SW_Push_DPDT
- added TP1, TP2, TP3, TP4, TP6, TP7: TestPoint, TestPoint:TestPoint_Pad_D2.0mm, symbol Connector:TestPoint
- added TV1: SRV05-4-P-T7, JLCPCB:SOT-23-6_L2.9-W1.6-P0.95-LS2.8-BR, symbol SRV05-4-P-T71_SRV05-4-P-T7-altium-import:root_0_SRV05-4-P-T7_C85364_
- added U1: MCP23S17T-E/SO, SOIC-28_L17.9-W7.5-P1.27-LS10.3-BL, symbol 1_P1-altium-import:root_0_MCP23S17T-E/SO_
- added U13, U5: MCP6004T-I/SL, SOIC-14_L8.7-W3.9-P1.27-LS6.0-BL, symbol 1_P1-altium-import:root_0_MCP6004T-I/SL_
- added U14, U17, U20, U7: MCP4922-E/SL, SOIC-14_L8.7-W3.9-P1.27-LS6.0-BL, symbol 1_P1-altium-import:root_0_MCP4922-E/SL_
- added U15: TPS7A2033PDBVR, Maxime:SOT-23-5_L2.9-W1.6-P0.95-LS2.8-BR, symbol SpikyOscilloscopce-altium-import:root_0_TPS7A2033PDBVR_
- added U16: TPS62162DSGR, Maxime:WSON-8_L2.0-W2.0-P0.50-TL-EP, symbol SpikyOscilloscopce-altium-import:root_0_TPS62162DSGR_
- added U2: TPS259530DSGR, WSON-8_L2.0-W2.0-P0.50-TL-EP, symbol 1_P1-altium-import:root_0_TPS259530DSGR_
- added U25: ESP32-S3-WROOM-1-N4, Maxime:WIFIM-SMD_ESP32-S3-WROOM-1-N8, symbol ESP32-S3-WROOM-1-N41_ESP32-S3-WROOM-1-N4-altium-import:root_0_ESP32-S3-WROOM-1-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
- added U26: REF5020AIDR, SOIC-8_L4.9-W3.9-P1.27-LS6.0-BL, symbol 1_P1-altium-import:root_0_REF5020AIDR_
- added U27: MCP3208-BI/SL, SOIC-16_L9.9-W3.9-P1.27-LS6.0-BL, symbol 1_P1-altium-import:root_0_MCP3208-BI/SL_
- added U29, U33, U34, U35: TS5A23166DCUR, VSON8_L2.0-W2.3-P0.50-LS3.1-BL, symbol 1_P1-altium-import:root_0_TS5A23166DCUR_
- added U3: TUSB320LAIRWBR, X2QFN-12_L1.6-W1.6-P0.40-TL, symbol 1_P1-altium-import:root_0_TUSB320LAIRWBR_
Connections:
- net +3.3V: now also C101.1, C102.1, C160.2, C161.2, C88.2, C90.2, C92.2, D49.2, D50.2, D51.2, D52.2, D53.2, D54.2, D55.2, D56.2, L6.2, R114.2, R115.2, R161.1, R189.2, R190.2, R191.2, R192.2, R193.2, R194.2, R195.2, R196.2, R197.2, R213.1, R214.1, R215.1, R222.1, R223.1, R224.1, R225.1, R226.1, R227.1, R228.1, R229.1, R230.1, R231.1, R232.1, R233.1, R250.1, R251.1, R252.1, R253.1, R91.2, TP2.1, U1.9 (VDD), U16.6 (VOS), U25.2 (3V3), U3.12 (VDD)
- net +3.3VA: now also C106.1, C116.2, C126.1, C127.1, C134.2, C135.2, C138.2, C139.1, C144.2, C145.2, C146.2, C147.2, C152.2, C153.2, C158.1, C159.1, C41.2, C42.2, C50.2, C51.2, C52.2, C53.2, C86.2, C89.2, D33.2 (K), D35.2 (K), D37.2 (K), D38.2 (K), D41.2 (K), D42.2 (K), D43.2 (K), D44.2 (K), R90.2, TP3.1, U13.4 (VDD), U14.1 (VDD), U15.5 (OUT), U17.1 (VDD), U20.1 (VDD), U27.16 (VDD), U29.8 (V+), U33.8 (V+), U34.8 (V+), U35.8 (V+), U5.4 (VDD), U7.1 (VDD)
- net +5VA: now also C124.2, C48.1, C83.2, C85.2, C93.2, C94.2, C95.1, L4.2, TP1.1, U15.1 (IN), U15.3 (EN), U26.2 (VIN)
- net ADC_Vm1: now also C1.1, R205.1, U27.1 (CH0)
- net ADC_Vm2: now also C2.1, R206.1, U27.2 (CH1)
- net ADC_Vm3: now also C9.1, R208.1, U27.3 (CH2)
- net ADC_Vm4: now also C7.1, R207.1, U27.4 (CH3)
- net ADC_Vm5: now also C34.1, R209.1, U27.5 (CH4)
- net ADC_Vm6: now also C37.1, R210.1, U27.6 (CH5)
- net ADC_Vm7: now also C39.1, R212.1, U27.7 (CH6)
- net ADC_Vm8: now also C38.1, R211.1, U27.8 (CH7)
- net CS_MCP4922_1/2: now also R119.1, U7.3 (CS#)
- net CS_MCP4922_3/4: now also R120.1, U17.3 (CS#)
- net CS_MCP4922_5/6: now also R121.1, U14.3 (CS#)
- net CS_MCP4922_7/8: now also R122.1, U20.3 (CS#)
- net GNDA: now also C1.2, C10.2, C105.1, C106.2, C11.2, C113.2, C114.2, C116.1, C124.1, C126.2, C127.2, C128.1, C129.1, C132.2, C133.2, C134.1, C135.1, C136.2, C137.1, C138.1, C139.2, C140.2, C141.2, C142.2, C143.2, C144.1, C145.1, C146.1, C147.1, C148.2, C149.1, C150.2, C151.1, C152.1, C153.1, C158.2, C159.2, C17.2, C18.2, C2.2, C20.2, C25.2, C28.2, C29.2, C34.2, C37.2, C38.2, C39.2, C40.2, C41.1, C42.1, C44.1, C47.1, C48.2, C49.2, C50.1, C51.1, C52.1, C53.1, C7.2, C83.1, C85.1, C86.1, C87.1, C89.1, C9.2, C93.1, C94.1, C95.2, C96.1, D31.1, D33.1 (A), D34.3 (GND), D35.1 (A), D36.3 (GND), D37.1 (A), D38.1 (A), D39.3 (GND), D40.3 (GND), D41.1 (A), D42.1 (A), D43.1 (A), D44.1 (A), D45.3 (GND), D46.3 (GND), D47.3 (GND), D48.3 (GND), J13.S, J14.S, J15.S, J16.S, J17.S, J18.S, J19.S, J20.S, R137.2, R138.1, R140.1, R141.2, R144.1, R145.1, R146.2, R147.2, R152.1, R153.1, R154.1, R155.1, R156.2, R157.2, R158.2, R159.2, R184.2, R185.2, R188.2, R200.2, R201.2, R202.2, R203.2, R204.2, R89.1, U13.11 (VSS), U14.12 (VSS), U15.2 (GND), U17.12 (VSS), U20.12 (VSS), U26.4 (GND), U27.14 (AGND), U29.4 (GND), U33.4 (GND), U34.4 (GND), U35.4 (GND), U5.11 (VSS), U7.12 (VSS)
- net GNDD: now also C101.2, C102.2, C103.2, C104.2, C160.1, C161.1, C162.1, C163.1, C164.1, C165.1, C166.1, C167.1, C168.1, C169.1, C172.1, C173.1, C23.2, C3.1, C4.2, C5.1, C6.1, C82.1, C84.1, C88.1, C90.1, C91.1, C92.1, D29.2 (A), D32.1, J1.1 (Pin_1), J12.A12B1 (GND), J12.B12A1 (GND), R160.1, R172.1, R173.1, R199.1, R234.1, R3.2, R82.2, R89.2, SW12.2, SW13.2 (B), SW14.3 (C), SW15.3 (C), SW16.3 (C), SW17.3 (C), SW18.3 (C), SW19.3 (C), SW20.3 (C), SW21.3 (C), TV1.2, U1.10 (VSS), U1.15 (A0), U1.16 (A1), U1.17 (A2), U16.1 (PGND), U16.4 (AGND), U16.5 (FB), U16.9 (EP), U2.8 (GND), U2.9 (EP), U25.1 (GND), U25.40 (GND), U25.41 (GND), U27.9 (DGND), U3.10 (GND), U3.11 (EN_N), U3.3 (PORT)
- net Rot_OutA: now also R217.1
- net Rot_OutB: now also R218.1
- net Rot_Switch: now also R216.1
- net SD_CS: now also J1.38 (Pin_38), R125.1
- net Vref_2V048: now also C113.1, C114.1, C128.2, C129.2, C132.1, C133.1, C140.1, C141.1, C142.1, C143.1, C47.2, R10.1, TP4.1, U14.11 (VREFB), U14.13 (VREFA), U17.11 (VREFB), U17.13 (VREFA), U20.11 (VREFB), U20.13 (VREFA), U26.6 (VOUT), U27.15 (VREF), U7.11 (VREFB), U7.13 (VREFA)
- new net: R150.1, R241.2, SW20.2 (B)
- new net: D55.1, R150.2
- new net: R117.2, R223.2, U25.39 (IO1)
- new net: D40.1 (IO1), J16.R, R147.1, R245.2
- new net: D34.1 (IO1), J13.R, R137.1, R221.2
- new net: D34.2 (IO2), J13.T, R13.2, R138.2
- new net: R165.1, U25.23 (IO21)
- new net: R148.1, R239.2, SW18.2 (B)
- new net: R220.1, R234.2, U25.33 (IO40)
- new net: R151.1, R242.2, SW21.2 (B)
- new net: R124.2, R253.2, U25.36 (RXD0)
- new net: D54.1, R149.2
- new net: R211.2, U13.13 (VIND-), U13.14 (VOUTD)
- new net: D56.1, R151.2
- new net: C173.2, R213.2, R217.2, U25.17 (IO9)
- new net: R206.2, U5.6 (VINB-), U5.7 (VOUTB)
- new net: R125.2, R225.2, U25.34 (IO41)
- new net: R176.2, R229.2, U25.8 (IO15)
- new net: R46.1, U20.14 (VOUTA)
- new net: R44.1, U17.14 (VOUTA)
- new net: R128.2, R250.2, U25.22 (IO14)
- new net: R170.1, R173.2, U25.26 (IO45)
- new net: R207.2, U5.13 (VIND-), U5.14 (VOUTD)
- new net: R212.2, U13.8 (VOUTC), U13.9 (VINC-)
- new net: R201.1, R27.1, U35.7 (IN1)
- new net: R2.2, U3.4 (VBUS_DET)
- new net: R142.1, R237.2, SW16.2 (B)
- new net: D51.1, R142.2
- new net: D45.1 (IO1), J17.R, R156.1, R246.2
- new net: D47.1 (IO1), J19.R, R158.1, R248.2
- new net: L6.1, U16.7 (SW)
- new net: R126.2, R252.2, U25.15 (IO3)
- new net: D46.1 (IO1), J18.R, R157.1, R247.2
- new net: D46.2 (IO2), J18.T, R153.2, R17.2
- new net: R203.1, R22.1, U33.7 (IN1)
- new net: D36.1 (IO1), J14.R, R141.1, R243.2
- new net: D36.2 (IO2), J14.T, R14.2, R140.2
- new net: R127.1, U7.10 (VOUTB)
- new net: R111.2, R227.2, U25.19 (IO11)
- new net: R171.1, R172.2, U25.16 (IO46)
- new net: D53.1, R148.2
- new net: R175.1, U25.24 (IO47)
- new net: R136.1, R235.2, SW14.2 (B)
- new net: D49.1, R136.2
- new net: R189.1, U1.18 (RESET#)
- new net: C172.2, R214.2, R218.2, U25.18 (IO10)
- new net: D50.1, R139.2
- new net: D47.2 (IO2), J19.T, R154.2, R18.2
- new net: R208.2, U5.8 (VOUTC), U5.9 (VINC-)
- new net: R149.1, R240.2, SW19.2 (B)
- new net: R184.1, R24.2, U29.3 (IN2)
- new net: R204.1, R21.1, U29.7 (IN1)
- new net: D39.1 (IO1), J15.R, R146.1, R244.2
- new net: D39.2 (IO2), J15.T, R144.2, R20.2
- new net: R120.2, R232.2, U25.5 (IO5)
- new net: D48.2 (IO2), J20.T, R155.2, R19.2
- new net: R119.2, R233.2, U25.4 (IO4)
- new net: R185.1, R23.2, U33.3 (IN2)
- new net: R174.1, U25.25 (IO48)
- new net: R106.2, U25.13 (IO19)
- new net: R177.1, U17.10 (VOUTB)
- new net: D45.2 (IO2), J17.T, R152.2, R16.2
- new net: D48.1 (IO1), J20.R, R159.1, R249.2
- new net: R187.2, R222.2, U25.12 (IO8)
- new net: R209.2, U13.1 (VOUTA), U13.2 (VINA-)
- new net: D31.2, R90.1
- new net: C91.2, U2.1 (dVdt)
- new net: R1.2, R160.2, U2.2 (EN/UVLO)
- new net: R3.1, U2.7 (ILM)
- new net: R180.1, U14.10 (VOUTB)
- new net: R205.2, U5.1 (VOUTA), U5.2 (VINA-)
- new net: R164.2, U25.11 (IO18)
- new net: R186.2, R228.2, U25.9 (IO16)
- new net: R121.2, R231.2, U25.6 (IO6)
- new net: R123.2, R251.2, U25.37 (TXD0)
- new net: R188.1, R26.2, U34.3 (IN2)
- new net: R181.1, U20.10 (VOUTB)
- new net: C40.1, R10.2
- new net: R139.1, R236.2, SW15.2 (B)
- new net: D52.1, R143.2
- new net: R219.1, U25.32 (IO39)
- new net: J1.6 (Pin_6), R161.2
- new net: R116.2, SW13.1 (A)
- new net: R215.2, R216.2, U25.35 (IO42)
- new net: R169.1, U25.31 (IO38)
- new net: R166.1, U25.28 (IO35)
- new net: R143.1, R238.2, SW17.2 (B)
- new net: C44.2, U26.5 (TRIM/NR)
- new net: R122.2, R230.2, U25.7 (IO7)
- new net: R45.1, U14.14 (VOUTA)
- new net: R167.1, U25.29 (IO36)
- new net: D40.2 (IO2), J16.T, R145.2, R15.2
- new net: R118.2, R224.2, U25.38 (IO2)
- new net: R202.1, R25.1, U34.7 (IN1)
- new net: R163.2, R199.2, U25.10 (IO17)
- new net: R107.2, U25.14 (IO20)
- new net: R112.2, U25.20 (IO12)
- new net: R113.1, R226.2, U25.21 (IO13)
- new net: R168.1, U25.30 (IO37)
- new net: R210.2, U13.6 (VINB-), U13.7 (VOUTB)
- new net: D32.2, R91.1
- new net: R200.1, R28.2, U35.3 (IN2)
- new net: R43.1, U7.14 (VOUTA)
- new net +5V_DSYS: TP6.1
- new net +5V_SYS: C3.2, C4.1, C5.2, C6.2, C82.2, C84.2, J1.18 (Pin_18), L4.1, U16.2 (VIN), U16.3 (EN), U2.5 (OUT)
- new net Boot: C103.1, R115.1, R116.1, U25.27 (IO0)
- new net CC1: J12.A5 (CC1), TV1.4, U3.1 (CC1)
- new net CC2: J12.B5 (CC2), TV1.6, U3.2 (CC2)
- new net CHASSIS: C23.1, H10.1, H11.1, H12.1, H5.1, H6.1, H7.1, H8.1, H9.1, J12.S1 (SHIELD), R82.1, SW12.3, SW12.4
- new net CS_MCP23S17: R186.1, U1.11 (CS#)
- new net CS_MCP3208: R176.1, U27.10 (CS#/SHDN)
- new net DAC_LDAC_N: R187.1, U14.8 (LDAC#), U17.8 (LDAC#), U20.8 (LDAC#), U7.8 (LDAC#)
- new net DAC_SHDN_N: R220.2, U14.9 (SHDN#), U17.9 (SHDN#), U20.9 (SHDN#), U7.9 (SHDN#)
- new net EFUSE_FLT_N: R126.1, U2.6 (FLT#)
- new net En: C104.1, R114.1, SW12.1, U25.3 (EN)
- new net LCD_BL: J1.19 (Pin_19), R163.1
- new net LCD_CS: J1.15 (Pin_15), R117.1
- new net LCD_DB0: J1.21 (Pin_21), R164.1
- new net LCD_DB1: J1.22 (Pin_22), R165.2
- new net LCD_DB2: J1.23 (Pin_23), R166.2
- new net LCD_DB3: J1.24 (Pin_24), R167.2
- new net LCD_DB4: J1.25 (Pin_25), R168.2
- new net LCD_DB5: J1.26 (Pin_26), R169.2
- new net LCD_DB6: J1.27 (Pin_27), R170.2
- new net LCD_DB7: J1.28 (Pin_28), R171.2
- new net LCD_RS: J1.4 (Pin_4), R174.2
- new net LCD_Reset: J1.17 (Pin_17), R118.1
- new net LCD_WR: J1.5 (Pin_5), R175.2
- new net SPI_MISO: J1.33 (Pin_33), J1.35 (Pin_35), R113.2, U1.14 (SO), U27.12 (DOUT)
- new net SPI_MOSI: J1.31 (Pin_31), J1.37 (Pin_37), R111.1, U1.13 (SI), U14.5 (SDI), U17.5 (SDI), U20.5 (SDI), U27.11 (DIN), U7.5 (SDI)
- new net SPI_SCK: J1.29 (Pin_29), J1.36 (Pin_36), R112.1, U1.12 (SCK), U14.4 (SCK), U17.4 (SCK), U20.4 (SCK), U27.13 (CLK), U7.4 (SCK)
- new net STIM1_ARM_SENSE_N: C162.2, R190.1, R235.1, U1.21 (GPA0)
- new net STIM1_EN_CMD: SW14.5 (B), U1.1 (GPB0)
- new net STIM2_ARM_SENSE_N: C163.2, R191.1, R236.1, U1.22 (GPA1)
- new net STIM2_EN_CMD: SW15.5 (B), U1.2 (GPB1)
- new net STIM3_ARM_SENSE_N: C164.2, R192.1, R237.1, U1.23 (GPA2)
- new net STIM3_EN_CMD: SW16.5 (B), U1.3 (GPB2)
- new net STIM4_ARM_SENSE_N: C165.2, R193.1, R238.1, U1.24 (GPA3)
- new net STIM4_EN_CMD: SW17.5 (B), U1.4 (GPB3)
- new net STIM5_ARM_SENSE_N: C166.2, R194.1, R239.1, U1.25 (GPA4)
- new net STIM5_EN_CMD: SW18.5 (B), U1.5 (GPB4)
- new net STIM6_ARM_SENSE_N: C168.2, R196.1, R241.1, U1.26 (GPA5)
- new net STIM6_EN_CMD: SW20.5 (B), U1.6 (GPB5)
- new net STIM7_ARM_SENSE_N: C167.2, R195.1, R240.1, U1.27 (GPA6)
- new net STIM7_EN_CMD: SW19.5 (B), U1.7 (GPB6)
- new net STIM8_ARM_SENSE_N: C169.2, R197.1, R242.1, U1.28 (GPA7)
- new net STIM8_EN_CMD: SW21.5 (B), U1.8 (GPB7)
- new net Stim1_Enable: R21.2, SW14.6 (C)
- new net Stim1_Filtered: C49.1, R43.2, U29.1 (NO1)
- new net Stim1_Output: R221.1, U29.2 (COM1)
- new net Stim2_Enable: R24.1, SW15.6 (C)
- new net Stim2_Filtered: C105.2, R127.2, U29.5 (NO2)
- new net Stim2_Output: R243.1, U29.6 (COM2)
- new net Stim3_Enable: R22.2, SW16.6 (C)
- new net Stim3_Filtered: C136.1, R44.2, U33.1 (NO1)
- new net Stim3_Output: R244.1, U33.2 (COM1)
- new net Stim4_Enable: R23.1, SW17.6 (C)
- new net Stim4_Filtered: C137.2, R177.2, U33.5 (NO2)
- new net Stim4_Output: R245.1, U33.6 (COM2)
- new net Stim5_Enable: R25.2, SW18.6 (C)
- new net Stim5_Filtered: C148.1, R45.2, U34.1 (NO1)
- new net Stim5_Output: R246.1, U34.2 (COM1)
- new net Stim6_Enable: R26.1, SW20.6 (C)
- new net Stim6_Filtered: C149.2, R180.2, U34.5 (NO2)
- new net Stim6_Output: R247.1, U34.6 (COM2)
- new net Stim7_Enable: R27.2, SW19.6 (C)
- new net Stim7_Filtered: C150.1, R46.2, U35.1 (NO1)
- new net Stim7_Output: R248.1, U35.2 (COM1)
- new net Stim8_Enable: R28.1, SW21.6 (C)
- new net Stim8_Filtered: C151.2, R181.2, U35.5 (NO2)
- new net Stim8_Output: R249.1, U35.6 (COM2)
- new net TOUCH_CS: J1.30 (Pin_30), R128.1
- new net TOUCH_IRQ: J1.34 (Pin_34), R219.2
- new net TUSB320_OUT1: R124.1, U3.7 (SDA/OUT1)
- new net TUSB320_OUT2: R123.1, U3.8 (SCL/OUT2)
- new net USB_D+: J12.A6 (D+), J12.B6 (D+), R107.1, TV1.1
- new net USB_D-: J12.A7 (D-), J12.B7 (D-), R106.1, TV1.3
- new net VBUS_RAW: C87.2, C96.2, D29.1 (C), J12.A9B4 (VBUS), J12.B9A4 (VBUS), R1.1, R2.1, TP7.1, TV1.5, U2.3 (IN), U2.4 (IN)
- new net Vm1_Input: C29.1, D33.3, R13.1, U5.3 (VINA+)
- new net Vm2_Input: C28.1, D35.3, R14.1, U5.5 (VINB+)
- new net Vm3_Input: C25.1, D37.3, R20.1, U5.10 (VINC+)
- new net Vm4_Input: C20.1, D38.3, R15.1, U5.12 (VIND+)
- new net Vm5_Input: C18.1, D41.3, R16.1, U13.3 (VINA+)
- new net Vm6_Input: C17.1, D42.3, R17.1, U13.5 (VINB+)
- new net Vm7_Input: C11.1, D43.3, R18.1, U13.10 (VINC+)
- new net Vm8_Input: C10.1, D44.3, R19.1, U13.12 (VIND+)
- no-connect marks 53 -> 56
Other:
- note added: "3.3 V Digital Rail Generation"
- note added: "Board power tree, source selection, battery management, control electronics, analogue acquisition and external signal interfaces. Distributes power from USB or battery operation and routes the front-panel controls, analogue readout and output signals to the main controller."
- note added: "Brings USB power and USB data onto the board. Provides the Type-C sink configuration, over-current protection and surge/ESD protection before VBUS and the USB data lines are passed into the rest of the system."
- note added: "Command/data selection"
- note added: "Converts the main +5V rail into the regulated +3.3V digital supply used by the controller and digital peripherals. Provides the main low-voltage logic rail for the board."
- note added: "DB8 - DB15 (pin 7 - 14): Unconnected in 8-bit mode"
- note added: "ESP32 Buttons"
- note added: "ESP32-S3 WROOM1 N4"
- note added: "External backlight enable"
- note added: "LCD controller chip select"
- note added: "LCD reset"
- note added: "Module power"
- note added: "NC"
- note added: "NC / Capacitive-touch I²C clock"
- note added: "NC / Capacitive-touch I²C data"
- note added: "NC / Capacitive-touch reset"
- note added: "Optional SPI flash chip select"
- note added: "Parallel write strobe"
- note added: "Power, control and signal interface"
- note added: "Precision voltage reference 2.048V"
- note added: "Protects external connectors and user-accessible signal lines against ESD events and transient over-voltage. Reduces risk of damage or latch-up when cables are plugged, unplugged or mispatched."
- note added: "RD"
- note added: "Reserved external 3.3 V"
- note added: "USB-C entry"
- note removed: "+5V Protected Power Entry & Split-rail Distribution"
- note removed: "Analog 3.3V rail filter"
- note removed: "ESP32"
- note removed: "Mid-rail bias (1.25 V) generator"
- note removed: "Power"
- note removed: "Precision voltage reference 2.5V"
- note removed: "SSD"
- moved on the sheet: J3

Commit message: update pcb oscilloscope
Parts:
- removed C10, C11, C17, C18, C25, C28, C29: 22nF, C0603, symbol 1_P1-altium-import:root_0_0603B223K500NT_
- removed C91: 100nF, JLCPCB:C_0603, symbol CL10B104KB8NNNC1_CL10B104KB8NNNC (2)-altium-import:root_0_CL10B104KB8NNNC_
- removed R189: 10kΩ, JLCPCB:R_0603, symbol FRC0603F1002TS1_FRC0603F1002TS-altium-import:root_0_FRC0603F1002TS_
- added C12: 10uF, C1206, symbol 1_P1-altium-import:root_0_1206B106K100NT_
- added C13: 100nF, C0603, symbol 1_P1-altium-import:root_0_C0603C104J5RAC7867_C490602_
- added C170: 10uF, JLCPCB:C_0805, symbol CL21A106KBYQNNE1_CL21A106KBYQNNE-altium-import:root_0_CL21A106KBYQNNE_
- added C171: 100nF, JLCPCB:C_0603, symbol CL10B104KB8NNNC1_CL10B104KB8NNNC (2)-altium-import:root_0_CL10B104KB8NNNC_
- added C174, C175, C176, C177, C178, C179, C180: 10nF, JLCPCB:C_0603, symbol CC0603KRX7R9BB1031_CC0603KRX7R9BB103 (1)-altium-import:root_0_CC0603KRX7R9BB103_
- added C8: 3.3nF, C0603, symbol Potentiometer_mount_4LED-altium-import:root_0_CC0603KRX7R9BB332_
- added R178, R179, R182, R183, R189, R254, R255, R256, R257: 47Ω, JLCPCB:R_0603, symbol 0603WAF470JT5E1_0603WAF470JT5E-altium-import:root_0_0603WAF470JT5E_
- added R258: 10kΩ, JLCPCB:R_0603, symbol FRC0603F1002TS1_FRC0603F1002TS-altium-import:root_0_FRC0603F1002TS_
- added U4: MCP23S17T-E/SO, SOIC-28_L17.9-W7.5-P1.27-LS10.3-BL, symbol 1_P1-altium-import:root_0_MCP23S17T-E/SO_
Connections:
- net +5V_DSYS is gone; now on net +5V_SYS: TP6.1
- net En is gone; now on net SYS_RESET: C104.1, R114.1, SW12.1, U25.3 (EN)
- net +3.3V: now also J1.2 (Pin_2), C12.2, C13.1, C170.2, C171.2, R258.1, U4.15 (A0), U4.9 (VDD)
- net CS_MCP23S17: now also U4.11 (CS#)
- net GNDA: now also C174.2, C175.2, C176.2, C177.2, C178.2, C179.2, C180.2
- net GNDD: now also C12.1, C13.2, C170.1, C171.1, C8.2, U4.10 (VSS), U4.16 (A1), U4.17 (A2)
- net SPI_MISO: now also U4.14 (SO)
- net SPI_MOSI: now also U4.13 (SI)
- net SPI_SCK: now also U4.12 (SCK)
- net Vm1_Input: now also C174.1
- net Vm2_Input: now also C175.1
- net Vm3_Input: now also C176.1
- net Vm5_Input: now also C177.1
- net Vm6_Input: now also C178.1
- net Vm7_Input: now also C179.1
- net Vm8_Input: now also C180.1
- net at R117.2, R223.2: now also U4.1 (GPB0); no longer U25.39 (IO1)
- net at R220.1, R234.2: now also U4.4 (GPB3); no longer U25.33 (IO40)
- net at R124.2, R253.2: now also U4.23 (GPA2); no longer U25.36 (RXD0)
- net at R126.2, R252.2: now also U4.21 (GPA0); no longer U25.15 (IO3)
- net SYS_RESET: now reaches U1.18 (RESET#)
- net SYS_RESET: now also U4.18 (RESET#)
- net at R222.2, U25.12 (IO8): now also R189.1; no longer R187.2
- net at U2.1 (dVdt): now also C8.1
- net at R123.2, R251.2: now also U4.22 (GPA1); no longer U25.37 (TXD0)
- net at R219.1: now also U4.24 (GPA3); no longer U25.32 (IO39)
- net at R215.2, R216.2: now also U4.25 (GPA4); no longer U25.35 (IO42)
- net at R118.2, R224.2: now also U4.2 (GPB1); no longer U25.38 (IO2)
- net at R163.2, R199.2: now also U4.3 (GPB2); no longer U25.10 (IO17)
- net LCD_DB11: now reaches J1.10 (Pin_10)
- net LCD_DB11: now also R255.2
- net LCD_DB12: now reaches J1.11 (Pin_11)
- net LCD_DB12: now also R257.2
- net LCD_DB13: now reaches J1.12 (Pin_12)
- net LCD_DB13: now also R256.2
- net LCD_DB14: now reaches J1.13 (Pin_13)
- net LCD_DB14: now also R183.2
- net LCD_DB15: now reaches J1.14 (Pin_14)
- net LCD_DB15: now also R254.2
- net LCD_Flash_CS: now reaches J1.16 (Pin_16)
- net LCD_Flash_CS: now also R189.2
- net LCD_DB8: now reaches J1.7 (Pin_7)
- net LCD_DB8: now also R178.2
- net LCD_DB9: now reaches J1.8 (Pin_8)
- net LCD_DB9: now also R179.2
- net LCD_DB10: now reaches J1.9 (Pin_9)
- net LCD_DB10: now also R182.2
- net Boot renamed BOOT
- net LCD_Reset renamed LCD_RESET
- net Rot_OutA renamed ROT_A
- net Rot_OutB renamed ROT_B
- net Rot_Switch renamed ROT_SW
- new net: R257.1, U25.33 (IO40)
- new net: R187.2, R258.2, U4.5 (GPB4)
- new net: R182.1, U25.10 (IO17)
- new net: R179.1, U25.38 (IO2)
- new net: R256.1, U25.35 (IO42)
- new net: R183.1, U25.37 (TXD0)
- new net: R178.1, U25.39 (IO1)
- new net: R255.1, U25.32 (IO39)
- new net: R254.1, U25.36 (RXD0)
- no-connect marks 56 -> 49
Other:
- note added: "Flash chip select"
- note removed: "DB8 - DB15 (pin 7 - 14): Unconnected in 8-bit mode"
- note removed: "Optional SPI flash chip select"
- note removed: "Reserved external 3.3 V"
- moved on the sheet: R117, R118, R123, R124, R126, R163, R187, R199, R215, R216, R219, R220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
